File: usb-charging-hub.kicad_pcb (KiCad board)
At the start: 4 copper layers, 100 x 100 mm, 0 parts

Commit message: gave up on single board, gonna make small modules
Signed-off-by: Toby Cm <toby@vsus.app>
Other:
- copper layers 4 -> 2
Changed lines of the file:
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@@
 	(layers
 		(0 "F.Cu" signal)
-		(4 "In1.Cu" signal)
-		(6 "In2.Cu" signal)
 		(2 "B.Cu" signal)
 		(9 "F.Adhes" user "F.Adhesive")
@@
 			)
 			(layer "dielectric 1"
-				(type "prepreg")
-				(thickness 0.1)
-				(material "FR4")
-				(epsilon_r 4.5)
-				(loss_tangent 0.02)
-			)
-			(layer "In1.Cu"
-				(type "copper")
-				(thickness 0.035)
-			)
-			(layer "dielectric 2"
 				(type "core")
-				(thickness 1.24)
-				(material "FR4")
-				(epsilon_r 4.5)
-				(loss_tangent 0.02)
-			)
-			(layer "In2.Cu"
-				(type "copper")
-				(thickness 0.035)
-			)
-			(layer "dielectric 3"
-				(type "prepreg")
-				(thickness 0.1)
+				(thickness 1.51)
 				(material "FR4")
 				(epsilon_r 4.5)
@@
 		)
 		(fill no)
+		(locked yes)
 		(layer "Edge.Cuts")
 	)

Commit message: updated journal, pin headers footprint, etc. added labels to rp2350b, finished pcb routing. time to start on other modules yay
Signed-off-by: Toby Cm <toby@vsus.app>
Parts:
- added C1: 50V,1000uF, Capacitor_THT:CP_Radial_D13.0mm_P7.50mm, F.Cu at (243.9, 101.4)
- added C10: 50V,1uF, Capacitor_SMD:C_0603_1608Metric_Pad1.08x0.95mm_HandSolder, F.Cu at (139.4, 150.4)
- added C11: 35V,470uF, Capacitor_THT:CP_Radial_D10.0mm_P5.00mm, B.Cu at (129.0, 140.0)
- added C12: 10V,10uF, Capacitor_SMD:C_0603_1608Metric_Pad1.08x0.95mm_HandSolder, F.Cu at (142.8, 150.4)
- added C13: 50V,10uF, Capacitor_SMD:C_1206_3216Metric_Pad1.33x1.80mm_HandSolder, F.Cu at (360.0, 192.4)
- added C14: 35V,180uF, Capacitor_THT:CP_Radial_D8.0mm_P5.00mm, F.Cu at (349.7, 195.6)
- added C15: 35V,22uF, Capacitor_SMD:C_0805_2012Metric_Pad1.18x1.45mm_HandSolder, F.Cu at (329.1, 174.6)
- added C16: 100nF, Capacitor_SMD:C_0201_0603Metric_Pad0.64x0.40mm_HandSolder, F.Cu at (105.4, 143.0)
- added C17: 100nF, Capacitor_SMD:C_0201_0603Metric_Pad0.64x0.40mm_HandSolder, F.Cu at (106.0, 143.5)
- added C18: 100nF, Capacitor_SMD:C_0201_0603Metric_Pad0.64x0.40mm_HandSolder, F.Cu at (92.8, 145.9)
- added C19: 100nF, Capacitor_SMD:C_0201_0603Metric_Pad0.64x0.40mm_HandSolder, F.Cu at (93.4, 142.1)
- added C2: 50V,1000uF, Capacitor_THT:CP_Radial_D13.0mm_P7.50mm, F.Cu at (273.8, 101.8)
- added C20: 100nF, Capacitor_SMD:C_0201_0603Metric_Pad0.64x0.40mm_HandSolder, F.Cu at (92.9, 150.5)
- added C21: 100nF, Capacitor_SMD:C_0201_0603Metric_Pad0.64x0.40mm_HandSolder, F.Cu at (94.1, 154.4)
- added C22: 100nF, Capacitor_SMD:C_0201_0603Metric_Pad0.64x0.40mm_HandSolder, F.Cu at (105.2, 148.3)
- added C23: 100nF, Capacitor_SMD:C_0201_0603Metric_Pad0.64x0.40mm_HandSolder, F.Cu at (105.5, 152.2)
- added C3: 100nF, Capacitor_SMD:C_0201_0603Metric_Pad0.64x0.40mm_HandSolder, F.Cu at (100.3, 141.8)
- added C4: 4.7uF, Capacitor_SMD:C_0603_1608Metric_Pad1.08x0.95mm_HandSolder, F.Cu at (101.7, 141.0)
- added C5: 4.7uF, Capacitor_SMD:C_0603_1608Metric_Pad1.08x0.95mm_HandSolder, F.Cu at (105.1, 139.1)
- added C6: 4.7uF, Capacitor_SMD:C_0603_1608Metric_Pad1.08x0.95mm_HandSolder, F.Cu at (107.0, 139.1)
- added C7: 18pF, Capacitor_SMD:C_0201_0603Metric_Pad0.64x0.40mm_HandSolder, F.Cu at (99.0, 156.7)
- added C8: 18pF, Capacitor_SMD:C_0201_0603Metric_Pad0.64x0.40mm_HandSolder, F.Cu at (93.6, 156.7)
- added C9: 50V,470uF, Capacitor_THT:CP_Radial_D10.0mm_P5.00mm, F.Cu at (157.2, 140.6)
- added D1: LED, LED_SMD:LED_0603_1608Metric_Pad1.05x0.95mm_HandSolder, F.Cu at (244.3, 87.1)
- added D10: 40V,10A, Diode_SMD:D_SMB_Handsoldering, F.Cu at (247.0, -68.4)
- added D2: Green, LED_SMD:LED_0603_1608Metric_Pad1.05x0.95mm_HandSolder, F.Cu at (107.6, 146.5)
- added D3: Green, LED_SMD:LED_0603_1608Metric_Pad1.05x0.95mm_HandSolder, F.Cu at (107.6, 148.0)
- added D4: Amber, LED_SMD:LED_0603_1608Metric_Pad1.05x0.95mm_HandSolder, F.Cu at (107.6, 149.4)
- added D5: Amber, LED_SMD:LED_0603_1608Metric_Pad1.05x0.95mm_HandSolder, F.Cu at (107.6, 150.9)
- added D6: Red, LED_SMD:LED_0603_1608Metric_Pad1.05x0.95mm_HandSolder, F.Cu at (107.6, 152.3)
- added D7: Red, LED_SMD:LED_0603_1608Metric_Pad1.05x0.95mm_HandSolder, F.Cu at (107.6, 153.8)
- added D8: 40V,10A, Diode_SMD:D_SMB_Handsoldering, F.Cu at (133.8, 139.8)
- added D9: 40V,10A, Diode_SMD:D_SMB_Handsoldering, F.Cu at (328.3, 213.9)
- added J1: Conn_01x01_Pin, MountingHole:MountingHole_4.3x6.2mm_M4_Pad_Via, F.Cu at (263.2, 88.8)
- added J10: Conn_01x04_Pin, Connector_PinHeader_2.54mm:PinHeader_1x04_P2.54mm_Vertical, F.Cu at (124.5, 142.2)
- added J11: Conn_01x04_Pin, Connector_PinHeader_2.54mm:PinHeader_1x04_P2.54mm_Vertical, F.Cu at (149.9, 134.6)
- added J12: Conn_01x04_Pin, Connector_PinHeader_2.54mm:PinHeader_1x04_P2.54mm_Vertical, F.Cu at (389.1, 201.0)
- added J13: Conn_01x04_Pin, Connector_PinHeader_2.54mm:PinHeader_1x04_P2.54mm_Vertical, F.Cu at (393.7, 201.0)
- added J14: Conn_01x04_Pin, Connector_PinHeader_2.54mm:PinHeader_1x04_P2.54mm_Vertical, F.Cu at (239.4, -62.1)
- added J15: Conn_01x04_Pin, Connector_PinHeader_2.54mm:PinHeader_1x04_P2.54mm_Vertical, F.Cu at (268.8, -54.1)
- added J16: TYPE-C 16PLT-H10.0, easyeda2kicad:TYPE-C-SMD_USB4120-03-C, F.Cu at (247.5, -79.9)
- added J17: Conn_01x04_Pin, Connector_PinHeader_2.54mm:PinHeader_1x04_P2.54mm_Vertical, F.Cu at (251.9, -59.4)
- added J2: Conn_01x01_Pin, MountingHole:MountingHole_4.3x6.2mm_M4_Pad_Via, F.Cu at (265.4, 113.1)
- added J20: Conn_01x02_Pin, Connector_PinHeader_2.54mm:PinHeader_1x02_P2.54mm_Vertical, F.Cu at (111.8, 134.6)
- added J21: Conn_01x04_Pin, Connector_PinHeader_2.54mm:PinHeader_2x02_P2.54mm_Vertical, F.Cu at (111.8, 147.3)
- added J23: Conn_01x02_Pin, Connector_PinHeader_2.54mm:PinHeader_1x02_P2.54mm_Vertical, F.Cu at (104.1, 134.6)
- added J3: Conn_01x10_Pin, Connector_PinHeader_2.54mm:PinHeader_1x10_P2.54mm_Vertical, F.Cu at (83.8, 134.6)
- added J4: Conn_01x10_Pin, Connector_PinHeader_2.54mm:PinHeader_1x10_P2.54mm_Vertical, F.Cu at (88.9, 134.6)
- added J7: Conn_01x10_Pin, Connector_PinHeader_2.54mm:PinHeader_1x10_P2.54mm_Vertical, F.Cu at (119.4, 157.5)
- added J8: Conn_01x06_Pin, Connector_PinHeader_2.54mm:PinHeader_1x06_P2.54mm_Vertical, F.Cu at (-59.6, 12.5)
- added J9: Conn_01x06_Pin, Connector_PinHeader_2.54mm:PinHeader_1x06_P2.54mm_Vertical, F.Cu at (-64.3, 40.3)
- added JP1: SolderJumper_2_Bridged, Jumper:SolderJumper-2_P1.3mm_Bridged_Pad1.0x1.5mm, F.Cu at (244.2, 90.1)
- added L1: AOTA-B201610S3R3-101-T, easyeda2kicad:IND-SMD_L2.0-W1.6_AOTA-B201610S3R3-101-T, F.Cu at (103.5, 140.7)
- added L2: 33uH,4.25A, misc:SDRI129-330MT, F.Cu at (129.5, 159.9)
- added L3: YPRH1508-680M, easyeda2kicad:IND-SMD_L15.0-W15.0, F.Cu at (355.9, 182.7)
- added R1: 1.5k, Resistor_SMD:R_1210_3225Metric_Pad1.30x2.65mm_HandSolder, F.Cu at (245.1, 83.7)
- added R10: 5.1k, Resistor_SMD:R_0402_1005Metric_Pad0.72x0.64mm_HandSolder, F.Cu at (246.5, -36.3)
- added R11: 5.1k, Resistor_SMD:R_0402_1005Metric_Pad0.72x0.64mm_HandSolder, F.Cu at (246.5, -34.3)
- added R12: 5.1k, Resistor_SMD:R_0402_1005Metric_Pad0.72x0.64mm_HandSolder, F.Cu at (239.2, -82.2)
- added R13: 5.1k, Resistor_SMD:R_0402_1005Metric_Pad0.72x0.64mm_HandSolder, F.Cu at (239.4, -85.0)
- added R14: 1k, Resistor_SMD:R_0402_1005Metric_Pad0.72x0.64mm_HandSolder, F.Cu at (108.1, 155.2)
- added R15: 1k, Resistor_SMD:R_0402_1005Metric_Pad0.72x0.64mm_HandSolder, F.Cu at (102.2, 155.2)
- added R2: 33, Resistor_SMD:R_0402_1005Metric_Pad0.72x0.64mm_HandSolder, F.Cu at (106.2, 141.5)
- added R3: 27, Resistor_SMD:R_0402_1005Metric_Pad0.72x0.64mm_HandSolder, F.Cu at (102.4, 136.9)
- added R4: 27, Resistor_SMD:R_0402_1005Metric_Pad0.72x0.64mm_HandSolder, F.Cu at (102.4, 138.0)
- added R5: 1k, Resistor_SMD:R_0402_1005Metric_Pad0.72x0.64mm_HandSolder, F.Cu at (97.6, 154.6)
- added R8: 100k, Resistor_SMD:R_0402_1005Metric_Pad0.72x0.64mm_HandSolder, F.Cu at (145.4, 151.0)
- added R9: 100k, Resistor_SMD:R_0402_1005Metric_Pad0.72x0.64mm_HandSolder, F.Cu at (342.5, 209.3)
- added SW1: Latching, easyeda2kicad:SW-TH_6P-L8.0-W8.0-P2.50, F.Cu at (111.7, 140.5)
- added SW2: TS24CA, easyeda2kicad:SW-SMD_TS24CA, F.Cu at (108.1, 157.1)
- added SW3: TS24CA, easyeda2kicad:SW-SMD_TS24CA, F.Cu at (102.2, 157.1)
- added SW4: TS24CA, easyeda2kicad:SW-SMD_TS24CA, F.Cu at (114.0, 157.1)
- added TP1: TestPoint, TestPoint:TestPoint_Pad_D2.0mm, F.Cu at (-103.0, 27.7)
- added TP2: TestPoint, TestPoint:TestPoint_Pad_D2.0mm, F.Cu at (-90.3, 17.2)
- added TP3: TestPoint, TestPoint:TestPoint_Pad_D2.0mm, F.Cu at (-107.5, 31.8)
- added U1: W25Q32JVSS, Package_SO:SOIC-8_5.3x5.3mm_P1.27mm, F.Cu at (96.8, 138.3)
- added U2: RP2350B_C42415655, easyeda2kicad:QFN-80_L10.0-W10.0-P0.40-TL-EP3.4, F.Cu at (99.0, 148.2)
- added U3: ABM8-272-T3_C20625731, easyeda2kicad:CRYSTAL-SMD_4P-L3.2-W2.5-BL, F.Cu at (96.3, 156.8)
- added U4: PUSB3FR4-ES, Package_DFN_QFN:Diodes_UDFN-10_1.0x2.5mm_P0.5mm, F.Cu at (-79.4, 31.5)
- added U5: XDUF-0426-081_C18202150, easyeda2kicad:USB-A-TH_XDUF-0426-081, F.Cu at (-99.6, 41.6)
- added U6: RH792A, easyeda2kicad:SOT-23-6_L2.9-W1.6-P0.95-LS2.9-BL, F.Cu at (-88.8, 27.8)
- added U7: LM2596S-3.3, Package_TO_SOT_SMD:TO-263-5_TabPin3, F.Cu at (142.0, 139.3)
- added U8: XXL1509-5.0, easyeda2kicad:SOIC-8_L4.9-W3.9-P1.27-LS6.0-BL, F.Cu at (386.4, 194.5)
- added U9: PUSB3FR4-ES, Package_DFN_QFN:Diodes_UDFN-10_1.0x2.5mm_P0.5mm, F.Cu at (251.0, -87.8)
Routing:
- net GND: track 0.00 -> 57.4 mm, vias 0 -> 35
- net +1V1: track 0.00 -> 42.0 mm, vias 0 -> 3
- net QSPI_SS: track 0.00 -> 28.4 mm, vias 0 -> 4
- net GPIO44: track 0.00 -> 27.4 mm, vias 0 -> 2
- net GPIO42: track 0.00 -> 25.4 mm, vias 0 -> 1
- net GPIO41: track 0.00 -> 24.7 mm, vias 0 -> 1
- net GPIO40: track 0.00 -> 21.8 mm, vias 0 -> 1
- net GPIO47: track 0.00 -> 21.1 mm, vias 0 -> 1
- net GPIO43: track 0.00 -> 19.9 mm, vias 0 -> 3
- net GPIO46: track 0.00 -> 19.2 mm, vias 0 -> 1
- net GPIO7: track 0.00 -> 19.1 mm, vias 0 -> 1
- net GPIO0: track 0.00 -> 18.7 mm, vias 0 -> 1
- net GPIO6: track 0.00 -> 18.0 mm, vias 0 -> 1
- net +3.3V: track 0.00 -> 17.8 mm, vias 0 -> 2
- net GPIO45: track 0.00 -> 17.6 mm, vias 0 -> 1
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- added copper zone on F.Cu, net +3.3V
- added copper zone on B.Cu, net GND
- added copper zone on F.Cu, net GND
Other:
- board size 100 x 100 mm -> 76 x 26 mm
- board text added: "0"
- board text added: "1"
- board text added: "1.1V>"
- board text added: "10"
- board text added: "11"
- board text added: "12"
- board text added: "13"
- board text added: "14"
- board text added: "15"
- board text added: "2"
- board text added: "3"
- board text added: "3.3V"
- board text added: "32"
- board text added: "33"
- board text added: "38"
- board text added: "39"
- board text added: "4"
- board text added: "40"
- board text added: "41"
- board text added: "42"
- board text added: "43"
- board text added: "44"
- board text added: "45"
- board text added: "46"
- board text added: "47"
- board text added: "5"
- board text added: "6"
- board text added: "7"
- board text added: "8"
- board text added: "9"
- board text added: "<USB"
- board text added: "D+"
- board text added: "D-"

Commit message: no more modules, its gonna work first try :fire: i love infineon and their ICs so much
Signed-off-by: Toby Cm <toby@vsus.app>
Parts:
- removed R8: 100k, Resistor_SMD:R_0402_1005Metric_Pad0.72x0.64mm_HandSolder
- removed TP1, TP2, TP3: TestPoint, TestPoint:TestPoint_Pad_D2.0mm
- added C100: 100nF, Capacitor_SMD:C_0201_0603Metric_Pad0.64x0.40mm_HandSolder, F.Cu at (65.6, 107.9)
- added C101: 1uF, Capacitor_SMD:C_0402_1005Metric_Pad0.74x0.62mm_HandSolder, F.Cu at (73.3, 130.1)
- added C102: 100nF, Capacitor_SMD:C_0201_0603Metric_Pad0.64x0.40mm_HandSolder, F.Cu at (65.6, 109.7)
- added C103: 1uF, Capacitor_SMD:C_0402_1005Metric_Pad0.74x0.62mm_HandSolder, F.Cu at (73.3, 132.1)
- added C104: 100nF, Capacitor_SMD:C_0201_0603Metric_Pad0.64x0.40mm_HandSolder, F.Cu at (65.6, 111.4)
- added C105: 100nF, Capacitor_SMD:C_0201_0603Metric_Pad0.64x0.40mm_HandSolder, F.Cu at (68.4, 106.2)
- added C106: 1uF, Capacitor_SMD:C_0402_1005Metric_Pad0.74x0.62mm_HandSolder, F.Cu at (73.3, 134.0)
- added C107: 1uF, Capacitor_SMD:C_0402_1005Metric_Pad0.74x0.62mm_HandSolder, F.Cu at (73.3, 136.0)
- added C108: 390pF 5% X7R, Capacitor_SMD:C_0603_1608Metric_Pad1.08x0.95mm_HandSolder, F.Cu at (69.5, 127.5)
- added C109: 390pF 5% X7R, Capacitor_SMD:C_0603_1608Metric_Pad1.08x0.95mm_HandSolder, F.Cu at (69.5, 130.0)
- added C110: 100pF, Capacitor_SMD:C_0201_0603Metric_Pad0.64x0.40mm_HandSolder, F.Cu at (68.4, 107.9)
- added C111: 1nF, Capacitor_SMD:C_0201_0603Metric_Pad0.64x0.40mm_HandSolder, F.Cu at (68.4, 109.7)
- added C112: 100nF, Capacitor_SMD:C_0201_0603Metric_Pad0.64x0.40mm_HandSolder, F.Cu at (68.4, 111.4)
- added C113: 50V,10uF, Capacitor_SMD:C_1206_3216Metric_Pad1.33x1.80mm_HandSolder, F.Cu at (178.5, 49.8)
- added C114: 50V,10uF, Capacitor_SMD:C_1206_3216Metric_Pad1.33x1.80mm_HandSolder, F.Cu at (178.5, 53.1)
- added C115: 35V,180uF, Capacitor_THT:CP_Radial_D8.0mm_P5.00mm, F.Cu at (167.4, 33.1)
- added C116: 35V,22uF, Capacitor_SMD:C_0805_2012Metric_Pad1.18x1.45mm_HandSolder, F.Cu at (183.0, 42.6)
- added C117: 35V,180uF, Capacitor_THT:CP_Radial_D8.0mm_P5.00mm, F.Cu at (167.4, 42.6)
- added C118: 35V,22uF, Capacitor_SMD:C_0805_2012Metric_Pad1.18x1.45mm_HandSolder, F.Cu at (183.0, 45.6)
- added C119: 100nF, Capacitor_SMD:C_0201_0603Metric_Pad0.64x0.40mm_HandSolder, F.Cu at (168.5, 49.0)
- added C120: 1uF, Capacitor_SMD:C_0402_1005Metric_Pad0.74x0.62mm_HandSolder, F.Cu at (179.0, 65.0)
- added C121: 1uF, Capacitor_SMD:C_0402_1005Metric_Pad0.74x0.62mm_HandSolder, F.Cu at (179.0, 67.0)
- added C122: 390pF 5% X7R, Capacitor_SMD:C_0603_1608Metric_Pad1.08x0.95mm_HandSolder, F.Cu at (175.2, 65.3)
- added C123: 390pF 5% X7R, Capacitor_SMD:C_0603_1608Metric_Pad1.08x0.95mm_HandSolder, F.Cu at (175.2, 67.8)
- added C124: 100pF, Capacitor_SMD:C_0201_0603Metric_Pad0.64x0.40mm_HandSolder, F.Cu at (168.5, 50.7)
- added C125: 1nF, Capacitor_SMD:C_0201_0603Metric_Pad0.64x0.40mm_HandSolder, F.Cu at (168.5, 52.5)
- added C126: 100nF, Capacitor_SMD:C_0201_0603Metric_Pad0.64x0.40mm_HandSolder, F.Cu at (168.5, 54.2)
- added C127: 1uF, Capacitor_SMD:C_0402_1005Metric_Pad0.74x0.62mm_HandSolder, F.Cu at (179.0, 69.0)
- added C128: 100nF, Capacitor_SMD:C_0201_0603Metric_Pad0.64x0.40mm_HandSolder, F.Cu at (171.3, 49.0)
- added C129: 1uF, Capacitor_SMD:C_0402_1005Metric_Pad0.74x0.62mm_HandSolder, F.Cu at (179.0, 71.0)
- added C130: 100nF, Capacitor_SMD:C_0201_0603Metric_Pad0.64x0.40mm_HandSolder, F.Cu at (171.3, 50.7)
- added C131: 1uF, Capacitor_SMD:C_0402_1005Metric_Pad0.74x0.62mm_HandSolder, F.Cu at (179.0, 72.9)
- added C132: 100nF, Capacitor_SMD:C_0201_0603Metric_Pad0.64x0.40mm_HandSolder, F.Cu at (171.3, 52.5)
- added C133: 1uF, Capacitor_SMD:C_0402_1005Metric_Pad0.74x0.62mm_HandSolder, F.Cu at (179.0, 74.9)
- added C134: 100nF, Capacitor_SMD:C_0201_0603Metric_Pad0.64x0.40mm_HandSolder, F.Cu at (171.3, 54.2)
- added C135: 100nF, Capacitor_SMD:C_0201_0603Metric_Pad0.64x0.40mm_HandSolder, F.Cu at (174.1, 49.0)
- added C136: 1uF, Capacitor_SMD:C_0402_1005Metric_Pad0.74x0.62mm_HandSolder, F.Cu at (179.0, 76.9)
- added C137: 1uF, Capacitor_SMD:C_0402_1005Metric_Pad0.74x0.62mm_HandSolder, F.Cu at (179.0, 78.8)
- added C138: 390pF 5% X7R, Capacitor_SMD:C_0603_1608Metric_Pad1.08x0.95mm_HandSolder, F.Cu at (175.2, 70.3)
- added C139: 390pF 5% X7R, Capacitor_SMD:C_0603_1608Metric_Pad1.08x0.95mm_HandSolder, F.Cu at (175.2, 72.8)
- added C140: 100pF, Capacitor_SMD:C_0201_0603Metric_Pad0.64x0.40mm_HandSolder, F.Cu at (174.1, 50.7)
- added C141: 1nF, Capacitor_SMD:C_0201_0603Metric_Pad0.64x0.40mm_HandSolder, F.Cu at (174.1, 52.5)
- added C142: 100nF, Capacitor_SMD:C_0201_0603Metric_Pad0.64x0.40mm_HandSolder, F.Cu at (174.1, 54.2)
- added C143: 50V,10uF, Capacitor_SMD:C_1206_3216Metric_Pad1.33x1.80mm_HandSolder, F.Cu at (72.8, 49.8)
- added C144: 50V,10uF, Capacitor_SMD:C_1206_3216Metric_Pad1.33x1.80mm_HandSolder, F.Cu at (72.8, 53.1)
- added C145: 35V,180uF, Capacitor_THT:CP_Radial_D8.0mm_P5.00mm, F.Cu at (61.6, 33.1)
- added C146: 35V,22uF, Capacitor_SMD:C_0805_2012Metric_Pad1.18x1.45mm_HandSolder, F.Cu at (77.3, 42.6)
- added C147: 35V,180uF, Capacitor_THT:CP_Radial_D8.0mm_P5.00mm, F.Cu at (61.6, 42.6)
- added C148: 35V,22uF, Capacitor_SMD:C_0805_2012Metric_Pad1.18x1.45mm_HandSolder, F.Cu at (77.3, 45.6)
- added C149: 100nF, Capacitor_SMD:C_0201_0603Metric_Pad0.64x0.40mm_HandSolder, F.Cu at (62.8, 49.0)
- added C150: 1uF, Capacitor_SMD:C_0402_1005Metric_Pad0.74x0.62mm_HandSolder, F.Cu at (73.3, 65.0)
- added C151: 1uF, Capacitor_SMD:C_0402_1005Metric_Pad0.74x0.62mm_HandSolder, F.Cu at (73.3, 67.0)
- added C152: 390pF 5% X7R, Capacitor_SMD:C_0603_1608Metric_Pad1.08x0.95mm_HandSolder, F.Cu at (69.5, 65.3)
- added C153: 390pF 5% X7R, Capacitor_SMD:C_0603_1608Metric_Pad1.08x0.95mm_HandSolder, F.Cu at (69.5, 67.8)
- added C154: 100pF, Capacitor_SMD:C_0201_0603Metric_Pad0.64x0.40mm_HandSolder, F.Cu at (62.8, 50.7)
- added C155: 1nF, Capacitor_SMD:C_0201_0603Metric_Pad0.64x0.40mm_HandSolder, F.Cu at (62.8, 52.5)
- added C156: 100nF, Capacitor_SMD:C_0201_0603Metric_Pad0.64x0.40mm_HandSolder, F.Cu at (62.8, 54.2)
- added C157: 1uF, Capacitor_SMD:C_0402_1005Metric_Pad0.74x0.62mm_HandSolder, F.Cu at (73.3, 69.0)
- added C158: 100nF, Capacitor_SMD:C_0201_0603Metric_Pad0.64x0.40mm_HandSolder, F.Cu at (65.6, 49.0)
- added C159: 1uF, Capacitor_SMD:C_0402_1005Metric_Pad0.74x0.62mm_HandSolder, F.Cu at (73.3, 71.0)
- added C160: 100nF, Capacitor_SMD:C_0201_0603Metric_Pad0.64x0.40mm_HandSolder, F.Cu at (65.6, 50.7)
- added C161: 1uF, Capacitor_SMD:C_0402_1005Metric_Pad0.74x0.62mm_HandSolder, F.Cu at (73.3, 72.9)
- added C162: 100nF, Capacitor_SMD:C_0201_0603Metric_Pad0.64x0.40mm_HandSolder, F.Cu at (65.6, 52.5)
- added C163: 1uF, Capacitor_SMD:C_0402_1005Metric_Pad0.74x0.62mm_HandSolder, F.Cu at (73.3, 74.9)
- added C164: 100nF, Capacitor_SMD:C_0201_0603Metric_Pad0.64x0.40mm_HandSolder, F.Cu at (65.6, 54.2)
- added C165: 100nF, Capacitor_SMD:C_0201_0603Metric_Pad0.64x0.40mm_HandSolder, F.Cu at (68.4, 49.0)
- added C166: 1uF, Capacitor_SMD:C_0402_1005Metric_Pad0.74x0.62mm_HandSolder, F.Cu at (73.3, 76.9)
- added C167: 1uF, Capacitor_SMD:C_0402_1005Metric_Pad0.74x0.62mm_HandSolder, F.Cu at (73.3, 78.8)
- added C168: 390pF 5% X7R, Capacitor_SMD:C_0603_1608Metric_Pad1.08x0.95mm_HandSolder, F.Cu at (69.5, 70.3)
- added C169: 390pF 5% X7R, Capacitor_SMD:C_0603_1608Metric_Pad1.08x0.95mm_HandSolder, F.Cu at (69.5, 72.8)
- added C170: 100pF, Capacitor_SMD:C_0201_0603Metric_Pad0.64x0.40mm_HandSolder, F.Cu at (68.4, 50.7)
- added C171: 1nF, Capacitor_SMD:C_0201_0603Metric_Pad0.64x0.40mm_HandSolder, F.Cu at (68.4, 52.5)
- added C172: 100nF, Capacitor_SMD:C_0201_0603Metric_Pad0.64x0.40mm_HandSolder, F.Cu at (68.4, 54.2)
- added C24: 50V,10uF, Capacitor_SMD:C_1206_3216Metric_Pad1.33x1.80mm_HandSolder, F.Cu at (125.7, 53.1)
- added C25: 35V,180uF, Capacitor_THT:CP_Radial_D8.0mm_P5.00mm, F.Cu at (114.5, 33.1)
- added C26: 35V,22uF, Capacitor_SMD:C_0805_2012Metric_Pad1.18x1.45mm_HandSolder, F.Cu at (130.1, 42.6)
- added C27: 35V,180uF, Capacitor_THT:CP_Radial_D8.0mm_P5.00mm, F.Cu at (114.5, 42.6)
- added C28: 35V,22uF, Capacitor_SMD:C_0805_2012Metric_Pad1.18x1.45mm_HandSolder, F.Cu at (130.1, 45.6)
- added C29: 100nF, Capacitor_SMD:C_0201_0603Metric_Pad0.64x0.40mm_HandSolder, F.Cu at (115.7, 49.0)
- added C30: 1uF, Capacitor_SMD:C_0402_1005Metric_Pad0.74x0.62mm_HandSolder, F.Cu at (126.1, 65.0)
- added C31: 1uF, Capacitor_SMD:C_0402_1005Metric_Pad0.74x0.62mm_HandSolder, F.Cu at (126.1, 67.0)
- added C32: 390pF 5% X7R, Capacitor_SMD:C_0603_1608Metric_Pad1.08x0.95mm_HandSolder, F.Cu at (122.3, 65.3)
- added C33: 390pF 5% X7R, Capacitor_SMD:C_0603_1608Metric_Pad1.08x0.95mm_HandSolder, F.Cu at (122.3, 67.8)
- added C34: 100pF, Capacitor_SMD:C_0201_0603Metric_Pad0.64x0.40mm_HandSolder, F.Cu at (115.7, 50.7)
- added C35: 1nF, Capacitor_SMD:C_0201_0603Metric_Pad0.64x0.40mm_HandSolder, F.Cu at (115.7, 52.5)
- added C36: 100nF, Capacitor_SMD:C_0201_0603Metric_Pad0.64x0.40mm_HandSolder, F.Cu at (115.7, 54.2)
- added C37: 1uF, Capacitor_SMD:C_0402_1005Metric_Pad0.74x0.62mm_HandSolder, F.Cu at (126.1, 69.0)
- added C38: 100nF, Capacitor_SMD:C_0201_0603Metric_Pad0.64x0.40mm_HandSolder, F.Cu at (118.5, 49.0)
- added C39: 1uF, Capacitor_SMD:C_0402_1005Metric_Pad0.74x0.62mm_HandSolder, F.Cu at (126.1, 71.0)
- added C40: 100nF, Capacitor_SMD:C_0201_0603Metric_Pad0.64x0.40mm_HandSolder, F.Cu at (118.5, 50.7)
- added C41: 1uF, Capacitor_SMD:C_0402_1005Metric_Pad0.74x0.62mm_HandSolder, F.Cu at (126.1, 72.9)
- added C42: 100nF, Capacitor_SMD:C_0201_0603Metric_Pad0.64x0.40mm_HandSolder, F.Cu at (118.5, 52.5)
- added C43: 1uF, Capacitor_SMD:C_0402_1005Metric_Pad0.74x0.62mm_HandSolder, F.Cu at (126.1, 74.9)
- added C44: 100nF, Capacitor_SMD:C_0201_0603Metric_Pad0.64x0.40mm_HandSolder, F.Cu at (118.5, 54.2)
- added C45: 100nF, Capacitor_SMD:C_0201_0603Metric_Pad0.64x0.40mm_HandSolder, F.Cu at (121.3, 49.0)
- added C46: 1uF, Capacitor_SMD:C_0402_1005Metric_Pad0.74x0.62mm_HandSolder, F.Cu at (126.1, 76.9)
- added C47: 1uF, Capacitor_SMD:C_0402_1005Metric_Pad0.74x0.62mm_HandSolder, F.Cu at (126.1, 78.8)
- added C48: 390pF 5% X7R, Capacitor_SMD:C_0603_1608Metric_Pad1.08x0.95mm_HandSolder, F.Cu at (122.3, 70.3)
- added C49: 390pF 5% X7R, Capacitor_SMD:C_0603_1608Metric_Pad1.08x0.95mm_HandSolder, F.Cu at (122.3, 72.8)
- added C50: 100pF, Capacitor_SMD:C_0201_0603Metric_Pad0.64x0.40mm_HandSolder, F.Cu at (121.3, 50.7)
- added C51: 1nF, Capacitor_SMD:C_0201_0603Metric_Pad0.64x0.40mm_HandSolder, F.Cu at (121.3, 52.5)
- added C52: 100nF, Capacitor_SMD:C_0201_0603Metric_Pad0.64x0.40mm_HandSolder, F.Cu at (121.3, 54.2)
- added C53: 50V,10uF, Capacitor_SMD:C_1206_3216Metric_Pad1.33x1.80mm_HandSolder, F.Cu at (125.7, 107.0)
- added C54: 50V,10uF, Capacitor_SMD:C_1206_3216Metric_Pad1.33x1.80mm_HandSolder, F.Cu at (125.7, 110.3)
- added C55: 35V,180uF, Capacitor_THT:CP_Radial_D8.0mm_P5.00mm, F.Cu at (114.5, 90.3)
- added C56: 35V,22uF, Capacitor_SMD:C_0805_2012Metric_Pad1.18x1.45mm_HandSolder, F.Cu at (130.1, 99.8)
- added C57: 35V,180uF, Capacitor_THT:CP_Radial_D8.0mm_P5.00mm, F.Cu at (114.5, 99.8)
- added C58: 35V,22uF, Capacitor_SMD:C_0805_2012Metric_Pad1.18x1.45mm_HandSolder, F.Cu at (130.1, 102.8)
- added C59: 100nF, Capacitor_SMD:C_0201_0603Metric_Pad0.64x0.40mm_HandSolder, F.Cu at (115.7, 106.2)
- added C60: 1uF, Capacitor_SMD:C_0402_1005Metric_Pad0.74x0.62mm_HandSolder, F.Cu at (126.1, 122.2)
- added C61: 1uF, Capacitor_SMD:C_0402_1005Metric_Pad0.74x0.62mm_HandSolder, F.Cu at (126.1, 124.2)
- added C62: 390pF 5% X7R, Capacitor_SMD:C_0603_1608Metric_Pad1.08x0.95mm_HandSolder, F.Cu at (122.3, 122.5)
- added C63: 390pF 5% X7R, Capacitor_SMD:C_0603_1608Metric_Pad1.08x0.95mm_HandSolder, F.Cu at (122.3, 125.0)
- added C64: 100pF, Capacitor_SMD:C_0201_0603Metric_Pad0.64x0.40mm_HandSolder, F.Cu at (115.7, 107.9)
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Connections:
- C10 pad 1: VDC -> GND
- C10 pad 2: GND -> +3.3V
- C11 pad 1: +3.3V -> GND
- C11 pad 2: GND -> +3.3V
- C12 pad 1: +3.3V -> GND
- C12 pad 2: GND -> +3.3V
- C13 pad 1: VDC -> GND
- C13 pad 2: GND -> +3.3V
- C14 pad 1: +5V -> GND
- C14 pad 2: GND -> Net-(C14-Pad2)
- C15 pad 1: +5V -> GND
- C15 pad 2: GND -> XIN
- C16 pad 1: GND -> VDC
- C16 pad 2: +3.3V -> GND
- C17 pad 1: GND -> VDC
- C17 pad 2: +3.3V -> GND
- C18 pad 1: GND -> +3.3V
- C18 pad 2: +3.3V -> GND
- C19 pad 1: GND -> +3.3V
- C19 pad 2: +3.3V -> GND
- C20 pad 1: GND -> VDC
- C20 pad 2: +3.3V -> GND
- C21 pad 1: GND -> +5V
- C21 pad 2: +3.3V -> GND
- C22 pad 1: GND -> +5V
- C22 pad 2: +3.3V -> GND
- C23 pad 1: GND -> VDC
- C23 pad 2: +3.3V -> GND
- C4 pad 2: +3.3V -> +1V1
- C6 pad 2: VREG_AVDD -> +1V1
- C7 pad 2: Net-(C7-Pad2) -> +3.3V
- C8 pad 2: XIN -> +3.3V
- C9 pad 1: VDC -> GND
- C9 pad 2: GND -> +3.3V
- D10 pad 1: VBUS -> Net-(D10-K)
- D4 pad 1: GND -> +5V
- D4 pad 2: Net-(D4-A) -> VBUS
- D8 pad 1: Net-(D8-K) -> GND
- D8 pad 2: GND -> Net-(D8-A)
- D9 pad 1: Net-(D9-K) -> Net-(D10-K)
- D9 pad 2: GND -> +5V
- J10 pad 1: +3.3V -> Net-(J10-U-VCC)
- J10 pad 2: +3.3V -> /USB 1/U_D-
- J10 pad 3: +3.3V -> /USB 1/U_D+
- J10 pad 4: 3.3V_BUCK_EN -> GND
- J12 pad 1: +5V -> Net-(J12-Pin_1)
- J12 pad 2: +5V -> Net-(J12-Pin_2)
- J12 pad 3: +5V -> GND
- J12 pad 4: 5V_BUCK_EN -> GND
- J14 pad 1: VDC -> Net-(J14-Pin_1)
- J14 pad 2: VDC -> Net-(J14-Pin_2)
- J14 pad 3: VDC -> GND
- J14 pad 4: VDC -> GND
- J15 pad 1: Net-(J15-Pin_1) -> Net-(J15-U-VCC)
- J15 pad 2: Net-(J15-Pin_2) -> /USB 2/U_D-
- J15 pad 3: CC2 -> /USB 2/U_D+
- J15 pad 4: CC1 -> GND
- J16 pad A1: GND -> Net-(U21-CSP)
- J16 pad A12: GND -> Net-(U21-CSP)
- J16 pad A4: VBUS -> Net-(Q4-S)
- J16 pad A5: CC1 -> Net-(J16-CC1)
- J16 pad A6: Net-(J15-Pin_2) -> Net-(J16-DP1)
- J16 pad A7: Net-(J15-Pin_1) -> Net-(J16-DN1)
- J16 pad A9: VBUS -> Net-(Q4-S)
- J16 pad B1: GND -> Net-(U21-CSP)
- J16 pad B12: GND -> Net-(U21-CSP)
- J16 pad B4: VBUS -> Net-(Q4-S)
- J16 pad B5: CC2 -> Net-(J16-CC2)
- J16 pad B6: Net-(J15-Pin_2) -> Net-(J16-DP1)
- J16 pad B7: Net-(J15-Pin_1) -> Net-(J16-DN1)
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Routing:
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- removed copper zone on F.Cu, net +3.3V
- removed copper zone on B.Cu, net GND
- removed copper zone on F.Cu, net GND
Other:
- board outline removed
- board text removed: "0"
- board text removed: "1"
- board text removed: "1.1V>"
- board text removed: "10"
- board text removed: "11"
- board text removed: "12"
- board text removed: "13"
- board text removed: "14"
- board text removed: "15"
- board text removed: "2"
- board text removed: "3"
- board text removed: "3.3V"
- board text removed: "32"
- board text removed: "33"
- board text removed: "38"
- board text removed: "39"
- board text removed: "4"
- board text removed: "40"
- board text removed: "41"
- board text removed: "42"
- board text removed: "43"
- board text removed: "44"
- board text removed: "45"
- board text removed: "46"
- board text removed: "47"
- board text removed: "5"
- board text removed: "6"
- board text removed: "7"
- board text removed: "8"
- board text removed: "9"
- board text removed: "<USB"
- board text removed: "D+"
- board text removed: "D-"

Commit message: finished schematic yay!! now onto pcb routing :fire:
Parts:
- removed C143, C144: 50V,10uF, Capacitor_SMD:C_1206_3216Metric_Pad1.33x1.80mm_HandSolder
- removed C145, C147: 35V,180uF, Capacitor_THT:CP_Radial_D8.0mm_P5.00mm
- removed C146, C148: 35V,22uF, Capacitor_SMD:C_0805_2012Metric_Pad1.18x1.45mm_HandSolder
- removed C149, C156, C158, C160, C162, C164, C165, C172: 100nF, Capacitor_SMD:C_0201_0603Metric_Pad0.64x0.40mm_HandSolder
- removed C150, C151, C157, C159, C161, C163, C166, C167: 1uF, Capacitor_SMD:C_0402_1005Metric_Pad0.74x0.62mm_HandSolder
- removed C152, C153, C168, C169: 390pF 5% X7R, Capacitor_SMD:C_0603_1608Metric_Pad1.08x0.95mm_HandSolder
- removed C154, C170: 100pF, Capacitor_SMD:C_0201_0603Metric_Pad0.64x0.40mm_HandSolder
- removed C155, C171: 1nF, Capacitor_SMD:C_0201_0603Metric_Pad0.64x0.40mm_HandSolder
- removed D21, D22: 40V,10A, Diode_SMD:D_SMB_Handsoldering
- removed J3, J31: TYPE-C 16PLT-H10.0, easyeda2kicad:TYPE-C-SMD_USB4120-03-C
- removed J30: XDUF-0426-081_C18202150, easyeda2kicad:USB-A-TH_XDUF-0426-081
- removed J32: Conn_01x04_Pin, Connector_PinHeader_2.54mm:PinHeader_2x02_P2.54mm_Vertical
- removed J5: Conn_01x04_Pin, Connector_PinHeader_2.54mm:PinHeader_1x04_P2.54mm_Vertical
- removed L19, L20: YPRH1508-680M, easyeda2kicad:IND-SMD_L15.0-W15.0
- removed L21, L22: 6.8uH,5.2A,8A(Isat), easyeda2kicad:IND-SMD_L8.0-W8.0-1
- removed Q10, Q9: PMOS, easyeda2kicad:PDFN-8_L5.2-W5.9-P1.27-LS6.2-BL
- removed R91, R93, R97: 10k, Resistor_SMD:R_0402_1005Metric_Pad0.72x0.64mm_HandSolder
- removed R92: 249k, Resistor_SMD:R_0402_1005Metric_Pad0.72x0.64mm_HandSolder
- removed R94: 40k, Resistor_SMD:R_0603_1608Metric_Pad0.98x0.95mm_HandSolder
- removed R95: 1k, Resistor_SMD:R_0402_1005Metric_Pad0.72x0.64mm_HandSolder
- removed R96: 6.8, Resistor_SMD:R_0402_1005Metric_Pad0.72x0.64mm_HandSolder
- removed R98: 5mOhm 1% Shunt, Resistor_SMD:R_1206_3216Metric_Pad1.30x1.75mm_HandSolder
- removed U38, U39: XXL1509-5.0, easyeda2kicad:SOIC-8_L4.9-W3.9-P1.27-LS6.0-BL
- removed U40, U44: NDP23511KC, easyeda2kicad:SOP-8_L4.9-W3.9-P1.27-LS6.0-BL
- removed U41, U45: CYPD3175-24LQXQ, Package_DFN_QFN:QFN-24-1EP_4x4mm_P0.5mm_EP2.75x2.75mm
- removed U42, U43: LS0505EVD22, LS0505EVD22:LS0505EVD22_LTF
- added J35: GT-USB-7010ASV, easyeda2kicad:USB-C-SMD_G-SWITCH_GT-USB-7010ASV, F.Cu at (262.2, 144.5)
- added LED1: SK6812MINI-E_C5149201, easyeda2kicad:LED-SMD_L3.2-W2.8-LS5.9_SK6812MINI-E, F.Cu at (261.8, 128.2)
- added LED10: SK6812MINI-E_C5149201, easyeda2kicad:LED-SMD_L3.2-W2.8-LS5.9_SK6812MINI-E, F.Cu at (138.7, 145.2)
- added LED11: SK6812MINI-E_C5149201, easyeda2kicad:LED-SMD_L3.2-W2.8-LS5.9_SK6812MINI-E, F.Cu at (138.7, 149.3)
- added LED12: SK6812MINI-E_C5149201, easyeda2kicad:LED-SMD_L3.2-W2.8-LS5.9_SK6812MINI-E, F.Cu at (138.7, 153.3)
- added LED13: SK6812MINI-E_C5149201, easyeda2kicad:LED-SMD_L3.2-W2.8-LS5.9_SK6812MINI-E, F.Cu at (138.7, 157.4)
- added LED14: SK6812MINI-E_C5149201, easyeda2kicad:LED-SMD_L3.2-W2.8-LS5.9_SK6812MINI-E, F.Cu at (138.7, 161.4)
- added LED15: SK6812MINI-E_C5149201, easyeda2kicad:LED-SMD_L3.2-W2.8-LS5.9_SK6812MINI-E, F.Cu at (146.8, 137.1)
- added LED16: SK6812MINI-E_C5149201, easyeda2kicad:LED-SMD_L3.2-W2.8-LS5.9_SK6812MINI-E, F.Cu at (146.8, 141.2)
- added LED17: SK6812MINI-E_C5149201, easyeda2kicad:LED-SMD_L3.2-W2.8-LS5.9_SK6812MINI-E, F.Cu at (146.8, 145.2)
- added LED18: SK6812MINI-E_C5149201, easyeda2kicad:LED-SMD_L3.2-W2.8-LS5.9_SK6812MINI-E, F.Cu at (146.8, 149.3)
- added LED19: SK6812MINI-E_C5149201, easyeda2kicad:LED-SMD_L3.2-W2.8-LS5.9_SK6812MINI-E, F.Cu at (146.8, 153.3)
- added LED2: SK6812MINI-E_C5149201, easyeda2kicad:LED-SMD_L3.2-W2.8-LS5.9_SK6812MINI-E, F.Cu at (130.6, 141.2)
- added LED20: SK6812MINI-E_C5149201, easyeda2kicad:LED-SMD_L3.2-W2.8-LS5.9_SK6812MINI-E, F.Cu at (146.8, 157.4)
- added LED3: SK6812MINI-E_C5149201, easyeda2kicad:LED-SMD_L3.2-W2.8-LS5.9_SK6812MINI-E, F.Cu at (130.6, 145.2)
- added LED4: SK6812MINI-E_C5149201, easyeda2kicad:LED-SMD_L3.2-W2.8-LS5.9_SK6812MINI-E, F.Cu at (130.6, 149.3)
- added LED5: SK6812MINI-E_C5149201, easyeda2kicad:LED-SMD_L3.2-W2.8-LS5.9_SK6812MINI-E, F.Cu at (130.6, 153.3)
- added LED6: SK6812MINI-E_C5149201, easyeda2kicad:LED-SMD_L3.2-W2.8-LS5.9_SK6812MINI-E, F.Cu at (130.6, 157.4)
- added LED7: SK6812MINI-E_C5149201, easyeda2kicad:LED-SMD_L3.2-W2.8-LS5.9_SK6812MINI-E, F.Cu at (130.6, 161.4)
- added LED8: SK6812MINI-E_C5149201, easyeda2kicad:LED-SMD_L3.2-W2.8-LS5.9_SK6812MINI-E, F.Cu at (138.7, 137.1)
- added LED9: SK6812MINI-E_C5149201, easyeda2kicad:LED-SMD_L3.2-W2.8-LS5.9_SK6812MINI-E, F.Cu at (138.7, 141.2)
- added R107: 470, Resistor_SMD:R_0402_1005Metric_Pad0.72x0.64mm_HandSolder, F.Cu at (258.2, 127.2)
- added R108: 10k, Resistor_SMD:R_0402_1005Metric_Pad0.72x0.64mm_HandSolder, F.Cu at (257.6, 129.2)
- added TP1: TestPoint, TestPoint:TestPoint_Pad_D2.5mm, F.Cu at (153.2, 137.4)
- C1, C16, C18, C2, L1: moved to B.Cu
- J20: value XDUF-0426-081_C18202150 -> GT-USB-7010ASV; footprint easyeda2kicad:USB-A-TH_XDUF-0426-081 -> easyeda2kicad:USB-C-SMD_G-SWITCH_GT-USB-7010ASV
- J21, J26: value TYPE-C 16PLT-H10.0 -> GT-USB-7010ASV; footprint easyeda2kicad:TYPE-C-SMD_USB4120-03-C -> easyeda2kicad:USB-C-SMD_G-SWITCH_GT-USB-7010ASV
- J22, J24: value Conn_01x04_Pin -> TYPE-C 16PLT-H10.0; footprint Connector_PinHeader_2.54mm:PinHeader_2x02_P2.54mm_Vertical -> easyeda2kicad:TYPE-C-SMD_USB4120-03-C
- J23: value TYPE-C 16PLT-H10.0 -> Conn_01x04_Pin; footprint easyeda2kicad:TYPE-C-SMD_USB4120-03-C -> Connector_PinHeader_2.54mm:PinHeader_2x02_P2.54mm_Vertical
- J25: value XDUF-0426-081_C18202150 -> Conn_01x04_Pin; footprint easyeda2kicad:USB-A-TH_XDUF-0426-081 -> Connector_PinHeader_2.54mm:PinHeader_2x02_P2.54mm_Vertical
- J27: value Conn_01x04_Pin -> GT-USB-7010ASV; footprint Connector_PinHeader_2.54mm:PinHeader_2x02_P2.54mm_Vertical -> easyeda2kicad:USB-C-SMD_G-SWITCH_GT-USB-7010ASV
- JP1: value SolderJumper_2_Bridged -> SolderJumper_2_Open; footprint Jumper:SolderJumper-2_P1.3mm_Bridged_Pad1.0x1.5mm -> Jumper:SolderJumper-2_P1.3mm_Open_RoundedPad1.0x1.5mm
- R57, R82, R89: value 5mOhm 1% Shunt -> 10k; footprint Resistor_SMD:R_1206_3216Metric_Pad1.30x1.75mm_HandSolder -> Resistor_SMD:R_0402_1005Metric_Pad0.72x0.64mm_HandSolder
- R58, R60, R76: value 249k -> 10k
- R59: value 10k -> 249k
- R61, R81: value 10k -> 5mOhm 1% Shunt; footprint Resistor_SMD:R_0402_1005Metric_Pad0.72x0.64mm_HandSolder -> Resistor_SMD:R_1206_3216Metric_Pad1.30x1.75mm_HandSolder
- R62, R69, R78, R85: value 40k -> 10k; footprint Resistor_SMD:R_0603_1608Metric_Pad0.98x0.95mm_HandSolder -> Resistor_SMD:R_0402_1005Metric_Pad0.72x0.64mm_HandSolder
- R63: value 1k -> 10k
- R64: value 6.8 -> 249k
- R66, R73: value 5mOhm 1% Shunt -> 40k; footprint Resistor_SMD:R_1206_3216Metric_Pad1.30x1.75mm_HandSolder -> Resistor_SMD:R_0603_1608Metric_Pad0.98x0.95mm_HandSolder
- R67: value 100k -> 1k
- R68: value 100k -> 6.8
- R70: value 1k -> 5mOhm 1% Shunt; footprint Resistor_SMD:R_0402_1005Metric_Pad0.72x0.64mm_HandSolder -> Resistor_SMD:R_1206_3216Metric_Pad1.30x1.75mm_HandSolder
- R71: value 6.8 -> 100k
- R72: value 10k -> 100k
- R74: value 249k -> 1k
- R75, R88: value 10k -> 6.8
- R79: value 1k -> 249k
- R80: value 6.8 -> 10k
- R83: value 100k -> 10k
- R84: value 100k -> 249k
- R86: value 1k -> 40k; footprint Resistor_SMD:R_0402_1005Metric_Pad0.72x0.64mm_HandSolder -> Resistor_SMD:R_0603_1608Metric_Pad0.98x0.95mm_HandSolder
- R87: value 6.8 -> 1k
- R90: value 249k -> 5mOhm 1% Shunt; footprint Resistor_SMD:R_0402_1005Metric_Pad0.72x0.64mm_HandSolder -> Resistor_SMD:R_1206_3216Metric_Pad1.30x1.75mm_HandSolder
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Connections:
- C1 pad 2: Net-(C1-Pad2) -> GND
- C101 pad 2: Net-(J20-D-VCC) -> Net-(U27-OUT)
- C102 pad 2: Net-(J20-D-VCC) -> Net-(U27-OUT)
- C108 pad 1: Net-(J21-CC2) -> Net-(J22-CC2)
- C109 pad 1: Net-(J21-CC1) -> Net-(J22-CC1)
- C122 pad 1: Net-(J23-CC2) -> Net-(J24-CC2)
- C123 pad 1: Net-(J23-CC1) -> Net-(J24-CC1)
- C127 pad 2: Net-(J25-U-VCC) -> Net-(U34-OUT)
- C128 pad 2: Net-(J25-U-VCC) -> Net-(U34-OUT)
- C131 pad 2: Net-(J25-D-VCC) -> Net-(U35-OUT)
- C132 pad 2: Net-(J25-D-VCC) -> Net-(U35-OUT)
- C138 pad 1: Net-(J26-CC2) -> Net-(J28-CC2)
- C139 pad 1: Net-(J26-CC1) -> Net-(J28-CC1)
- C2 pad 1: Net-(C1-Pad2) -> VDC
- C97 pad 2: Net-(J20-U-VCC) -> Net-(U26-OUT)
- C98 pad 2: Net-(J20-U-VCC) -> Net-(U26-OUT)
- J20 pad 1: Net-(J20-U-VCC) -> GND
- J20 pad 2: /USB 3/U_D- -> GND
- J20 pad 3: /USB 3/U_D+ -> GND
- J21 pad A6: Net-(J21-DP1) -> /USB 3/D_D+
- J21 pad A7: Net-(J21-DN1) -> /USB 3/D_D-
- J21 pad B6: Net-(J21-DP1) -> /USB 3/D_D+
- J21 pad B7: Net-(J21-DN1) -> /USB 3/D_D-
- J25 pad 1: Net-(J25-U-VCC) -> Net-(J25-Pin_1)
- J25 pad 2: /USB 4/U_D- -> Net-(J25-Pin_2)
- J25 pad 3: /USB 4/U_D+ -> GND
- J26 pad A6: Net-(J26-DP1) -> /USB 4/U_D+
- J26 pad A7: Net-(J26-DN1) -> /USB 4/U_D-
- J26 pad B6: Net-(J26-DP1) -> /USB 4/U_D+
- J26 pad B7: Net-(J26-DN1) -> /USB 4/U_D-
- J27 pad 1: Net-(J27-Pin_1) -> GND
- J27 pad 2: Net-(J27-Pin_2) -> GND
- J28 pad A1: Net-(U41-CSP) -> Net-(U37-CSP)
- J28 pad A12: Net-(U41-CSP) -> Net-(U37-CSP)
- J28 pad A4: Net-(Q9-S) -> Net-(Q8-S)
- J28 pad A9: Net-(Q9-S) -> Net-(Q8-S)
- J28 pad B1: Net-(U41-CSP) -> Net-(U37-CSP)
- J28 pad B12: Net-(U41-CSP) -> Net-(U37-CSP)
- J28 pad B4: Net-(Q9-S) -> Net-(Q8-S)
- J28 pad B9: Net-(Q9-S) -> Net-(Q8-S)
- L10 pad 1: Net-(U20-SW) -> Net-(L10-Pad1)
- L13 pad 1: Net-(U24-SW) -> Net-(L13-Pad1)
- L14 pad 1: Net-(U28-SW) -> Net-(L14-Pad1)
- L17 pad 1: Net-(U32-SW) -> Net-(L17-Pad1)
- L18 pad 1: Net-(U36-SW) -> Net-(L18-Pad1)
- L5 pad 1: Net-(U8-SW) -> Net-(L5-Pad1)
- L6 pad 1: Net-(U12-SW) -> Net-(L6-Pad1)
- L9 pad 1: Net-(U16-SW) -> Net-(L9-Pad1)
- R23 pad 1: Net-(U8-SW) -> Net-(L5-Pad1)
- R32 pad 1: Net-(U12-SW) -> Net-(L6-Pad1)
- R39 pad 1: Net-(U16-SW) -> Net-(L9-Pad1)
- R48 pad 1: Net-(U20-SW) -> Net-(L10-Pad1)
- R55 pad 1: Net-(U24-SW) -> Net-(L13-Pad1)
- R57 pad 1: Net-(U25-CSP) -> Net-(U26-OUT)
- R57 pad 2: GND -> Net-(J20-CC1)
- R58 pad 1: Net-(U26-ILIM) -> Net-(U26-OUT)
- R58 pad 2: GND -> Net-(J20-CC2)
- R59 pad 1: /USB 3/U_EN -> Net-(U26-ILIM)
- R60 pad 1: Net-(U27-ILIM) -> /USB 3/U_EN
- R61 pad 1: /USB 3/D_EN -> Net-(U25-CSP)
- R62 pad 1: Net-(Q6-D) -> Net-(U27-OUT)
- R62 pad 2: Net-(U28-VFB) -> Net-(J21-CC1)
- R63 pad 1: Net-(Q6-D) -> Net-(U27-OUT)
- R63 pad 2: Net-(U29-FB) -> Net-(J21-CC2)
- R64 pad 1: Net-(U28-SW) -> Net-(U27-ILIM)
- R64 pad 2: Net-(C111-Pad1) -> GND
- R65 pad 1: Net-(U28-VFB) -> /USB 3/D_EN
- R66 pad 1: Net-(U29-CSP) -> Net-(Q6-D)
- R66 pad 2: GND -> Net-(U28-VFB)
- R67 pad 1: GND -> Net-(Q6-D)
- R67 pad 2: /USB 4/U_BUCK_EN -> Net-(U29-FB)
- R68 pad 1: GND -> Net-(L14-Pad1)
- R68 pad 2: /USB 4/D_BUCK_EN -> Net-(C111-Pad1)
- R69 pad 1: Net-(Q7-D) -> Net-(U28-VFB)
- R69 pad 2: Net-(U32-VFB) -> GND
- R70 pad 1: Net-(Q7-D) -> Net-(U29-CSP)
- R70 pad 2: Net-(U33-FB) -> GND
- R71 pad 1: Net-(U32-SW) -> GND
- R71 pad 2: Net-(C125-Pad1) -> /USB 4/U_BUCK_EN
- R72 pad 1: Net-(U32-VFB) -> GND
- R72 pad 2: GND -> /USB 4/D_BUCK_EN
- R73 pad 1: Net-(U33-CSP) -> Net-(Q7-D)
- R73 pad 2: GND -> Net-(U32-VFB)
- R74 pad 1: Net-(U34-ILIM) -> Net-(Q7-D)
- R74 pad 2: GND -> Net-(U33-FB)
- R75 pad 1: /USB 4/U_EN -> Net-(L17-Pad1)
- R75 pad 2: GND -> Net-(C125-Pad1)
- R76 pad 1: Net-(U35-ILIM) -> Net-(U32-VFB)
- R77 pad 1: /USB 4/D_EN -> Net-(U34-OUT)
- R77 pad 2: GND -> Net-(J26-CC1)
- R78 pad 1: Net-(Q8-D) -> Net-(U34-OUT)
- R78 pad 2: Net-(U36-VFB) -> Net-(J26-CC2)
- R79 pad 1: Net-(Q8-D) -> Net-(U34-ILIM)
- R79 pad 2: Net-(U37-FB) -> GND
- R80 pad 1: Net-(U36-SW) -> /USB 4/U_EN
- R80 pad 2: Net-(C141-Pad1) -> GND
- R81 pad 1: Net-(U36-VFB) -> Net-(U33-CSP)
- R82 pad 1: Net-(U37-CSP) -> Net-(U35-OUT)
- R82 pad 2: GND -> Net-(J27-CC1)
- R83 pad 1: GND -> Net-(U35-OUT)
- R83 pad 2: /USB 5/U_BUCK_EN -> Net-(J27-CC2)
- R84 pad 1: GND -> Net-(U35-ILIM)
- R84 pad 2: /USB 5/D_BUCK_EN -> GND
- R85 pad 1: Net-(Q9-D) -> /USB 4/D_EN
- R85 pad 2: Net-(U40-VFB) -> GND
- R86 pad 1: Net-(Q9-D) -> Net-(Q8-D)
- R86 pad 2: Net-(U41-FB) -> Net-(U36-VFB)
- R87 pad 1: Net-(U40-SW) -> Net-(Q8-D)
- R87 pad 2: Net-(C155-Pad1) -> Net-(U37-FB)
- R88 pad 1: Net-(U40-VFB) -> Net-(L18-Pad1)
- R88 pad 2: GND -> Net-(C141-Pad1)
- R89 pad 1: Net-(U41-CSP) -> Net-(U36-VFB)
- R90 pad 1: Net-(U42-ILIM) -> Net-(U37-CSP)
- SW1 pad 4: Net-(U3-GPIO18) -> Net-(U3-GPIO19)
- SW2 pad 1: Net-(U3-GPIO19) -> Net-(U3-GPIO18)
- U12 pad 5: (no net) -> Net-(L6-Pad1)
- U12 pad 6: (no net) -> Net-(L6-Pad1)
- U16 pad 5: (no net) -> Net-(L9-Pad1)
- U16 pad 6: (no net) -> Net-(L9-Pad1)
- U20 pad 5: (no net) -> Net-(L10-Pad1)
- U20 pad 6: (no net) -> Net-(L10-Pad1)
- U24 pad 5: (no net) -> Net-(L13-Pad1)
- U24 pad 6: (no net) -> Net-(L13-Pad1)
- U26 pad 8: Net-(J20-U-VCC) -> Net-(U26-OUT)
- U27 pad 8: Net-(J20-D-VCC) -> Net-(U27-OUT)
- U28 pad 5: (no net) -> Net-(L14-Pad1)
- U28 pad 6: (no net) -> Net-(L14-Pad1)
- U29 pad 14: Net-(J21-CC2) -> Net-(J22-CC2)
- U29 pad 15: Net-(J21-CC1) -> Net-(J22-CC1)
- U29 pad 16: Net-(J21-DN1) -> Net-(J22-DN1)
- U29 pad 17: Net-(J21-DP1) -> Net-(J22-DP1)
- U29 pad 7: Net-(J22-Pin_1) -> Net-(J23-Pin_1)
- U29 pad 8: Net-(J22-Pin_2) -> Net-(J23-Pin_2)
- U3 pad 18: GPIO15 -> Net-(U3-GPIO15)
- U3 pad 27: GPIO16 -> SDA
- U3 pad 28: GPIO17 -> SCL
- U32 pad 5: (no net) -> Net-(L17-Pad1)
- U32 pad 6: (no net) -> Net-(L17-Pad1)
- U33 pad 14: Net-(J23-CC2) -> Net-(J24-CC2)
- U33 pad 15: Net-(J23-CC1) -> Net-(J24-CC1)
- U33 pad 16: Net-(J23-DN1) -> Net-(J24-DN1)
- U33 pad 17: Net-(J23-DP1) -> Net-(J24-DP1)
- U33 pad 7: Net-(J24-Pin_1) -> Net-(J25-Pin_1)
- U33 pad 8: Net-(J24-Pin_2) -> Net-(J25-Pin_2)
- U34 pad 8: Net-(J25-U-VCC) -> Net-(U34-OUT)
- U35 pad 8: Net-(J25-D-VCC) -> Net-(U35-OUT)
- U36 pad 5: (no net) -> Net-(L18-Pad1)
- U36 pad 6: (no net) -> Net-(L18-Pad1)
- U37 pad 14: Net-(J26-CC2) -> Net-(J28-CC2)
- U37 pad 15: Net-(J26-CC1) -> Net-(J28-CC1)
- U37 pad 16: Net-(J26-DN1) -> Net-(J28-DN1)
- U37 pad 17: Net-(J26-DP1) -> Net-(J28-DP1)
- U37 pad 7: Net-(J27-Pin_1) -> Net-(J29-Pin_1)
- U37 pad 8: Net-(J27-Pin_2) -> Net-(J29-Pin_2)
- U8 pad 5: (no net) -> Net-(L5-Pad1)
- U8 pad 6: (no net) -> Net-(L5-Pad1)
- U9 pad 12: unconnected-(U9-P2.2-Pad12) -> SDA
- U9 pad 13: unconnected-(U9-P2.3-Pad13) -> SCL
Routing:
- net GND: track 0.00 -> 32.3 mm
- net VBUS: track 0.00 -> 20.1 mm
- net Net-(D10-K): track 0.00 -> 20.1 mm
- net Net-(U3-GPIO19): track 0.00 -> 19.2 mm, vias 0 -> 2
- net +3.3V: track 0.00 -> 13.5 mm
- net 3.3V_BUCK_EN: track 0.00 -> 10.9 mm, vias 0 -> 1
- net Net-(D11-K): track 0.00 -> 7.10 mm
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- added copper zone on B.Cu, net +3.3V
- added copper zone on F.Cu, net +3.3V
- added copper zone on In1.Cu, net +3.3V
- added copper zone on F.Cu, net GND
- added copper zone on In2.Cu, net GND
- added copper zone on B.Cu, net Net-(D11-K)
- added copper zone on F.Cu, net Net-(D11-K)
- added copper zone on In1.Cu, net Net-(D11-K)
- added copper zone on In1.Cu, net VDC
Other:
- board outline added: 100 x 100 mm
- copper layers 2 -> 4
