File: usb-charging-hub.kicad_pcb (KiCad board)
At the start: 4 copper layers, 100 x 100 mm, 369 parts, among them J1 Conn_01x01_Pin, J10 XDUF-0426-081_C18202150, J11 TYPE-C 16PLT-H10.0, J12 Conn_01x04_Pin, J13 TYPE-C 16PLT-H10.0, J14 Conn_01x04_Pin, J15 XDUF-0426-081_C18202150, J16 TYPE-C 16PLT-H10.0, J17 Conn_01x04_Pin, J18 TYPE-C 16PLT-H10.0, J19 Conn_01x04_Pin, J2 Conn_01x01_Pin, J20 GT-USB-7010ASV, J21 GT-USB-7010ASV, J22 TYPE-C 16PLT-H10.0, J23 Conn_01x04_Pin, J24 TYPE-C 16PLT-H10.0, J25 Conn_01x04_Pin, J26 GT-USB-7010ASV, J27 GT-USB-7010ASV, J28 TYPE-C 16PLT-H10.0, J29 Conn_01x04_Pin, J35 GT-USB-7010ASV, J4 Conn_01x04_Pin, J6 Conn_01x04_Pin, J7 Conn_01x04_Pin, J8 TYPE-C 16PLT-H10.0, J9 Conn_01x04_Pin, Q1 PMOS, Q2 PMOS, Q3 PMOS, Q4 PMOS, Q5 PMOS, Q6 PMOS, Q7 PMOS, Q8 PMOS, SW1 TS24CA, SW2 Latching, SW3 TS24CA, SW4 TS24CA, U1 W25Q32JVSS, U10 LS0505EVD22, U11 LS0505EVD22, U12 NDP23511KC, U13 CYPD3175-24LQXQ, U14 XXL1509-5.0, U15 XXL1509-5.0, U16 NDP23511KC, U17 CYPD3175-24LQXQ, U18 LS0505EVD22, U19 LS0505EVD22, U2 ABM8-272-T3_C20625731, U20 NDP23511KC, U21 CYPD3175-24LQXQ, U22 XXL1509-5.0, U23 XXL1509-5.0, U24 NDP23511KC, U25 CYPD3175-24LQXQ, U26 LS0505EVD22, U27 LS0505EVD22, U28 NDP23511KC, U29 CYPD3175-24LQXQ, U3 RP2040, U30 XXL1509-5.0, U31 XXL1509-5.0, U32 NDP23511KC, U33 CYPD3175-24LQXQ, U34 LS0505EVD22, U35 LS0505EVD22, U36 NDP23511KC, U37 CYPD3175-24LQXQ, U4 LM2596S-3.3, U5 XXL1509-5.0, U6 XXL1509-5.0, U7 XXL1509-5.0, U8 NDP23511KC, U9 CYPD3175-24LQXQ

Commit message: made huge progress today, finished wiring up the rp2040, finished one usb a and usb c layout :fire::fire::fire:
Parts:
- added SW10: Latching, easyeda2kicad:SW-TH_6P-L8.0-W8.0-P2.50, F.Cu at (71.4, 43.6)
- added SW11: Latching, easyeda2kicad:SW-TH_6P-L8.0-W8.0-P2.50, F.Cu at (71.4, 55.6)
- added SW12: Latching, easyeda2kicad:SW-TH_6P-L8.0-W8.0-P2.50, F.Cu at (71.4, 67.6)
- added SW13: Latching, easyeda2kicad:SW-TH_6P-L8.0-W8.0-P2.50, F.Cu at (29.4, 31.6)
- added SW14: Latching, easyeda2kicad:SW-TH_6P-L8.0-W8.0-P2.50, F.Cu at (29.4, 43.6)
- added SW15: Latching, easyeda2kicad:SW-TH_6P-L8.0-W8.0-P2.50, F.Cu at (29.4, 55.6)
- added SW16: Latching, easyeda2kicad:SW-TH_6P-L8.0-W8.0-P2.50, F.Cu at (29.4, 67.6)
- added SW17: Latching, easyeda2kicad:SW-TH_6P-L8.0-W8.0-P2.50, F.Cu at (57.4, 31.6)
- added SW18: Latching, easyeda2kicad:SW-TH_6P-L8.0-W8.0-P2.50, F.Cu at (57.4, 43.6)
- added SW19: Latching, easyeda2kicad:SW-TH_6P-L8.0-W8.0-P2.50, F.Cu at (57.4, 55.6)
- added SW20: Latching, easyeda2kicad:SW-TH_6P-L8.0-W8.0-P2.50, F.Cu at (57.4, 67.6)
- added SW5: Latching, easyeda2kicad:SW-TH_6P-L8.0-W8.0-P2.50, F.Cu at (199.4, 74.6)
- added SW6: Latching, easyeda2kicad:SW-TH_6P-L8.0-W8.0-P2.50, F.Cu at (179.8, 74.6)
- added SW7: Latching, easyeda2kicad:SW-TH_6P-L8.0-W8.0-P2.50, F.Cu at (197.9, 129.7)
- added SW8: Latching, easyeda2kicad:SW-TH_6P-L8.0-W8.0-P2.50, F.Cu at (197.9, 141.7)
- added SW9: Latching, easyeda2kicad:SW-TH_6P-L8.0-W8.0-P2.50, F.Cu at (71.4, 31.6)
- C25, C27, J10, L3, L4, L5, L6: moved to B.Cu
- LED1, LED10, LED11, LED12, LED13, LED14, LED15, LED16, LED17, LED18, LED19, LED2, LED20, LED3, LED4, LED5, LED6, LED7, LED8, LED9: footprint easyeda2kicad:LED-SMD_L3.2-W2.8-LS5.9_SK6812MINI-E -> Keebio-Parts:SK6812-MINI-E
- U13, U17, U21, U25, U29, U33, U37, U9: footprint Package_DFN_QFN:QFN-24-1EP_4x4mm_P0.5mm_EP2.75x2.75mm -> Package_DFN_QFN:QFN-24-1EP_4x4mm_P0.5mm_EP2.7x2.7mm_ThermalVias
- moved L6 173.5 mm to (202.7, 119.7)
- moved L5 172.5 mm to (208.8, 94.6), turned to -90 degrees
- moved C45 171.8 mm to (218.8, 120.1)
- moved C48 171.8 mm to (219.9, 141.5)
- moved C50 171.8 mm to (218.8, 121.8)
- moved C51 171.8 mm to (218.8, 123.6)
- moved C52 171.8 mm to (218.8, 125.3)
- moved J12 171.8 mm to (212.9, 136.4)
- moved Q2 171.8 mm to (208.6, 123.1)
- moved R30 171.8 mm to (219.9, 149.0)
- moved R33 171.8 mm to (205.6, 153.6)
- moved U12 171.8 mm to (227.1, 131.1)
- moved U13 171.8 mm to (213.7, 150.7)
- moved C46 171.8 mm to (223.7, 148.0)
- moved C47 171.8 mm to (223.7, 150.0)
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Connections:
- net Net-(J35-DN1) renamed /rp2040/USB_R_D-
- net Net-(J35-DP1) renamed /rp2040/USB_R_D+
- net Net-(U3-USB_DM) renamed /rp2040/USB_D-
- net Net-(U3-USB_DP) renamed /rp2040/USB_D+
- U12 pad 3: unconnected-(U12-EN-Pad3) -> /USB 1/2_BUCK_EN
- U12 pad 4: unconnected-(U12-VIN-Pad4) -> VDC
- U13 pad 1: /USB 1/D_EN -> /USB 1/2_BUCK_EN
- U13 pad 10: unconnected-(U13-P2.1-Pad10) -> Net-(U13-P2.1)
- U13 pad 12: unconnected-(U13-P2.2-Pad12) -> SDA
- U13 pad 13: unconnected-(U13-P2.3-Pad13) -> SCL
- U13 pad 9: unconnected-(U13-P2.0/AXRES-Pad9) -> Net-(U13-P2.0/AXRES)
- U16 pad 3: unconnected-(U16-EN-Pad3) -> /USB 2/1_BUCK_EN
- U16 pad 4: unconnected-(U16-VIN-Pad4) -> VDC
- U17 pad 1: /USB 2/U_EN -> /USB 2/1_BUCK_EN
- U17 pad 10: unconnected-(U17-P2.1-Pad10) -> Net-(U17-P2.1)
- U17 pad 12: unconnected-(U17-P2.2-Pad12) -> SDA
- U17 pad 13: unconnected-(U17-P2.3-Pad13) -> SCL
- U17 pad 9: unconnected-(U17-P2.0/AXRES-Pad9) -> Net-(U17-P2.0/AXRES)
- U20 pad 3: unconnected-(U20-EN-Pad3) -> /USB 2/2_BUCK_EN
- U20 pad 4: unconnected-(U20-VIN-Pad4) -> VDC
- U21 pad 1: /USB 2/D_EN -> /USB 2/2_BUCK_EN
- U21 pad 10: unconnected-(U21-P2.1-Pad10) -> Net-(U21-P2.1)
- U21 pad 12: unconnected-(U21-P2.2-Pad12) -> SDA
- U21 pad 13: unconnected-(U21-P2.3-Pad13) -> SCL
- U21 pad 9: unconnected-(U21-P2.0/AXRES-Pad9) -> Net-(U21-P2.0/AXRES)
- U24 pad 3: unconnected-(U24-EN-Pad3) -> /USB 3/1_BUCK_EN
- U24 pad 4: unconnected-(U24-VIN-Pad4) -> VDC
- U25 pad 1: /USB 3/U_EN -> /USB 3/1_BUCK_EN
- U25 pad 10: unconnected-(U25-P2.1-Pad10) -> Net-(U25-P2.1)
- U25 pad 12: unconnected-(U25-P2.2-Pad12) -> SDA
- U25 pad 13: unconnected-(U25-P2.3-Pad13) -> SCL
- U25 pad 9: unconnected-(U25-P2.0/AXRES-Pad9) -> Net-(U25-P2.0/AXRES)
- U28 pad 3: unconnected-(U28-EN-Pad3) -> /USB 3/2_BUCK_EN
- U28 pad 4: unconnected-(U28-VIN-Pad4) -> VDC
- U29 pad 1: /USB 3/D_EN -> /USB 3/2_BUCK_EN
- U29 pad 10: unconnected-(U29-P2.1-Pad10) -> Net-(U29-P2.1)
- U29 pad 12: unconnected-(U29-P2.2-Pad12) -> SDA
- U29 pad 13: unconnected-(U29-P2.3-Pad13) -> SCL
- U29 pad 9: unconnected-(U29-P2.0/AXRES-Pad9) -> Net-(U29-P2.0/AXRES)
- U32 pad 3: unconnected-(U32-EN-Pad3) -> /USB 4/1_BUCK_EN
- U32 pad 4: unconnected-(U32-VIN-Pad4) -> VDC
- U33 pad 1: /USB 4/U_EN -> /USB 4/1_BUCK_EN
- U33 pad 10: unconnected-(U33-P2.1-Pad10) -> Net-(U33-P2.1)
- U33 pad 12: unconnected-(U33-P2.2-Pad12) -> SDA
- U33 pad 13: unconnected-(U33-P2.3-Pad13) -> SCL
- U33 pad 9: unconnected-(U33-P2.0/AXRES-Pad9) -> Net-(U33-P2.0/AXRES)
- U36 pad 3: unconnected-(U36-EN-Pad3) -> /USB 4/2_BUCK_EN
- U36 pad 4: unconnected-(U36-VIN-Pad4) -> VDC
- U37 pad 1: /USB 4/D_EN -> /USB 4/2_BUCK_EN
- U37 pad 10: unconnected-(U37-P2.1-Pad10) -> Net-(U37-P2.1)
- U37 pad 12: unconnected-(U37-P2.2-Pad12) -> SDA
- U37 pad 13: unconnected-(U37-P2.3-Pad13) -> SCL
- U37 pad 9: unconnected-(U37-P2.0/AXRES-Pad9) -> Net-(U37-P2.0/AXRES)
- U8 pad 3: unconnected-(U8-EN-Pad3) -> /USB 1/1_BUCK_EN
- U8 pad 4: unconnected-(U8-VIN-Pad4) -> VDC
- U9 pad 1: /USB 1/U_EN -> /USB 1/1_BUCK_EN
- U9 pad 10: unconnected-(U9-P2.1-Pad10) -> Net-(U9-P2.1)
- U9 pad 9: unconnected-(U9-P2.0/AXRES-Pad9) -> Net-(U9-P2.0/AXRES)
Routing:
- net RUN: track 0.00 -> 27.4 mm, vias 0 -> 2
- net QSPI_SD0: track 0.00 -> 19.6 mm, vias 0 -> 2
- net QSPI_SS: track 0.00 -> 19.6 mm
- net /rp2040/USB_D+: track 0.00 -> 18.3 mm, vias 0 -> 2
- net /rp2040/USB_D-: track 0.00 -> 18.3 mm, vias 0 -> 2
- net QSPI_SCLK: track 0.00 -> 16.9 mm, vias 0 -> 2
- net +3.3V: track 13.5 -> 28.8 mm, vias 0 -> 7
- net QSPI_SD3: track 0.00 -> 13.1 mm, vias 0 -> 2
- net QSPI_SD1: track 0.00 -> 12.0 mm
- net QSPI_SD2: track 0.00 -> 11.2 mm
- net XIN: track 3.14 -> 8.88 mm
- net +1V1: track 5.22 -> 9.13 mm
- net Net-(D8-A): track 0.00 -> 2.63 mm
- net Net-(D7-A): track 0.00 -> 2.11 mm
- net Net-(D6-A): track 0.00 -> 1.86 mm
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- added copper zone on B.Cu, net +5V
- added copper zone on F.Cu, net +5V
- added copper zone on B.Cu, net GND
- added copper zone on F.Cu, net Net-(D10-K)
Other:
- board text added: "{ "ViaStitching": "0.2", "stitch_zone_0": { "HSpacing": "1", "VSpacing": "1", "HOffset": "0", "VOffset": "0", "Clearance": "0", "Randomize": false } }"
- board text added: "{ "ViaStitching": "0.2", "stitch_zone_0": { "HSpacing": "1", "VSpacing": "1", "HOffset": "0", "VOffset": "0", "Clearance": "0.5", "Randomize": false } }"

Commit message: holyyy i actually finished all of the bare pcb adding lots of art soon:tm:
Signed-off-by: Toby Cm <toby@vsus.app>
Parts:
- removed C100, C102, C104, C105, C112, C119, C126, C128, C130, C132, C134, C135, C142, C89, C96, C98: 100nF, Capacitor_SMD:C_0201_0603Metric_Pad0.64x0.40mm_HandSolder
- removed C101, C103, C106, C107, C120, C121, C127, C129, C131, C133, C136, C137, C90, C91, C97, C99: 1uF, Capacitor_SMD:C_0402_1005Metric_Pad0.74x0.62mm_HandSolder
- removed C108, C109, C122, C123, C138, C139, C92, C93: 390pF 5% X7R, Capacitor_SMD:C_0603_1608Metric_Pad1.08x0.95mm_HandSolder
- removed C110, C124, C140, C94: 100pF, Capacitor_SMD:C_0201_0603Metric_Pad0.64x0.40mm_HandSolder
- removed C111, C125, C141, C95: 1nF, Capacitor_SMD:C_0201_0603Metric_Pad0.64x0.40mm_HandSolder
- removed C113, C114, C83, C84: 50V,10uF, Capacitor_SMD:C_1206_3216Metric_Pad1.33x1.80mm_HandSolder
- removed C115, C117, C85, C87: 35V,180uF, Capacitor_THT:CP_Radial_D8.0mm_P5.00mm
- removed C116, C118, C86, C88: 35V,22uF, Capacitor_SMD:C_0805_2012Metric_Pad1.18x1.45mm_HandSolder
- removed D17, D18, D19, D20: 40V,10A, Diode_SMD:D_SMB_Handsoldering
- removed J18, J22, J24, J28: TYPE-C 16PLT-H10.0, easyeda2kicad:TYPE-C-SMD_USB4120-03-C
- removed J19, J23, J25, J29: Conn_01x04_Pin, Connector_PinHeader_2.54mm:PinHeader_2x02_P2.54mm_Vertical
- removed J20, J21, J26, J27: GT-USB-7010ASV, easyeda2kicad:USB-C-SMD_G-SWITCH_GT-USB-7010ASV
- removed L11, L12, L15, L16: YPRH1508-680M, easyeda2kicad:IND-SMD_L15.0-W15.0
- removed L13, L14, L17, L18: 6.8uH,5.2A,8A(Isat), easyeda2kicad:IND-SMD_L8.0-W8.0-1
- removed LED10, LED11, LED12, LED13, LED14, LED15, LED16, LED17, LED18, LED19, LED20, LED6, LED7, LED8, LED9: SK6812MINI-E_C5149201, Keebio-Parts:SK6812-MINI-E
- removed Q5, Q6, Q7, Q8: PMOS, easyeda2kicad:PDFN-8_L5.2-W5.9-P1.27-LS6.2-BL
- removed R51, R52, R71, R72: 100k, Resistor_SMD:R_0402_1005Metric_Pad0.72x0.64mm_HandSolder
- removed R53, R66, R73, R86: 40k, Resistor_SMD:R_0603_1608Metric_Pad0.98x0.95mm_HandSolder
- removed R54, R67, R74, R87: 1k, Resistor_SMD:R_0402_1005Metric_Pad0.72x0.64mm_HandSolder
- removed R55, R68, R75, R88: 6.8, Resistor_SMD:R_0402_1005Metric_Pad0.72x0.64mm_HandSolder
- removed R56, R57, R58, R60, R62, R63, R65, R69, R76, R77, R78, R80, R82, R83, R85, R89: 10k, Resistor_SMD:R_0402_1005Metric_Pad0.72x0.64mm_HandSolder
- removed R59, R64, R79, R84: 249k, Resistor_SMD:R_0402_1005Metric_Pad0.72x0.64mm_HandSolder
- removed R61, R70, R81, R90: 5mOhm 1% Shunt, Resistor_SMD:R_1206_3216Metric_Pad1.30x1.75mm_HandSolder
- removed SW10, SW11, SW12, SW13, SW14, SW15, SW16, SW17, SW18, SW19, SW20, SW5, SW6, SW7, SW8, SW9: Latching, easyeda2kicad:SW-TH_6P-L8.0-W8.0-P2.50
- removed U22, U23, U30, U31: XXL1509-5.0, easyeda2kicad:SOIC-8_L4.9-W3.9-P1.27-LS6.0-BL
- removed U24, U28, U32, U36: NDP23511KC, easyeda2kicad:SOP-8_L4.9-W3.9-P1.27-LS6.0-BL
- removed U25, U29, U33, U37: CYPD3175-24LQXQ, Package_DFN_QFN:QFN-24-1EP_4x4mm_P0.5mm_EP2.7x2.7mm_ThermalVias
- removed U26, U27, U34, U35: LS0505EVD22, LS0505EVD22:LS0505EVD22_LTF
- added H1: MountingHole_Pad, MountingHole:MountingHole_4mm_Pad_Via, F.Cu at (243.0, 67.5)
- added H2: MountingHole_Pad, MountingHole:MountingHole_4mm_Pad_Via, F.Cu at (195.2, 98.5)
- added H3: MountingHole_Pad, MountingHole:MountingHole_4mm_Pad_Via, F.Cu at (233.0, 139.7)
- added H4: MountingHole_Pad, MountingHole:MountingHole_4mm_Pad_Via, F.Cu at (238.8, 92.5)
- C55, C57, J15, L10, L2, L7, L8, L9: moved to B.Cu
- moved R38 194.2 mm to (227.7, 67.0), turned to 180 degrees
- moved R40 187.6 mm to (226.8, 71.6), turned to -90 degrees
- moved R39 184.7 mm to (219.2, 73.6), turned to 90 degrees
- moved L7 183.3 mm to (216.0, 61.9), turned to 180 degrees
- moved Q3 182.1 mm to (224.6, 62.8), turned to 90 degrees
- moved L9 181.9 mm to (230.5, 68.7), turned to -90 degrees
- moved R35 181.4 mm to (216.0, 68.5), turned to 180 degrees
- moved D15 177.9 mm to (217.3, 63.0), turned to 90 degrees
- moved J15 175.1 mm to (202.5, 68.2), turned to 90 degrees
- moved C78 173.3 mm to (232.5, 75.5), turned to 90 degrees
- moved R43 171.8 mm to (207.8, 69.2), turned to 180 degrees
- moved U14 171.7 mm to (211.9, 65.4)
- moved C79 171.1 mm to (229.5, 75.5), turned to 90 degrees
- moved C63 171.1 mm to (223.8, 54.5), turned to 180 degrees
- moved C64 170.9 mm to (226.1, 66.6), turned to -90 degrees
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Connections:
- net Net-(J11-DN1) renamed /USB 1/2_D-
- net Net-(J11-DP1) renamed /USB 1/2_D+
- net Net-(J13-DN1) renamed /USB 2/1_D-
- net Net-(J13-DP1) renamed /USB 2/1_D+
- net Net-(J16-DN1) renamed /USB 2/2_D-
- net Net-(J16-DP1) renamed /USB 2/2_D+
- net Net-(J8-DN1) renamed /USB 1/1_D-
- net Net-(J8-DP1) renamed /USB 1/1_D+
- J11 pad 0: GND -> Net-(J11-EH)
- J11 pad A1: Net-(U13-CSP) -> Net-(J11-EH)
- J11 pad A12: Net-(U13-CSP) -> Net-(J11-EH)
- J11 pad B1: Net-(U13-CSP) -> Net-(J11-EH)
- J11 pad B12: Net-(U13-CSP) -> Net-(J11-EH)
- J13 pad 0: GND -> Net-(J13-EH)
- J13 pad A1: Net-(U17-CSP) -> Net-(J13-EH)
- J13 pad A12: Net-(U17-CSP) -> Net-(J13-EH)
- J13 pad B1: Net-(U17-CSP) -> Net-(J13-EH)
- J13 pad B12: Net-(U17-CSP) -> Net-(J13-EH)
- J16 pad 0: GND -> Net-(J16-EH)
- J16 pad A1: Net-(U21-CSP) -> Net-(J16-EH)
- J16 pad A12: Net-(U21-CSP) -> Net-(J16-EH)
- J16 pad B1: Net-(U21-CSP) -> Net-(J16-EH)
- J16 pad B12: Net-(U21-CSP) -> Net-(J16-EH)
- J8 pad 0: GND -> Net-(J8-EH)
- J8 pad A1: Net-(U9-CSP) -> Net-(J8-EH)
- J8 pad A12: Net-(U9-CSP) -> Net-(J8-EH)
- J8 pad B1: Net-(U9-CSP) -> Net-(J8-EH)
- J8 pad B12: Net-(U9-CSP) -> Net-(J8-EH)
- R25 pad 1: Net-(U9-CSP) -> Net-(J8-EH)
- R34 pad 1: Net-(U13-CSP) -> Net-(J11-EH)
- R34 pad 2: GND -> Net-(R34-Pad2)
- R41 pad 1: Net-(U17-CSP) -> Net-(J13-EH)
- R50 pad 1: Net-(U21-CSP) -> Net-(J16-EH)
- TP1 pad 1: Net-(LED20-DOUT) -> Net-(LED5-DOUT)
- U13 pad 19: Net-(U13-CSP) -> Net-(J11-EH)
- U13 pad 22: GND -> Net-(R34-Pad2)
- U13 pad 25: GND -> Net-(R34-Pad2)
- U17 pad 19: Net-(U17-CSP) -> Net-(J13-EH)
- U21 pad 19: Net-(U21-CSP) -> Net-(J16-EH)
- U9 pad 19: Net-(U9-CSP) -> Net-(J8-EH)
Routing:
- net SDA: track 0.00 -> 185.0 mm, vias 0 -> 12
- net SCL: track 0.00 -> 153.8 mm, vias 0 -> 10
- net +5V: track 4.20 -> 151.5 mm, vias 2 -> 46
- net Net-(Q1-D): track 0.00 -> 131.3 mm, vias 0 -> 25
- net Net-(Q3-D): track 0.00 -> 117.1 mm, vias 0 -> 25
- net /USB 2/D_5V: track 0.00 -> 91.5 mm, vias 0 -> 62
- net /USB 1/D_5V: track 0.00 -> 82.4 mm, vias 0 -> 53
- net GND: track 34.1 -> 111.1 mm, vias 5 -> 52
- net Net-(Q3-S): track 0.00 -> 75.3 mm, vias 0 -> 20
- net Net-(Q1-S): track 0.00 -> 75.3 mm, vias 0 -> 21
- net Net-(J16-EH): track 0.00 -> 56.5 mm, vias 0 -> 9
- net Net-(Q2-D): track 0.00 -> 54.6 mm, vias 0 -> 12
- net Net-(D13-K): track 0.00 -> 51.6 mm, vias 0 -> 30
- net Net-(Q4-D): track 0.00 -> 51.5 mm, vias 0 -> 9
- net /USB 1/U_5V: track 0.00 -> 51.4 mm, vias 0 -> 6
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- added copper zone on In1.Cu, net +5V
- added copper zone on In1.Cu, net /USB 1/D_5V
- added copper zone on In1.Cu, net /USB 2/D_5V
- added copper zone on F.Cu, net Net-(D12-K)
- added copper zone on In2.Cu, net Net-(D12-K)
- added copper zone on F.Cu, net Net-(J10-D-VCC)
- added copper zone on F.Cu, net Net-(J15-D-VCC)
- added copper zone on F.Cu, net Net-(Q2-S)
- added copper zone on In2.Cu, net Net-(Q2-S)
- added copper zone on F.Cu, net Net-(Q4-S)
- added copper zone on In2.Cu, net Net-(Q4-S)
- added copper zone on F.Cu, net VDC
Other:
- board size 100 x 100 mm -> 80 x 95 mm
- board text added: "istg everything better fit..."
