File: usb-charging-hub.kicad_pcb (KiCad board)
At the start: 4 copper layers, 80 x 95 mm, 214 parts, among them J1 Conn_01x01_Pin, J10 XDUF-0426-081_C18202150, J11 TYPE-C 16PLT-H10.0, J12 Conn_01x04_Pin, J13 TYPE-C 16PLT-H10.0, J14 Conn_01x04_Pin, J15 XDUF-0426-081_C18202150, J16 TYPE-C 16PLT-H10.0, J17 Conn_01x04_Pin, J2 Conn_01x01_Pin, J35 GT-USB-7010ASV, J4 Conn_01x04_Pin, J6 Conn_01x04_Pin, J7 Conn_01x04_Pin, J8 TYPE-C 16PLT-H10.0, J9 Conn_01x04_Pin, Q1 PMOS, Q2 PMOS, Q3 PMOS, Q4 PMOS, SW1 TS24CA, SW2 Latching, SW3 TS24CA, SW4 TS24CA, U1 W25Q32JVSS, U10 LS0505EVD22, U11 LS0505EVD22, U12 NDP23511KC, U13 CYPD3175-24LQXQ, U14 XXL1509-5.0, U15 XXL1509-5.0, U16 NDP23511KC, U17 CYPD3175-24LQXQ, U18 LS0505EVD22, U19 LS0505EVD22, U2 ABM8-272-T3_C20625731, U20 NDP23511KC, U21 CYPD3175-24LQXQ, U3 RP2040, U4 LM2596S-3.3, U5 XXL1509-5.0, U6 XXL1509-5.0, U7 XXL1509-5.0, U8 NDP23511KC, U9 CYPD3175-24LQXQ

Commit message: fix some errors and add some art :3
Signed-off-by: Toby Cm <toby@vsus.app>
Parts:
- moved H3 1.60 mm to (234.6, 139.7)
Routing:
- net Net-(D14-K): track 19.1 -> 24.2 mm, vias 32 -> 42
- net Net-(U3-GPIO19): track 19.2 -> 19.8 mm
- net SCL: vias 10 -> 9
- net Net-(Q1-S): vias 21 -> 20
- net Net-(J10-D-VCC): vias 2 -> 3
- net Net-(D13-K): vias 30 -> 29
- net Net-(D11-K): vias 37 -> 17
- added copper zone on In1.Cu, net Net-(J10-D-VCC)
Other:
- outline, holes or cut-outs redrawn
- board text added: "- tobycm 2025"
- board text added: "100W+?"
- board text added: "30V Max pretty sure"
- board text added: "4xUSB C: 100W+? 4xUSB A: Max 5V 3A"
- board text added: "Itai"
- board text added: "Mom"
- board text added: "RUN"
- board text added: "Scarlett Steyn"
- board text added: "Special thanks to"
- board text added: "Status"
- board text added: "USB Charging Hub!"
- board text added: "beloved"
- board text added: "benny"
- board text added: "copyup 2025 @tobycm"
- board text added: "dinhq"
- board text added: "elysia.dev"
- board text added: "ender"
- board text added: "for running #reflow"
- board text added: "fosly"
- board text added: "kenji"
- board text added: "mintyminh"
- board text added: "my"
- board text added: "nbth"
- board text added: "nguyen.dev"
- board text added: "none"
- board text added: "tobycm.dev toby@vsus.app"
