File: ti_usb_c.kicad_sch (KiCad schematic)
At the start: 2 parts, among them J3 TYPE-C 16PLT-H10.0, U7 PTPS25751DREFR

Commit message: gave up on single board, gonna make small modules
Signed-off-by: Toby Cm <toby@vsus.app>
Parts:
- U7: footprint WQFN38_REF_TEX -> TPS25751DREFR:WQFN38_REF_TEX
Changed lines of the file:
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@@
 			)
 		)
-		(property "Footprint" "WQFN38_REF_TEX"
+		(property "Footprint" "TPS25751DREFR:WQFN38_REF_TEX"
 			(at 140.97 36.83 0)
 			(effects
@@
 		(dnp no)
 		(fields_autoplaced yes)
-		(property "Reference" "#PWR0110"
+		(property "Reference" "#PWR0111"
 			(at 147.32 36.83 0)
 			(effects
@@
 			(project "usb-charging-hub"
 				(path "/04e54dfe-f06f-40ed-b860-573373578cb0/5742c913-e105-4d4e-8f73-4e0de26022fb"
-					(reference "#PWR0110")
+					(reference "#PWR0111")
 					(unit 1)
 				)
@@
 		(dnp no)
 		(fields_autoplaced yes)
-		(property "Reference" "#PWR0111"
+		(property "Reference" "#PWR0110"
 			(at 58.42 77.47 0)
 			(effects
@@
 			(project "usb-charging-hub"
 				(path "/04e54dfe-f06f-40ed-b860-573373578cb0/5742c913-e105-4d4e-8f73-4e0de26022fb"
-					(reference "#PWR0111")
+					(reference "#PWR0110")
 					(unit 1)
 				)
