File: neopixel.kicad_sch (KiCad schematic)
At the start: 4 parts, among them J14 Conn_01x03_Pin, J15 Conn_01x02_Pin, J3 Conn_01x03_Pin

Commit message: updated journal, pin headers footprint, etc. added labels to rp2350b, finished pcb routing. time to start on other modules yay
Signed-off-by: Toby Cm <toby@vsus.app>
Parts:
- J5: renamed from J3; footprint (none) -> Connector_PinHeader_2.54mm:PinHeader_1x03_P2.54mm_Vertical
- J6: renamed from J14; footprint (none) -> Connector_PinHeader_2.54mm:PinHeader_1x03_P2.54mm_Vertical
- J7: renamed from J15; footprint (none) -> Connector_PinHeader_2.54mm:PinHeader_1x02_P2.54mm_Vertical
- renumbered LED20 to LED1
Changed lines of the file:
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@@
 		(on_board yes)
 		(dnp no)
-		(property "Reference" "J15"
+		(property "Reference" "J7"
 			(at 188.976 61.468 0)
 			(effects
@@
 			)
 		)
-		(property "Footprint" ""
+		(property "Footprint" "Connector_PinHeader_2.54mm:PinHeader_1x02_P2.54mm_Vertical"
 			(at 185.42 62.23 0)
 			(effects
@@
 			(project "usb-charging-hub"
 				(path "/04e54dfe-f06f-40ed-b860-573373578cb0/7fcba1a5-c6dd-4722-bd30-8c494eb4bcd7"
-					(reference "J15")
+					(reference "J7")
 					(unit 1)
 				)
@@
 		(dnp no)
 		(fields_autoplaced yes)
-		(property "Reference" "#PWR0105"
+		(property "Reference" "#PWR041"
 			(at 171.45 52.07 0)
 			(effects
@@
 			(project "usb-charging-hub"
 				(path "/04e54dfe-f06f-40ed-b860-573373578cb0/7fcba1a5-c6dd-4722-bd30-8c494eb4bcd7"
-					(reference "#PWR0105")
+					(reference "#PWR041")
 					(unit 1)
 				)
@@
 		(on_board yes)
 		(dnp no)
-		(property "Reference" "J3"
+		(property "Reference" "J5"
 			(at 148.971 41.148 0)
 			(effects
@@
 			)
 		)
-		(property "Footprint" ""
+		(property "Footprint" "Connector_PinHeader_2.54mm:PinHeader_1x03_P2.54mm_Vertical"
 			(at 151.13 43.18 0)
 			(effects
@@
 			(project "usb-charging-hub"
 				(path "/04e54dfe-f06f-40ed-b860-573373578cb0/7fcba1a5-c6dd-4722-bd30-8c494eb4bcd7"
-					(reference "J3")
+					(reference "J5")
 					(unit 1)
 				)
@@
 		(on_board yes)
 		(dnp no)
-		(property "Reference" "J14"
+		(property "Reference" "J6"
 			(at 148.971 56.388 0)
 			(effects
@@
 			)
 		)
-		(property "Footprint" ""
+		(property "Footprint" "Connector_PinHeader_2.54mm:PinHeader_1x03_P2.54mm_Vertical"
 			(at 151.13 58.42 0)
 			(effects
@@
 			(project "usb-charging-hub"
 				(path "/04e54dfe-f06f-40ed-b860-573373578cb0/7fcba1a5-c6dd-4722-bd30-8c494eb4bcd7"
-					(reference "J14")
+					(reference "J6")
 					(unit 1)
 				)
@@
 		(on_board yes)
 		(dnp no)
-		(property "Reference" "LED20"
+		(property "Reference" "LED1"
 			(at 184.15 34.798 0)
 			(effects
@@
 			(project "usb-charging-hub"
 				(path "/04e54dfe-f06f-40ed-b860-573373578cb0/7fcba1a5-c6dd-4722-bd30-8c494eb4bcd7"
-					(reference "LED20")
+					(reference "LED1")
 					(unit 1)
 				)
@@
 		(dnp no)
 		(fields_autoplaced yes)
-		(property "Reference" "#PWR0106"
+		(property "Reference" "#PWR042"
 			(at 196.85 57.15 0)
 			(effects
@@
 			(project "usb-charging-hub"
 				(path "/04e54dfe-f06f-40ed-b860-573373578cb0/7fcba1a5-c6dd-4722-bd30-8c494eb4bcd7"
-					(reference "#PWR0106")
+					(reference "#PWR042")
 					(unit 1)
 				)
@@
 		(dnp no)
 		(fields_autoplaced yes)
-		(property "Reference" "#PWR0107"
+		(property "Reference" "#PWR040"
 			(at 156.21 44.45 0)
 			(effects
@@
 			(project "usb-charging-hub"
 				(path "/04e54dfe-f06f-40ed-b860-573373578cb0/7fcba1a5-c6dd-4722-bd30-8c494eb4bcd7"
-					(reference "#PWR0107")
+					(reference "#PWR040")
 					(unit 1)
 				)
@@
 		(dnp no)
 		(fields_autoplaced yes)
-		(property "Reference" "#PWR067"
+		(property "Reference" "#PWR043"
 			(at 156.21 67.31 0)
 			(effects
@@
 			(project "usb-charging-hub"
 				(path "/04e54dfe-f06f-40ed-b860-573373578cb0/7fcba1a5-c6dd-4722-bd30-8c494eb4bcd7"
-					(reference "#PWR067")
-					(unit 1)
-				)
+					(reference "#PWR043")
+					(unit 1)
+				)
