File: usbc.kicad_sch (KiCad schematic)
At the start: 9 parts, among them J11 TYPE-C 16PLT-H10.0, J12 Conn_01x04_Pin, J13 Conn_01x08_Pin, U11 PUSB3FR4-ES

Commit message: updated journal, pin headers footprint, etc. added labels to rp2350b, finished pcb routing. time to start on other modules yay
Signed-off-by: Toby Cm <toby@vsus.app>
Parts:
- removed J13: Conn_01x08_Pin, symbol Connector:Conn_01x08_Pin
- added J14, J17: Conn_01x04_Pin, Connector_PinHeader_2.54mm:PinHeader_1x04_P2.54mm_Vertical, symbol Connector:Conn_01x04_Pin
- J15: renamed from J12; footprint (none) -> Connector_PinHeader_2.54mm:PinHeader_1x04_P2.54mm_Vertical
- renumbered D14 to D10, J11 to J16, R16 to R10, R17 to R11, R15 to R13, U11 to U9
Connections:
- net GND: now also J17.1 (Pin_1), J17.2 (Pin_2), J17.3 (Pin_3), J17.4 (Pin_4)
- net VDC: now also J14.1 (Pin_1), J14.2 (Pin_2), J14.3 (Pin_3), J14.4 (Pin_4)
