File: 3.3v.kicad_sch (KiCad schematic)
At the start: 10 parts, among them J4 Conn_01x04_Pin, J5 Conn_01x04_Pin, U12 LM2596S-3.3

Commit message: updated journal, pin headers footprint, etc. added labels to rp2350b, finished pcb routing. time to start on other modules yay
Signed-off-by: Toby Cm <toby@vsus.app>
Parts:
- C10: renamed from C17; footprint (none) -> Capacitor_SMD:C_0603_1608Metric_Pad1.08x0.95mm_HandSolder
- C11: renamed from C15; footprint Capacitor_THT:CP_Radial_D17.0mm_P7.50mm -> Capacitor_THT:CP_Radial_D10.0mm_P5.00mm
- C12: renamed from C16; footprint (none) -> Capacitor_SMD:C_0603_1608Metric_Pad1.08x0.95mm_HandSolder
- C9: renamed from C12; footprint Capacitor_THT:CP_Radial_D17.0mm_P7.50mm -> Capacitor_THT:CP_Radial_D10.0mm_P5.00mm
- L2: renamed from L5; value 33uH,2.7(Isat) -> 33uH,4.25A; footprint (none) -> misc:SDRI129-330MT
- renumbered D12 to D8, J5 to J10, J4 to J11, R13 to R8, U12 to U7
Changed lines of the file:
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@@
 		(on_board yes)
 		(dnp no)
-		(property "Reference" "C15"
+		(property "Reference" "C11"
 			(at 100.33 54.6988 0)
 			(effects
@@
 			)
 		)
-		(property "Footprint" "Capacitor_THT:CP_Radial_D17.0mm_P7.50mm"
+		(property "Footprint" "Capacitor_THT:CP_Radial_D10.0mm_P5.00mm"
 			(at 102.87 57.15 0)
 			(effects
@@
 			(project "usb-charging-hub"
 				(path "/04e54dfe-f06f-40ed-b860-573373578cb0/cdc79840-31c5-4d0c-9732-2009c0e35a21"
-					(reference "C15")
+					(reference "C11")
 					(unit 1)
 				)
@@
 		(dnp no)
 		(fields_autoplaced yes)
-		(property "Reference" "#PWR0124"
+		(property "Reference" "#PWR058"
 			(at 39.37 68.58 0)
 			(effects
@@
 			(project "usb-charging-hub"
 				(path "/04e54dfe-f06f-40ed-b860-573373578cb0/cdc79840-31c5-4d0c-9732-2009c0e35a21"
-					(reference "#PWR0124")
+					(reference "#PWR058")
 					(unit 1)
 				)
@@
 		(dnp no)
 		(fields_autoplaced yes)
-		(property "Reference" "L5"
+		(property "Reference" "L2"
 			(at 92.71 44.45 90)
 			(effects
@@
 			)
 		)
-		(property "Value" "33uH,2.7(Isat)"
+		(property "Value" "33uH,4.25A"
 			(at 92.71 48.26 90)
 			(effects
@@
 			)
 		)
-		(property "Footprint" ""
+		(property "Footprint" "misc:SDRI129-330MT"
 			(at 92.71 52.07 0)
 			(effects
@@
 			(project "usb-charging-hub"
 				(path "/04e54dfe-f06f-40ed-b860-573373578cb0/cdc79840-31c5-4d0c-9732-2009c0e35a21"
-					(reference "L5")
+					(reference "L2")
 					(unit 1)
 				)
@@
 		(on_board yes)
 		(dnp no)
-		(property "Reference" "#PWR0128"
+		(property "Reference" "#PWR057"
 			(at 147.32 67.31 0)
 			(effects
@@
 			(project ""
 				(path "/04e54dfe-f06f-40ed-b860-573373578cb0/cdc79840-31c5-4d0c-9732-2009c0e35a21"
-					(reference "#PWR0128")
+					(reference "#PWR057")
 					(unit 1)
 				)
@@
 		(dnp no)
 		(fields_autoplaced yes)
-		(property "Reference" "C17"
+		(property "Reference" "C10"
 			(at 36.83 32.3912 0)
 			(effects
@@
 			)
 		)
-		(property "Footprint" ""
+		(property "Footprint" "Capacitor_SMD:C_0603_1608Metric_Pad1.08x0.95mm_HandSolder"
 			(at 34.29 34.29 0)
 			(effects
@@
 			(project ""
 				(path "/04e54dfe-f06f-40ed-b860-573373578cb0/cdc79840-31c5-4d0c-9732-2009c0e35a21"
-					(reference "C17")
+					(reference "C10")
 					(unit 1)
 				)
@@
 		(on_board yes)
 		(dnp no)
-		(property "Reference" "C12"
+		(property "Reference" "C9"
 			(at 26.67 31.8388 0)
 			(effects
@@
 			)
 		)
-		(property "Footprint" "Capacitor_THT:CP_Radial_D17.0mm_P7.50mm"
+		(property "Footprint" "Capacitor_THT:CP_Radial_D10.0mm_P5.00mm"
 			(at 29.21 34.29 0)
 			(effects
@@
 			(project "usb-charging-hub"
 				(path "/04e54dfe-f06f-40ed-b860-573373578cb0/cdc79840-31c5-4d0c-9732-2009c0e35a21"
-					(reference "C12")
+					(reference "C9")
 					(unit 1)
 				)
@@
 		(dnp no)
 		(fields_autoplaced yes)
-		(property "Reference" "#PWR0132"
+		(property "Reference" "#PWR054"
 			(at 147.32 57.15 0)
 			(effects
@@
 			(project ""
 				(path "/04e54dfe-f06f-40ed-b860-573373578cb0/cdc79840-31c5-4d0c-9732-2009c0e35a21"
-					(reference "#PWR0132")
+					(reference "#PWR054")
 					(unit 1)
 				)
@@
 		(on_board yes)
 		(dnp no)
-		(property "Reference" "J5"
+		(property "Reference" "J10"
 			(at 177.546 47.498 0)
 			(effects
@@
 			(project ""
 				(path "/04e54dfe-f06f-40ed-b860-573373578cb0/cdc79840-31c5-4d0c-9732-2009c0e35a21"
-					(reference "J5")
+					(reference "J10")
 					(unit 1)
 				)
@@
 		(dnp no)
 		(fields_autoplaced yes)
-		(property "Reference" "#PWR0125"
+		(property "Reference" "#PWR051"
 			(at 46.99 46.99 0)
 			(effects
@@
 			(project "usb-charging-hub"
 				(path "/04e54dfe-f06f-40ed-b860-573373578cb0/cdc79840-31c5-4d0c-9732-2009c0e35a21"
-					(reference "#PWR0125")
+					(reference "#PWR051")
 					(unit 1)
 				)
@@
 		(dnp no)
 		(fields_autoplaced yes)
-		(property "Reference" "#PWR0130"
+		(property "Reference" "#PWR055"
 			(at 182.88 57.15 0)
 			(effects
@@
 			(project ""
 				(path "/04e54dfe-f06f-40ed-b860-573373578cb0/cdc79840-31c5-4d0c-9732-2009c0e35a21"
-					(reference "#PWR0130")
+					(reference "#PWR055")
 					(unit 1)
 				)
@@
 		(dnp no)
 		(fields_autoplaced yes)
-		(property "Reference" "#PWR0126"
+		(property "Reference" "#PWR056"
 			(at 55.88 63.5 0)
 			(effects
@@
 			(project "usb-charging-hub"
 				(path "/04e54dfe-f06f-40ed-b860-573373578cb0/cdc79840-31c5-4d0c-9732-2009c0e35a21"
-					(reference "#PWR0126")
+					(reference "#PWR056")
 					(unit 1)
 				)
@@
 		(dnp no)
 		(fields_autoplaced yes)
-		(property "Reference" "J4"
+		(property "Reference" "J11"
 			(at 153.67 55.2449 0)
 			(effects
@@
 			(project ""
 				(path "/04e54dfe-f06f-40ed-b860-573373578cb0/cdc79840-31c5-4d0c-9732-2009c0e35a21"
-					(reference "J4")
+					(reference "J11")
 					(unit 1)
 				)
@@
 		(dnp no)
 		(fields_autoplaced yes)
-		(property "Reference" "#PWR0122"
+		(property "Reference" "#PWR049"
 			(at 31.75 35.56 0)
 			(effects
@@
 			(project "usb-charging-hub"
 				(path "/04e54dfe-f06f-40ed-b860-573373578cb0/cdc79840-31c5-4d0c-9732-2009c0e35a21"
-					(reference "#PWR0122")
+					(reference "#PWR049")
 					(unit 1)
 				)
@@
 		(dnp no)
 		(fields_autoplaced yes)
-		(property "Reference" "#PWR0129"
+		(property "Reference" "#PWR059"
 			(at 85.09 68.58 0)
 			(effects
@@
 			(project "usb-charging-hub"
 				(path "/04e54dfe-f06f-40ed-b860-573373578cb0/cdc79840-31c5-4d0c-9732-2009c0e35a21"
-					(reference "#PWR0129")
+					(reference "#PWR059")
 					(unit 1)
 				)
@@
 		(dnp no)
 		(fields_autoplaced yes)
-		(property "Reference" "#PWR0127"
+		(property "Reference" "#PWR052"
 			(at 64.77 46.99 0)
 			(effects
@@
 			(project "usb-charging-hub"
 				(path "/04e54dfe-f06f-40ed-b860-573373578cb0/cdc79840-31c5-4d0c-9732-2009c0e35a21"
-					(reference "#PWR0127")
+					(reference "#PWR052")
 					(unit 1)
 				)
@@
 		(dnp no)
 		(fields_autoplaced yes)
-		(property "Reference" "#PWR0123"
+		(property "Reference" "#PWR050"
 			(at 31.75 43.18 0)
 			(effects
@@
 			(project "usb-charging-hub"
 				(path "/04e54dfe-f06f-40ed-b860-573373578cb0/cdc79840-31c5-4d0c-9732-2009c0e35a21"
-					(reference "#PWR0123")
+					(reference "#PWR050")
 					(unit 1)
 				)
@@
 		(on_board yes)
 		(dnp no)
-		(property "Reference" "C16"
+		(property "Reference" "C12"
 			(at 113.03 54.61 0)
 			(effects
@@
 			)
 		)
-		(property "Footprint" ""
+		(property "Footprint" "Capacitor_SMD:C_0603_1608Metric_Pad1.08x0.95mm_HandSolder"
 			(at 115.57 57.15 0)
 			(effects
@@
 			(project ""
 				(path "/04e54dfe-f06f-40ed-b860-573373578cb0/cdc79840-31c5-4d0c-9732-2009c0e35a21"
-					(reference "C16")
+					(reference "C12")
 					(unit 1)
 				)
@@
 		(dnp no)
 		(fields_autoplaced yes)
-		(property "Reference" "#PWR0131"
+		(property "Reference" "#PWR053"
 			(at 114.3 52.07 0)
 			(effects
@@
 			(project "usb-charging-hub"
 				(path "/04e54dfe-f06f-40ed-b860-573373578cb0/cdc79840-31c5-4d0c-9732-2009c0e35a21"
-					(reference "#PWR0131")
+					(reference "#PWR053")
 					(unit 1)
 				)
@@
 		(on_board yes)
 		(dnp no)
-		(property "Reference" "R13"
+		(property "Reference" "R8"
 			(at 35.814 56.134 0)
 			(effects
@@
 			(project "usb-charging-hub"
 				(path "/04e54dfe-f06f-40ed-b860-573373578cb0/cdc79840-31c5-4d0c-9732-2009c0e35a21"
-					(reference "R13")
+					(reference "R8")
 					(unit 1)
 				)
@@
 		(on_board yes)
 		(dnp no)
-		(property "Reference" "D12"
+		(property "Reference" "D8"
 			(at 82.55 54.9274 90)
 			(effects
@@
 			(project "usb-charging-hub"
 				(path "/04e54dfe-f06f-40ed-b860-573373578cb0/cdc79840-31c5-4d0c-9732-2009c0e35a21"
-					(reference "D12")
+					(reference "D8")
 					(unit 1)
 				)
@@
 		(dnp no)
 		(fields_autoplaced yes)
-		(property "Reference" "U12"
+		(property "Reference" "U7"
 			(at 55.88 38.1 0)
 			(effects
@@
 			(project "usb-charging-hub"
 				(path "/04e54dfe-f06f-40ed-b860-573373578cb0/cdc79840-31c5-4d0c-9732-2009c0e35a21"
-					(reference "U12")
-					(unit 1)
-				)
+					(reference "U7")
+					(unit 1)
+				)

Commit message: no more modules, its gonna work first try :fire: i love infineon and their ICs so much
Signed-off-by: Toby Cm <toby@vsus.app>
Parts:
- added D10: 60V,10A, Diode_SMD:D_SMB_Handsoldering, symbol Device:D_Schottky
- added D9: 40V,10A, Diode_SMD:D_SMB_Handsoldering, symbol Device:D_Schottky
- renumbered C9 to C16, C10 to C17, C11 to C18, C12 to C19, D8 to D11, J10 to J4, J11 to J5, L2 to L1, R8 to R17, U7 to U4
Connections:
- net VDC: now also D10.2 (A); no longer U4.1 (VIN)
- new net: D10.1 (K), D9.1 (K), U4.1 (VIN)
- new net +5V: D9.2 (A)
Other:
- moved on the sheet: C16, C17

Commit message: finished schematic yay!! now onto pcb routing :fire:
Other:
- moved on the sheet: C16, C17, C18, C19, D10, D11, D9, J4, J5, L1, R17, U4
