File: 5v.kicad_sch (KiCad schematic)
At the start: 9 parts, among them J7 Conn_01x04_Pin, J8 Conn_01x04_Pin, U13 XXL1509-5.0

Commit message: updated journal, pin headers footprint, etc. added labels to rp2350b, finished pcb routing. time to start on other modules yay
Signed-off-by: Toby Cm <toby@vsus.app>
Parts:
- C13: renamed from C18; footprint (none) -> Capacitor_SMD:C_1206_3216Metric_Pad1.33x1.80mm_HandSolder
- C14: renamed from C19; value 180uF,35V -> 35V,180uF
- C15: renamed from C20; value 22uF,35V -> 35V,22uF; footprint (none) -> Capacitor_SMD:C_0805_2012Metric_Pad1.18x1.45mm_HandSolder
- renumbered D13 to D9, J8 to J12, J7 to J13, L6 to L3, R14 to R9, U13 to U8
Changed lines of the file:
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@@
 		(on_board yes)
 		(dnp no)
-		(property "Reference" "#PWR0143"
+		(property "Reference" "#PWR067"
 			(at 168.91 53.34 0)
 			(effects
@@
 			(project "usb-charging-hub"
 				(path "/04e54dfe-f06f-40ed-b860-573373578cb0/8b94d9f0-b4ab-48ff-a9ac-e3216038869f"
-					(reference "#PWR0143")
+					(reference "#PWR067")
 					(unit 1)
 				)
@@
 		(dnp no)
 		(fields_autoplaced yes)
-		(property "Reference" "#PWR0142"
+		(property "Reference" "#PWR063"
 			(at 168.91 43.18 0)
 			(effects
@@
 			(project "usb-charging-hub"
 				(path "/04e54dfe-f06f-40ed-b860-573373578cb0/8b94d9f0-b4ab-48ff-a9ac-e3216038869f"
-					(reference "#PWR0142")
+					(reference "#PWR063")
 					(unit 1)
 				)
@@
 		(dnp no)
 		(fields_autoplaced yes)
-		(property "Reference" "#PWR0144"
+		(property "Reference" "#PWR064"
 			(at 204.47 43.18 0)
 			(effects
@@
 			(project ""
 				(path "/04e54dfe-f06f-40ed-b860-573373578cb0/8b94d9f0-b4ab-48ff-a9ac-e3216038869f"
-					(reference "#PWR0144")
+					(reference "#PWR064")
 					(unit 1)
 				)
@@
 		(dnp no)
 		(fields_autoplaced yes)
-		(property "Reference" "#PWR0139"
+		(property "Reference" "#PWR069"
 			(at 104.14 60.96 0)
 			(effects
@@
 			(project "usb-charging-hub"
 				(path "/04e54dfe-f06f-40ed-b860-573373578cb0/8b94d9f0-b4ab-48ff-a9ac-e3216038869f"
-					(reference "#PWR0139")
+					(reference "#PWR069")
 					(unit 1)
 				)
@@
 		(on_board yes)
 		(dnp no)
-		(property "Reference" "C19"
+		(property "Reference" "C14"
 			(at 129.54 48.26 0)
 			(effects
@@
 			)
 		)
-		(property "Value" "180uF,35V"
+		(property "Value" "35V,180uF"
 			(at 129.54 50.8888 0)
 			(effects
@@
 			(project "usb-charging-hub"
 				(path "/04e54dfe-f06f-40ed-b860-573373578cb0/8b94d9f0-b4ab-48ff-a9ac-e3216038869f"
-					(reference "C19")
+					(reference "C14")
 					(unit 1)
 				)
@@
 		(dnp no)
 		(fields_autoplaced yes)
-		(property "Reference" "C18"
+		(property "Reference" "C13"
 			(at 34.29 38.7412 0)
 			(effects
@@
 			)
 		)
-		(property "Footprint" ""
+		(property "Footprint" "Capacitor_SMD:C_1206_3216Metric_Pad1.33x1.80mm_HandSolder"
 			(at 31.75 40.64 0)
 			(effects
@@
 			(project ""
 				(path "/04e54dfe-f06f-40ed-b860-573373578cb0/8b94d9f0-b4ab-48ff-a9ac-e3216038869f"
-					(reference "C18")
+					(reference "C13")
 					(unit 1)
 				)
@@
 		(dnp no)
 		(fields_autoplaced yes)
-		(property "Reference" "#PWR0135"
+		(property "Reference" "#PWR065"
 			(at 31.75 49.53 0)
 			(effects
@@
 			(project "usb-charging-hub"
 				(path "/04e54dfe-f06f-40ed-b860-573373578cb0/8b94d9f0-b4ab-48ff-a9ac-e3216038869f"
-					(reference "#PWR0135")
+					(reference "#PWR065")
 					(unit 1)
 				)
@@
 		(on_board yes)
 		(dnp no)
-		(property "Reference" "J8"
+		(property "Reference" "J12"
 			(at 198.882 33.274 0)
 			(effects
@@
 			(project "usb-charging-hub"
 				(path "/04e54dfe-f06f-40ed-b860-573373578cb0/8b94d9f0-b4ab-48ff-a9ac-e3216038869f"
-					(reference "J8")
+					(reference "J12")
 					(unit 1)
 				)
@@
 		(on_board yes)
 		(dnp no)
-		(property "Reference" "D13"
+		(property "Reference" "D9"
 			(at 106.68 47.3074 90)
 			(effects
@@
 			(project "usb-charging-hub"
 				(path "/04e54dfe-f06f-40ed-b860-573373578cb0/8b94d9f0-b4ab-48ff-a9ac-e3216038869f"
-					(reference "D13")
+					(reference "D9")
 					(unit 1)
 				)
@@
 		(dnp no)
 		(fields_autoplaced yes)
-		(property "Reference" "#PWR0134"
+		(property "Reference" "#PWR062"
 			(at 31.75 41.91 0)
 			(effects
@@
 			(project "usb-charging-hub"
 				(path "/04e54dfe-f06f-40ed-b860-573373578cb0/8b94d9f0-b4ab-48ff-a9ac-e3216038869f"
-					(reference "#PWR0134")
+					(reference "#PWR062")
 					(unit 1)
 				)
@@
 		(on_board yes)
 		(dnp no)
-		(property "Reference" "R14"
+		(property "Reference" "R9"
 			(at 67.564 43.688 0)
 			(effects
@@
 			(project "usb-charging-hub"
 				(path "/04e54dfe-f06f-40ed-b860-573373578cb0/8b94d9f0-b4ab-48ff-a9ac-e3216038869f"
-					(reference "R14")
+					(reference "R9")
 					(unit 1)
 				)
@@
 		(dnp no)
 		(fields_autoplaced yes)
-		(property "Reference" "#PWR0138"
+		(property "Reference" "#PWR061"
 			(at 95.25 36.83 0)
 			(effects
@@
 			(project "usb-charging-hub"
 				(path "/04e54dfe-f06f-40ed-b860-573373578cb0/8b94d9f0-b4ab-48ff-a9ac-e3216038869f"
-					(reference "#PWR0138")
+					(reference "#PWR061")
 					(unit 1)
 				)
@@
 		(dnp no)
 		(fields_autoplaced yes)
-		(property "Reference" "J7"
+		(property "Reference" "J13"
 			(at 175.26 41.2749 0)
 			(effects
@@
 			(project "usb-charging-hub"
 				(path "/04e54dfe-f06f-40ed-b860-573373578cb0/8b94d9f0-b4ab-48ff-a9ac-e3216038869f"
-					(reference "J7")
+					(reference "J13")
 					(unit 1)
 				)
@@
 		(dnp no)
 		(fields_autoplaced yes)
-		(property "Reference" "#PWR0136"
+		(property "Reference" "#PWR068"
 			(at 69.85 58.42 0)
 			(effects
@@
 			(project "usb-charging-hub"
 				(path "/04e54dfe-f06f-40ed-b860-573373578cb0/8b94d9f0-b4ab-48ff-a9ac-e3216038869f"
-					(reference "#PWR0136")
+					(reference "#PWR068")
 					(unit 1)
 				)
@@
 		(dnp no)
 		(fields_autoplaced yes)
-		(property "Reference" "L6"
+		(property "Reference" "L3"
 			(at 116.84 36.83 0)
 			(effects
@@
 			(project ""
 				(path "/04e54dfe-f06f-40ed-b860-573373578cb0/8b94d9f0-b4ab-48ff-a9ac-e3216038869f"
-					(reference "L6")
+					(reference "L3")
 					(unit 1)
 				)
@@
 		(dnp no)
 		(fields_autoplaced yes)
-		(property "Reference" "U13"
+		(property "Reference" "U8"
 			(at 87.63 27.94 0)
 			(effects
@@
 			(project "usb-charging-hub"
 				(path "/04e54dfe-f06f-40ed-b860-573373578cb0/8b94d9f0-b4ab-48ff-a9ac-e3216038869f"
-					(reference "U13")
+					(reference "U8")
 					(unit 1)
 				)
@@
 		(dnp no)
 		(fields_autoplaced yes)
-		(property "Reference" "#PWR0141"
+		(property "Reference" "#PWR066"
 			(at 147.32 44.45 0)
 			(effects
@@
 			(project "usb-charging-hub"
 				(path "/04e54dfe-f06f-40ed-b860-573373578cb0/8b94d9f0-b4ab-48ff-a9ac-e3216038869f"
-					(reference "#PWR0141")
+					(reference "#PWR066")
 					(unit 1)
 				)
@@
 		(on_board yes)
 		(dnp no)
-		(property "Reference" "C20"
+		(property "Reference" "C15"
 			(at 146.05 46.99 0)
 			(effects
@@
 			)
 		)
-		(property "Value" "22uF,35V"
+		(property "Value" "35V,22uF"
 			(at 146.05 50.8 0)
 			(effects
@@
 			)
 		)
-		(property "Footprint" ""
+		(property "Footprint" "Capacitor_SMD:C_0805_2012Metric_Pad1.18x1.45mm_HandSolder"
 			(at 143.51 49.53 0)
 			(effects
@@
 			(project "usb-charging-hub"
 				(path "/04e54dfe-f06f-40ed-b860-573373578cb0/8b94d9f0-b4ab-48ff-a9ac-e3216038869f"
-					(reference "C20")
+					(reference "C15")
 					(unit 1)
 				)
@@
 		(dnp no)
 		(fields_autoplaced yes)
-		(property "Reference" "#PWR0137"
+		(property "Reference" "#PWR060"
 			(at 80.01 36.83 0)
 			(effects
@@
 			(project "usb-charging-hub"
 				(path "/04e54dfe-f06f-40ed-b860-573373578cb0/8b94d9f0-b4ab-48ff-a9ac-e3216038869f"
-					(reference "#PWR0137")
-					(unit 1)
-				)
+					(reference "#PWR060")
+					(unit 1)
+				)

Commit message: no more modules, its gonna work first try :fire: i love infineon and their ICs so much
Signed-off-by: Toby Cm <toby@vsus.app>
Parts:
- renumbered C13 to C20, C14 to C21, C15 to C22, D9 to D12, J12 to J6, J13 to J7, L3 to L2, R9 to R18, U8 to U5
Changed lines of the file:
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@@
 		(on_board yes)
 		(dnp no)
-		(property "Reference" "#PWR067"
+		(property "Reference" "#PWR050"
 			(at 168.91 53.34 0)
 			(effects
@@
 			(project "usb-charging-hub"
 				(path "/04e54dfe-f06f-40ed-b860-573373578cb0/8b94d9f0-b4ab-48ff-a9ac-e3216038869f"
-					(reference "#PWR067")
+					(reference "#PWR050")
 					(unit 1)
 				)
@@
 		(dnp no)
 		(fields_autoplaced yes)
-		(property "Reference" "#PWR063"
+		(property "Reference" "#PWR046"
 			(at 168.91 43.18 0)
 			(effects
@@
 			(project "usb-charging-hub"
 				(path "/04e54dfe-f06f-40ed-b860-573373578cb0/8b94d9f0-b4ab-48ff-a9ac-e3216038869f"
-					(reference "#PWR063")
+					(reference "#PWR046")
 					(unit 1)
 				)
@@
 		(dnp no)
 		(fields_autoplaced yes)
-		(property "Reference" "#PWR064"
+		(property "Reference" "#PWR047"
 			(at 204.47 43.18 0)
 			(effects
@@
 			(project ""
 				(path "/04e54dfe-f06f-40ed-b860-573373578cb0/8b94d9f0-b4ab-48ff-a9ac-e3216038869f"
-					(reference "#PWR064")
+					(reference "#PWR047")
 					(unit 1)
 				)
@@
 		(dnp no)
 		(fields_autoplaced yes)
-		(property "Reference" "#PWR069"
+		(property "Reference" "#PWR052"
 			(at 104.14 60.96 0)
 			(effects
@@
 			(project "usb-charging-hub"
 				(path "/04e54dfe-f06f-40ed-b860-573373578cb0/8b94d9f0-b4ab-48ff-a9ac-e3216038869f"
-					(reference "#PWR069")
+					(reference "#PWR052")
 					(unit 1)
 				)
@@
 		(on_board yes)
 		(dnp no)
-		(property "Reference" "C14"
+		(property "Reference" "C21"
 			(at 129.54 48.26 0)
 			(effects
@@
 			(project "usb-charging-hub"
 				(path "/04e54dfe-f06f-40ed-b860-573373578cb0/8b94d9f0-b4ab-48ff-a9ac-e3216038869f"
-					(reference "C14")
+					(reference "C21")
 					(unit 1)
 				)
@@
 		(dnp no)
 		(fields_autoplaced yes)
-		(property "Reference" "C13"
+		(property "Reference" "C20"
 			(at 34.29 38.7412 0)
 			(effects
@@
 			(project ""
 				(path "/04e54dfe-f06f-40ed-b860-573373578cb0/8b94d9f0-b4ab-48ff-a9ac-e3216038869f"
-					(reference "C13")
+					(reference "C20")
 					(unit 1)
 				)
@@
 		(dnp no)
 		(fields_autoplaced yes)
-		(property "Reference" "#PWR065"
+		(property "Reference" "#PWR048"
 			(at 31.75 49.53 0)
 			(effects
@@
 			(project "usb-charging-hub"
 				(path "/04e54dfe-f06f-40ed-b860-573373578cb0/8b94d9f0-b4ab-48ff-a9ac-e3216038869f"
-					(reference "#PWR065")
+					(reference "#PWR048")
 					(unit 1)
 				)
@@
 		(on_board yes)
 		(dnp no)
-		(property "Reference" "J12"
+		(property "Reference" "J6"
 			(at 198.882 33.274 0)
 			(effects
@@
 			(project "usb-charging-hub"
 				(path "/04e54dfe-f06f-40ed-b860-573373578cb0/8b94d9f0-b4ab-48ff-a9ac-e3216038869f"
-					(reference "J12")
+					(reference "J6")
 					(unit 1)
 				)
@@
 		(on_board yes)
 		(dnp no)
-		(property "Reference" "D9"
+		(property "Reference" "D12"
 			(at 106.68 47.3074 90)
 			(effects
@@
 			(project "usb-charging-hub"
 				(path "/04e54dfe-f06f-40ed-b860-573373578cb0/8b94d9f0-b4ab-48ff-a9ac-e3216038869f"
-					(reference "D9")
+					(reference "D12")
 					(unit 1)
 				)
@@
 		(dnp no)
 		(fields_autoplaced yes)
-		(property "Reference" "#PWR062"
+		(property "Reference" "#PWR045"
 			(at 31.75 41.91 0)
 			(effects
@@
 			(project "usb-charging-hub"
 				(path "/04e54dfe-f06f-40ed-b860-573373578cb0/8b94d9f0-b4ab-48ff-a9ac-e3216038869f"
-					(reference "#PWR062")
+					(reference "#PWR045")
 					(unit 1)
 				)
@@
 		(on_board yes)
 		(dnp no)
-		(property "Reference" "R9"
+		(property "Reference" "R18"
 			(at 67.564 43.688 0)
 			(effects
@@
 			(project "usb-charging-hub"
 				(path "/04e54dfe-f06f-40ed-b860-573373578cb0/8b94d9f0-b4ab-48ff-a9ac-e3216038869f"
-					(reference "R9")
+					(reference "R18")
 					(unit 1)
 				)
@@
 		(dnp no)
 		(fields_autoplaced yes)
-		(property "Reference" "#PWR061"
+		(property "Reference" "#PWR044"
 			(at 95.25 36.83 0)
 			(effects
@@
 			(project "usb-charging-hub"
 				(path "/04e54dfe-f06f-40ed-b860-573373578cb0/8b94d9f0-b4ab-48ff-a9ac-e3216038869f"
-					(reference "#PWR061")
+					(reference "#PWR044")
 					(unit 1)
 				)
@@
 		(dnp no)
 		(fields_autoplaced yes)
-		(property "Reference" "J13"
+		(property "Reference" "J7"
 			(at 175.26 41.2749 0)
 			(effects
@@
 			(project "usb-charging-hub"
 				(path "/04e54dfe-f06f-40ed-b860-573373578cb0/8b94d9f0-b4ab-48ff-a9ac-e3216038869f"
-					(reference "J13")
+					(reference "J7")
 					(unit 1)
 				)
@@
 		(dnp no)
 		(fields_autoplaced yes)
-		(property "Reference" "#PWR068"
+		(property "Reference" "#PWR051"
 			(at 69.85 58.42 0)
 			(effects
@@
 			(project "usb-charging-hub"
 				(path "/04e54dfe-f06f-40ed-b860-573373578cb0/8b94d9f0-b4ab-48ff-a9ac-e3216038869f"
-					(reference "#PWR068")
+					(reference "#PWR051")
 					(unit 1)
 				)
@@
 		(dnp no)
 		(fields_autoplaced yes)
-		(property "Reference" "L3"
+		(property "Reference" "L2"
 			(at 116.84 36.83 0)
 			(effects
@@
 			(project ""
 				(path "/04e54dfe-f06f-40ed-b860-573373578cb0/8b94d9f0-b4ab-48ff-a9ac-e3216038869f"
-					(reference "L3")
+					(reference "L2")
 					(unit 1)
 				)
@@
 		(dnp no)
 		(fields_autoplaced yes)
-		(property "Reference" "U8"
+		(property "Reference" "U5"
 			(at 87.63 27.94 0)
 			(effects
@@
 			(project "usb-charging-hub"
 				(path "/04e54dfe-f06f-40ed-b860-573373578cb0/8b94d9f0-b4ab-48ff-a9ac-e3216038869f"
-					(reference "U8")
+					(reference "U5")
 					(unit 1)
 				)
@@
 		(dnp no)
 		(fields_autoplaced yes)
-		(property "Reference" "#PWR066"
+		(property "Reference" "#PWR049"
 			(at 147.32 44.45 0)
 			(effects
@@
 			(project "usb-charging-hub"
 				(path "/04e54dfe-f06f-40ed-b860-573373578cb0/8b94d9f0-b4ab-48ff-a9ac-e3216038869f"
-					(reference "#PWR066")
+					(reference "#PWR049")
 					(unit 1)
 				)
@@
 		(on_board yes)
 		(dnp no)
-		(property "Reference" "C15"
+		(property "Reference" "C22"
 			(at 146.05 46.99 0)
 			(effects
@@
 			(project "usb-charging-hub"
 				(path "/04e54dfe-f06f-40ed-b860-573373578cb0/8b94d9f0-b4ab-48ff-a9ac-e3216038869f"
-					(reference "C15")
+					(reference "C22")
 					(unit 1)
 				)
@@
 		(dnp no)
 		(fields_autoplaced yes)
-		(property "Reference" "#PWR060"
+		(property "Reference" "#PWR043"
 			(at 80.01 36.83 0)
 			(effects
@@
 			(project "usb-charging-hub"
 				(path "/04e54dfe-f06f-40ed-b860-573373578cb0/8b94d9f0-b4ab-48ff-a9ac-e3216038869f"
-					(reference "#PWR060")
-					(unit 1)
-				)
+					(reference "#PWR043")
+					(unit 1)
+				)

Commit message: finished schematic yay!! now onto pcb routing :fire:
Parts:
- U5: symbol EasyEDA:XXL1509-5.0 -> easyeda2kicad:XXL1509-5.0
Changed lines of the file:
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@@
-	)
-	(junction
-		(at 76.2 52.07)
-		(diameter 0)
-		(color 0 0 0 0)
-	)
-	(junction
-		(at 76.2 49.53)
-		(diameter 0)
-		(color 0 0 0 0)
 	)
 	(junction
@@
 	)
 	(junction
-		(at 76.2 46.99)
-		(diameter 0)
-		(color 0 0 0 0)
-	)
-	(junction
 		(at 69.85 52.07)
 		(diameter 0)
@@
 	(wire
 		(pts
-			(xy 76.2 44.45) (xy 76.2 46.99)
-		)
-		(stroke
-			(width 0)
-			(type default)
-		)
-	)
-	(wire
-		(pts
 			(xy 168.91 44.45) (xy 168.91 46.99)
 		)
@@
 	(wire
 		(pts
-			(xy 76.2 52.07) (xy 76.2 49.53)
-		)
-		(stroke
-			(width 0)
-			(type default)
-		)
-	)
-	(wire
-		(pts
 			(xy 99.06 44.45) (xy 104.14 44.45)
 		)
@@
 		(pts
 			(xy 121.92 44.45) (xy 127 44.45)
-		)
-		(stroke
-			(width 0)
-			(type default)
-		)
-	)
-	(wire
-		(pts
-			(xy 76.2 49.53) (xy 76.2 46.99)
 		)
 		(stroke
@@
 	)
 	(symbol
-		(lib_id "EasyEDA:XXL1509-5.0")
+		(lib_id "easyeda2kicad:XXL1509-5.0")
 		(at 87.63 44.45 0)
 		(mirror y)
