File: neopixels.kicad_sch (KiCad schematic)
At the start: 4 parts, among them J14 Conn_01x03_Pin, J15 Conn_01x02_Pin, J3 Conn_01x03_Pin

Commit message: finished schematic yay!! now onto pcb routing :fire:
Parts:
- removed J14, J3: Conn_01x03_Pin, symbol Connector:Conn_01x03_Pin
- removed J15: Conn_01x02_Pin, symbol Connector:Conn_01x02_Pin
- removed LED20: SK6812MINI-E_C5149201, easyeda2kicad:LED-SMD_L3.2-W2.8-LS5.9_SK6812MINI-E, symbol EasyEDA:SK6812MINI-E_C5149201
- added LED1, LED10, LED11, LED12, LED13, LED14, LED15, LED16, LED17, LED18, LED19, LED2, LED20, LED3, LED4, LED5, LED6, LED7, LED8, LED9: SK6812MINI-E_C5149201, easyeda2kicad:LED-SMD_L3.2-W2.8-LS5.9_SK6812MINI-E, symbol easyeda2kicad:SK6812MINI-E_C5149201
- added TP1: TestPoint, TestPoint:TestPoint_Pad_D2.5mm, symbol Connector:TestPoint
Connections:
- net +5V: now also LED1.1 (VDD), LED10.1 (VDD), LED11.1 (VDD), LED12.1 (VDD), LED13.1 (VDD), LED14.1 (VDD), LED15.1 (VDD), LED16.1 (VDD), LED17.1 (VDD), LED18.1 (VDD), LED19.1 (VDD), LED2.1 (VDD), LED20.1 (VDD), LED3.1 (VDD), LED4.1 (VDD), LED5.1 (VDD), LED6.1 (VDD), LED7.1 (VDD), LED8.1 (VDD), LED9.1 (VDD)
- net GND: now also LED1.3 (GND), LED10.3 (GND), LED11.3 (GND), LED12.3 (GND), LED13.3 (GND), LED14.3 (GND), LED15.3 (GND), LED16.3 (GND), LED17.3 (GND), LED18.3 (GND), LED19.3 (GND), LED2.3 (GND), LED20.3 (GND), LED3.3 (GND), LED4.3 (GND), LED5.3 (GND), LED6.3 (GND), LED7.3 (GND), LED8.3 (GND), LED9.3 (GND)
- new net: LED12.2 (DOUT), LED13.4 (DIN)
- new net: LED11.2 (DOUT), LED12.4 (DIN)
- new net: LED4.2 (DOUT), LED5.4 (DIN)
- new net: LED3.2 (DOUT), LED4.4 (DIN)
- new net: LED15.2 (DOUT), LED16.4 (DIN)
- new net: LED14.2 (DOUT), LED15.4 (DIN)
- new net: LED8.2 (DOUT), LED9.4 (DIN)
- new net: LED7.2 (DOUT), LED8.4 (DIN)
- new net: LED18.2 (DOUT), LED19.4 (DIN)
- new net: LED17.2 (DOUT), LED18.4 (DIN)
- new net: LED20.2 (DOUT), TP1.1
- new net: LED2.2 (DOUT), LED3.4 (DIN)
- new net: LED13.2 (DOUT), LED14.4 (DIN)
- new net: LED1.2 (DOUT), LED2.4 (DIN)
- new net: LED10.2 (DOUT), LED11.4 (DIN)
- new net: LED6.2 (DOUT), LED7.4 (DIN)
- new net: LED5.2 (DOUT), LED6.4 (DIN)
- new net: LED10.4 (DIN), LED9.2 (DOUT)
- new net: LED19.2 (DOUT), LED20.4 (DIN)
- new net: LED16.2 (DOUT), LED17.4 (DIN)
- new net Pixels: LED1.4 (DIN)

Commit message: made huge progress today, finished wiring up the rp2040, finished one usb a and usb c layout :fire::fire::fire:
Parts:
- LED1, LED10, LED11, LED12, LED13, LED14, LED15, LED16, LED17, LED18, LED19, LED2, LED20, LED3, LED4, LED5, LED6, LED7, LED8, LED9: footprint easyeda2kicad:LED-SMD_L3.2-W2.8-LS5.9_SK6812MINI-E -> Keebio-Parts:SK6812-MINI-E
Changed lines of the file:
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@@
 			)
 		)
-		(property "Footprint" "easyeda2kicad:LED-SMD_L3.2-W2.8-LS5.9_SK6812MINI-E"
+		(property "Footprint" "Keebio-Parts:SK6812-MINI-E"
 			(at 116.84 93.98 0)
 			(effects
@@
 			)
 		)
-		(property "Footprint" "easyeda2kicad:LED-SMD_L3.2-W2.8-LS5.9_SK6812MINI-E"
+		(property "Footprint" "Keebio-Parts:SK6812-MINI-E"
 			(at 195.58 50.8 0)
 			(effects
@@
 			)
 		)
-		(property "Footprint" "easyeda2kicad:LED-SMD_L3.2-W2.8-LS5.9_SK6812MINI-E"
+		(property "Footprint" "Keebio-Parts:SK6812-MINI-E"
 			(at 234.95 93.98 0)
 			(effects
@@
 			)
 		)
-		(property "Footprint" "easyeda2kicad:LED-SMD_L3.2-W2.8-LS5.9_SK6812MINI-E"
+		(property "Footprint" "Keebio-Parts:SK6812-MINI-E"
 			(at 156.21 72.39 0)
 			(effects
@@
 			)
 		)
-		(property "Footprint" "easyeda2kicad:LED-SMD_L3.2-W2.8-LS5.9_SK6812MINI-E"
+		(property "Footprint" "Keebio-Parts:SK6812-MINI-E"
 			(at 156.21 115.57 0)
 			(effects
@@
 			)
 		)
-		(property "Footprint" "easyeda2kicad:LED-SMD_L3.2-W2.8-LS5.9_SK6812MINI-E"
+		(property "Footprint" "Keebio-Parts:SK6812-MINI-E"
 			(at 156.21 50.8 0)
 			(effects
@@
 			)
 		)
-		(property "Footprint" "easyeda2kicad:LED-SMD_L3.2-W2.8-LS5.9_SK6812MINI-E"
+		(property "Footprint" "Keebio-Parts:SK6812-MINI-E"
 			(at 156.21 93.98 0)
 			(effects
@@
 			)
 		)
-		(property "Footprint" "easyeda2kicad:LED-SMD_L3.2-W2.8-LS5.9_SK6812MINI-E"
+		(property "Footprint" "Keebio-Parts:SK6812-MINI-E"
 			(at 195.58 93.98 0)
 			(effects
@@
 			)
 		)
-		(property "Footprint" "easyeda2kicad:LED-SMD_L3.2-W2.8-LS5.9_SK6812MINI-E"
+		(property "Footprint" "Keebio-Parts:SK6812-MINI-E"
 			(at 77.47 50.8 0)
 			(effects
@@
 			)
 		)
-		(property "Footprint" "easyeda2kicad:LED-SMD_L3.2-W2.8-LS5.9_SK6812MINI-E"
+		(property "Footprint" "Keebio-Parts:SK6812-MINI-E"
 			(at 77.47 93.98 0)
 			(effects
@@
 			)
 		)
-		(property "Footprint" "easyeda2kicad:LED-SMD_L3.2-W2.8-LS5.9_SK6812MINI-E"
+		(property "Footprint" "Keebio-Parts:SK6812-MINI-E"
 			(at 77.47 72.39 0)
 			(effects
@@
 			)
 		)
-		(property "Footprint" "easyeda2kicad:LED-SMD_L3.2-W2.8-LS5.9_SK6812MINI-E"
+		(property "Footprint" "Keebio-Parts:SK6812-MINI-E"
 			(at 116.84 72.39 0)
 			(effects
@@
 			)
 		)
-		(property "Footprint" "easyeda2kicad:LED-SMD_L3.2-W2.8-LS5.9_SK6812MINI-E"
+		(property "Footprint" "Keebio-Parts:SK6812-MINI-E"
 			(at 234.95 72.39 0)
 			(effects
@@
 			)
 		)
-		(property "Footprint" "easyeda2kicad:LED-SMD_L3.2-W2.8-LS5.9_SK6812MINI-E"
+		(property "Footprint" "Keebio-Parts:SK6812-MINI-E"
 			(at 116.84 50.8 0)
 			(effects
@@
 			)
 		)
-		(property "Footprint" "easyeda2kicad:LED-SMD_L3.2-W2.8-LS5.9_SK6812MINI-E"
+		(property "Footprint" "Keebio-Parts:SK6812-MINI-E"
 			(at 234.95 115.57 0)
 			(effects
@@
 			)
 		)
-		(property "Footprint" "easyeda2kicad:LED-SMD_L3.2-W2.8-LS5.9_SK6812MINI-E"
+		(property "Footprint" "Keebio-Parts:SK6812-MINI-E"
 			(at 195.58 72.39 0)
 			(effects
@@
 			)
 		)
-		(property "Footprint" "easyeda2kicad:LED-SMD_L3.2-W2.8-LS5.9_SK6812MINI-E"
+		(property "Footprint" "Keebio-Parts:SK6812-MINI-E"
 			(at 234.95 50.8 0)
 			(effects
@@
 			)
 		)
-		(property "Footprint" "easyeda2kicad:LED-SMD_L3.2-W2.8-LS5.9_SK6812MINI-E"
+		(property "Footprint" "Keebio-Parts:SK6812-MINI-E"
 			(at 195.58 115.57 0)
 			(effects
@@
 			)
 		)
-		(property "Footprint" "easyeda2kicad:LED-SMD_L3.2-W2.8-LS5.9_SK6812MINI-E"
+		(property "Footprint" "Keebio-Parts:SK6812-MINI-E"
 			(at 77.47 115.57 0)
 			(effects
@@
 			)
 		)
-		(property "Footprint" "easyeda2kicad:LED-SMD_L3.2-W2.8-LS5.9_SK6812MINI-E"
+		(property "Footprint" "Keebio-Parts:SK6812-MINI-E"
 			(at 116.84 115.57 0)
 			(effects

Commit message: holyyy i actually finished all of the bare pcb adding lots of art soon:tm:
Signed-off-by: Toby Cm <toby@vsus.app>
Connections:
- net at TP1.1: now also LED5.2 (DOUT), LED6.4 (DIN); no longer LED20.2 (DOUT)
Other:
- moved on the sheet: TP1
Changed lines of the file:
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@@
 	(generator_version "9.0")
 	(paper "A4")
+	(junction
+		(at 247.65 50.8)
+		(diameter 0)
+		(color 0 0 0 0)
+	)
 	(wire
 		(pts
@@
 	(wire
 		(pts
-			(xy 245.11 107.95) (xy 260.35 107.95)
-		)
-		(stroke
-			(width 0)
-			(type default)
-		)
-	)
-	(wire
-		(pts
 			(xy 96.52 43.18) (xy 96.52 40.64)
 		)
@@
 		(exclude_from_sim no)
 		(in_bom yes)
-		(on_board yes)
+		(on_board no)
 		(dnp no)
 		(fields_autoplaced yes)
@@
 		(exclude_from_sim no)
 		(in_bom yes)
-		(on_board yes)
+		(on_board no)
 		(dnp no)
 		(fields_autoplaced yes)
@@
 		(exclude_from_sim no)
 		(in_bom yes)
-		(on_board yes)
+		(on_board no)
 		(dnp no)
 		(fields_autoplaced yes)
@@
 		(exclude_from_sim no)
 		(in_bom yes)
-		(on_board yes)
+		(on_board no)
 		(dnp no)
 		(fields_autoplaced yes)
@@
 	(symbol
 		(lib_id "Connector:TestPoint")
-		(at 260.35 107.95 0)
+		(at 247.65 50.8 270)
 		(unit 1)
 		(exclude_from_sim no)
@@
 		(fields_autoplaced yes)
 		(property "Reference" "TP1"
-			(at 262.89 102.7429 0)
+			(at 252.73 48.8949 90)
 			(effects
 				(font
@@
 		)
 		(property "Value" "TestPoint"
-			(at 262.89 106.5529 0)
+			(at 252.73 52.7049 90)
 			(effects
 				(font
@@
 		)
 		(property "Footprint" "TestPoint:TestPoint_Pad_D2.5mm"
-			(at 265.43 107.95 0)
+			(at 247.65 55.88 0)
 			(effects
 				(font
@@
 		)
 		(property "Datasheet" "~"
-			(at 265.43 107.95 0)
+			(at 247.65 55.88 0)
 			(effects
 				(font
@@
 		)
 		(property "Description" "test point"
-			(at 260.35 107.95 0)
+			(at 247.65 50.8 0)
 			(effects
 				(font
@@
 		)
 		(instances
-			(project ""
+			(project "usb-charging-hub"
 				(path "/04e54dfe-f06f-40ed-b860-573373578cb0/4f7e225d-95a1-444f-b5b1-f7e4555fb7c8"
 					(reference "TP1")
@@
 		(exclude_from_sim no)
 		(in_bom yes)
-		(on_board yes)
+		(on_board no)
 		(dnp no)
 		(fields_autoplaced yes)
@@
 		(exclude_from_sim no)
 		(in_bom yes)
-		(on_board yes)
+		(on_board no)
 		(dnp no)
 		(fields_autoplaced yes)
@@
 		(exclude_from_sim no)
 		(in_bom yes)
-		(on_board yes)
+		(on_board no)
 		(dnp no)
 		(fields_autoplaced yes)
@@
 		(exclude_from_sim no)
 		(in_bom yes)
-		(on_board yes)
+		(on_board no)
 		(dnp no)
 		(fields_autoplaced yes)
@@
 		(exclude_from_sim no)
 		(in_bom yes)
-		(on_board yes)
+		(on_board no)
 		(dnp no)
 		(fields_autoplaced yes)
@@
 		(exclude_from_sim no)
 		(in_bom yes)
-		(on_board yes)
+		(on_board no)
 		(dnp no)
 		(fields_autoplaced yes)
@@
 		(exclude_from_sim no)
 		(in_bom yes)
-		(on_board yes)
+		(on_board no)
 		(dnp no)
 		(fields_autoplaced yes)
@@
 		(exclude_from_sim no)
 		(in_bom yes)
-		(on_board yes)
+		(on_board no)
 		(dnp no)
 		(fields_autoplaced yes)
@@
 		(exclude_from_sim no)
 		(in_bom yes)
-		(on_board yes)
+		(on_board no)
 		(dnp no)
 		(fields_autoplaced yes)
@@
 		(exclude_from_sim no)
 		(in_bom yes)
-		(on_board yes)
+		(on_board no)
 		(dnp no)
 		(fields_autoplaced yes)
@@
 		(exclude_from_sim no)
 		(in_bom yes)
-		(on_board yes)
+		(on_board no)
 		(dnp no)
 		(fields_autoplaced yes)
