File: rp2040.kicad_sch (KiCad schematic)
At the start: 43 parts, among them J3 TYPE-C 16PLT-H10.0, SW1 TS24CA, SW2 Latching, SW3 TS24CA, SW4 TS24CA, U1 W25Q32JVSS, U2 ABM8-272-T3_C20625731, U3 RP2040

Commit message: finished schematic yay!! now onto pcb routing :fire:
Parts:
- removed J3: TYPE-C 16PLT-H10.0, easyeda2kicad:TYPE-C-SMD_USB4120-03-C, symbol EasyEDA:TYPE-C16PLT-H10.0
- removed R7: 470, Resistor_SMD:R_0402_1005Metric_Pad0.72x0.64mm_HandSolder, symbol Device:R_Small
- removed R8: 10k, Resistor_SMD:R_0402_1005Metric_Pad0.72x0.64mm_HandSolder, symbol Device:R_Small
- added J35: GT-USB-7010ASV, easyeda2kicad:USB-C-SMD_G-SWITCH_GT-USB-7010ASV, symbol easyeda2kicad:GT-USB-7010ASV
- added R107: 470, Resistor_SMD:R_0402_1005Metric_Pad0.72x0.64mm_HandSolder, symbol Device:R_Small
- added R108: 10k, Resistor_SMD:R_0402_1005Metric_Pad0.72x0.64mm_HandSolder, symbol Device:R_Small
Connections:
- net GND: now also J35.1 (SHELL), J35.2 (SHELL), J35.3 (SHELL), J35.4 (SHELL), J35.A1B12 (GND), J35.B1A12 (GND), R108.2
- net VBUS: now also J35.A4B9 (VBUS), J35.B4A9 (VBUS)
- net at SW1.4: now also U3.30 (GPIO19); no longer U3.29 (GPIO18)
- net at R3.1: now also J35.B5 (CC2)
- net at R5.1: now also J35.A7 (DN1), J35.B7 (DN2)
- net at R4.1: now also J35.A6 (DP1), J35.B6 (DP2)
- net at R2.1: now also J35.A5 (CC1)
- net at SW2.1: now also U3.29 (GPIO18); no longer U3.30 (GPIO19)
- net GPIO15: no longer names the net of U3.18 (GPIO15)
- net GPIO15: now also R107.1, R108.1
- net GPIO16 renamed SDA
- net GPIO17 renamed SCL
- new net Pixels: R107.2
Other:
- moved on the sheet: SW1, SW2

Commit message: made huge progress today, finished wiring up the rp2040, finished one usb a and usb c layout :fire::fire::fire:
Connections:
- net USB_R_D-: now reaches J35.A7 (DN1), J35.B7 (DN2), R5.1
- net USB_D-: now reaches R5.2, U3.46 (USB_DM)
- net USB_R_D+: now reaches J35.A6 (DP1), J35.B6 (DP2), R4.1
- net USB_D+: now reaches R4.2, U3.47 (USB_DP)
Changed lines of the file:
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@@
 			"AAAAAAAAAAAAAAAAAAAAAAAAAAAAAAAAAAAAAAAAAAAAAAAAAAAAAAAAAAAAAAAAAAAAAAAAAAAA"
 			"AAAAAAAAAAAAAAAAAAAAAAAAAAAAAAAAAAAAAAAAAAAAAAAAAAAAAAAAAAAAAAAAAAAAAAAAAAAA"
-			"AAAAAAAAAAAAAAAAAAAAAAAAAAAAAAAAAAAAAAAAAAAAAAAAAAAAAAAAAAAAAA=="
+			"AAAAAAAAAAAAAAAAAAAAAAAAAAAAAAAAAAAAAAAAAAAAAAAAAAAAAAAAAAAAAAAAAAAAAAAAAAAA"
+			"AAAAAAAAAAAAAAAAAAAAAAAAAAAAAAAAAAAAAAAAAAAAAAAAAAAAAAAAAAAAAAAAAAAAAAAAAAAA"
+			"AAAAAAAAAAAAAAAAAAAAAAAAAAAAAAAAAAAAAAAAAAAAAAAAAAAAAAAAAAAAAAAAAAAAAAAAAAAA"
+			"AAAAAAAAAAAAAAAAAAAAAAAAAAAAAAAAAAAAAAAAAAAAAAAAAAAAAAAAAAAAAAAAAAAAAAAAAAAA"
+			"AAAAAAAAAAAAAAAAAAAAAAAAAAAAAAAAAAAAAAAAAAAAAAAAAAAAAAAAAAAAAAAAAAAAAAAAAAAA"
+			"AAAAAAAAAAAAAAAAAAAAAAAAAAAAAAAAAAAAAAAAAAAAAAAAAAAAAAAAAAAAAAAAAAAAAAAAAAAA"
+			"AAAAAAAAAAAAAAAAAAAAAAAAAAAAAAAAAAAAAAAAAAAAAAAAAAAAAAAAAAAAAAAAAAAAAAAAAAAA"
+			"AAAAAAAAAAAAAAAAAAAAAAAAAAAAAAAAAAAAAAAAAAAAAAAAAAAAAAAAAAAAAAAAAAAAAAAAAAAA"
+			"AAAAAAAAAAAAAAAAAAAAAAAAAAAAAAAAAAAAAAAAAAAAAAAAAAAAAAAAAAAAAAAAAAAAAAAAAAAA"
+			"AAAAAAAAAAAAAAAAAAAAAAAAAAAAAAAAAAAAAAAAAAAAAAAAAAAAAAAAAAAAAAAAAAAAAAAAAAAA"
+			"AAAAAAAAAAAAAAAAAAAAAAAAAAAAAAAAAAAAAAAAAAAAAAAAAAAAAAAAAAAAAAAAAAAAAAAAAAAA"
+			"AAAAAAAAAAAAAAAAAAAAAAAAAAAAAAAAAAAAAAAAAAAAAAAAAAAAAAAAAAAAAAAAAAAAAAAAAAAA"
+			"AAAAAAAAAAAAAAAAAAAAAAAAAAAAAAAAAAAAAAAAAAAAAAAAAAAAAAAAAAAAAAAAAAAAAAAAAAAA"
+			"AAAAAAAAAAAAAAAAAAAAAAAAAAAAAAAAAAAAAAAAAAAAAAAAAAAAAAAAAAAAAAAAAAAAAAAAAAAA"
+			"AAAAAAAAAAAAAAAAAAAAAAAAAAAAAAAAAAAAAAAAAAAAAAAAAAAAAAAAAAAAAAAAAAAAAAAAAAAA"
+			"AAAAAAAAAAAAAAAAAAAAAAAAAAAAAAAAAAAAAAAAAAAAAAAAAAAAAAAAAAAAAAAAAAAAAAAAAAAA"
+			"AAAAAAAAAAAAAAAAAAAAAAAAAAAAAAAAAAAAAAAAAAAAAAAAAAAAAAAAAAAAAAAAAAAAAAAAAAAA"
+			"AAAAAAAAAAAAAAAAAAAAAAAAAAAAAAAAAAAAAAAAAAAAAAAAAAAAAAAAAAAAAAAAAAAAAAAAAAAA"
+			"AAAAAAAAAAAAAAAAAAAAAAAAAAAAAAAAAAAAAAAAAAAAAAAAAAAAAAAAAAAAAAAAAAAAAAAAAAAA"
+			"AAAAAAAAAAAAAAAAAAAAAAAAAAAAAAAAAAAAAAAAAAAAAAAAAAAAAAAAAAAAAAAAAAAAAAAAAAAA"
+			"AAAAAAAAAAAAAAAAAAAAAAAAAAAAAAAAAAAAAAAAAAAAAAAAAAAAAAAAAAAAAAAAAAAAAAAAAAAA"
+			"AAAAAAAAAAAAAAAAAAAAAAAAAAAAAAAAAAAAAAAAAAAAAAAAAAAAAAAAAAAAAAAAAAAAAAAAAAAA"
+			"AAAAAAAAAAAAAAAAAAAAAAAAAAAAAAAAAAAAAAAAAAAAAAAAAAAAAAAAAAAAAAAAAAAAAAAAAAAA"
+			"AAAAAAAAAAAAAAAAAAAAAAAAAAAAAAAAAAAAAAAAAAAAAAAAAAAAAAAAAAAAAAAAAAAAAAAAAAAA"
+			"AAAAAAAAAAAAAAAAAAAAAAAAAAAAAAAAAAAAAAAAAAAAAAAAAAAAAAAAAAAAAAAAAAAAAAAAAAAA"
+			"AAAAAAAAAAAAAAAAAAAAAAAAAAAAAAAAAAAAAAAAAAAAAAAAAAAAAAAAAAAAAAAAAAAAAAAAAAAA"
+			"AAAAAAAAAAAAAAAAAAAAAAAAAAAAAAAAAAAAAAAAAAAAAAAAAAAAAAAAAAAAAAAAAAAAAAAAAAAA"
+			"AAAAAAAAAAAAAAAAAAAAAAAAAAAAAAAAAAAAAAAAAAAAAAAAAAAAAAAAAAAAAAAAAAAAAAAAAAAA"
+			"AAAAAAAAAAAAAAAAAAAAAAAAAAAAAAAAAAAAAAAAAAAAAAAAAAAAAAAAAAAAAAAAAAAAAAAAAAAA"
+			"AAAAAAAAAAAAAAAAAAAAAAAAAAAAAAAAAAAAAAAAAAAAAAAAAAAAAAAAAAAAAAAAAAAAAAAAAAAA"
+			"AAAAAAAAAAAAAAAAAAAAAAAAAAAAAAAAAAAAAAAAAAAAAAAAAAAAAAAAAAAAAAAAAAAAAAAAAAAA"
+			"AAAAAAAAAAAAAAAAAAAAAAAAAAAAAAAAAAAAAAAAAAAAAAAAAAAAAAAAAAAAAAAAAAAAAAAAAAAA"
+			"AAAAAAAAAAAAAAAAAAAAAAAAAAAAAAAAAAAAAAAAAAAAAAAAAAAAAAAAAAAAAAAAAAAAAAAAAAAA"
+			"AAAAAAAAAAAAAAAAAAAAAAAAAAAAAAAAAAAAAAAAAAAAAAAAAAAAAAAAAAAAAAAAAAAAAAAAAAAA"
+			"AAAAAAAAAAAAAAAAAAAAAAAAAAAAAAAAAAAAAAAAAAAAAAAAAAAAAAAAAAAAAAAAAAAAAAAAAAAA"
+			"AAAAAAAAAAAAAAAAAAAAAAAAAAAAAAAAAAAAAAAAAAAAAAAAAAAAAAAAAAAAAAAAAAAAAAAAAAAA"
+			"AAAAAAAAAAAAAAAAAAAAAAAAAAAAAAAAAAAAAAAAAAAAAAAAAAAAAAAAAAAAAAAAAAAAAAAAAAAA"
+			"AAAAAAAAAAAAAAAAAAAAAAAAAAAAAAAAAAAAAAAAAAAAAAAAAAAAAAAAAAAAAAAAAAAAAAAAAAAA"
+			"AAAAAAAAAAAAAAAAAAAAAAAAAAAAAAAAAAAAAAAAAAAAAAAAAAAAAAAAAAAAAAAAAAAAAAAAAAAA"
+			"AAAAAAAAAAAAAAAAAAAAAAAAAAAAAAAAAAAAAAAAAAAAAAAAAAAAAAAAAAAAAAAAAAAAAAAAAAAA"
+			"AAAAAAAAAAAAAAAAAAAAAAAAAAAAAAAAAAAAAAAAAAAAAAAAAAAAAAAAAAAAAAAAAAAAAAAAAAAA"
+			"AAAAAAAAAAAAAAAAAAAAAAAAAAAAAAAAAAAAAAAAAAAAAAAAAAAAAAAAAAAAAAAAAAAAAAAAAAAA"
+			"AAAAAAAAAAAAAAAAAAAAAAAAAAAAAAAAAAAAAAAAAAAAAAAAAAAAAAAAAAAAAAAAAAAAAAAAAAAA"
+			"AAAAAAAAAAAAAAAAAAAAAAAAAAAAAAAAAAAAAAAAAAAAAAAAAAAAAAAAAAAAAAAAAAAAAAAAAAAA"
+			"AAAAAAAAAAAAAAAAAAAAAAAAAAAAAAAAAAAAAAAAAAAAAAAAAAAAAAAAAAAAAAAAAAAAAAAAAAAA"
+			"AAAAAAAAAAAAAAAAAAAAAAAAAAAAAAAAAAAAAAAAAAAAAAAAAAAAAAAAAAAAAAAAAAAAAAAAAAAA"
+			"AAAAAAAAAAAAAAAAAAAAAAAAAAAAAAAAAAAAAAAAAAAAAAAAAAAAAAAAAAAAAAAAAAAAAAAAAAAA"
+			"AAAAAAAAAAAAAAAAAAAAAAAAAAAAAAAAAAAAAAAAAAAAAAAAAAAAAAAAAAAAAAAAAAAAAAAAAAAA"
+			"AAAAAAAAAAAAAAAAAAAAAAAAAAAAAAAAAAAAAAAAAAAAAAAAAAAAAAAAAAAAAAAAAAAAAAAAAAAA"
+			"AAAAAAAAAAAAAAAAAAAAAAAAAAAAAAAAAAAAAAAAAAAAAAAAAAAAAAAAAAAAAAAAAAAAAAAAAAAA"
+			"AAAAAAAAAAAAAAAAAAAAAAAAAAAAAAAAAAAAAAAAAAAAAAAAAAAAAAAAAAAAAAAAAAAAAAAAAAAA"
+			"AAAAAAAAAAAAAAAAAAAAAAAAAAAAAAAAAAAAAAAAAAAAAAAAAAAAAAAAAAAAAAAAAAAAAAAAAAAA"
+			"AAAAAAAAAAAAAAAAAAAAAAAAAAAAAAAAAAAAAAAAAAAAAAAAAAAAAAAAAAAAAAAAAAAAAAAAAAAA"
+			"AAAAAAAAAAAAAAAAAAAAAAAAAAAAAAAAAAAAAAAAAAAAAAAAAAAAAAAAAAAAAAAAAAAAAAAAAAAA"
+			"AAAAAAAAAAAAAAAAAAAAAAAAAAAAAAAAAAAAAAAAAAAAAAAAAAAAAAAAAAAAAADQed9bnFsAADCb"
+			"alycWwAABgAAAAAAAABgtINbnFsAAMDa7VucWwAA4EwkWpxbAACwF6danFsAAHD9pFqcWwAAAAAA"
+			"AAAAAADgBnxanFsAAAAAAAAAAAAAcHvfW5xbAAAQjmpcnFsAAAAAAAAAAAAAYLWDW5xbAABQ2+1b"
+			"nFsAAKBNJFqcWwAAsBinWpxbAABw/qRanFsAAAAAAAAAAAAAcAd8WpxbAAAAAAAAAAAAAGB631uc"
+			"WwAAYIFqXJxbAAAgtLhanFsAAIC2g1ucWwAAoLHnW5xbAAAwTiRanFsAANAZp1qcWwAA8AClWpxb"
+			"AAAAAAAAAAAAAAAIfFqcWwAAAAAAAAAAAADwet9bnFsAACCCalycWwAA4LS4WpxbAACQvINbnFsA"
+			"AOAn6lucWwAAEP0jWpxbAABQMadanFsAAIADpVqcWwAAAAAAAAAAAADgCHxanFsAAAAAAAAAAAAA"
+			"MHvfW5xbAACAQWpcnFsAALC2uFqcWwAA4MGDW5xbAADgIelbnFsAAMB/JFqcWwAAoDKnWpxbAABg"
+			"BaVanFsAAAAAAAAAAAAAcAl8WpxbAAAAAAAAAAAAAFB831ucWwAA4JNqXJxbAABAt7hanFsAAJDD"
+			"g1ucWwAAEC/nW5xbAACwzyNanFsAADAyp1qcWwAAIAalWpxbAAAAAAAAAAAAAFARfFqcWwAAAAAA"
+			"AAAAAADgfN9bnFsAALCUalycWwAAILi4WpxbAAAgw4NbnFsAAPAs51ucWwAA0DskWpxbAADwNada"
+			"nFsAAOAGpVqcWwAAAAAAAAAAAACwk2NanFsAAAAAAAAAAAAAoH3fW5xbAACgnGpcnFsAACC5uFqc"
+			"WwAAwMWDW5xbAAAAkudbnFsAAGA8JFqcWwAA8DanWpxbAAAwaaxanFsAACAWc1ycWwAAEFR8Wpxb"
+			"AAAAAAAAAAAAADB+31ucWwAAgJ1qXJxbAADAurhanFsAAMDGg1ucWwAAAAAAAAAAAABgDCRanFsA"
+			"AHAlp1qcWwAAUGqsWpxbAABwVhFcnFsAAPCTY1qcWwAAAAAAAAAAAAAAAAAAAAAAANCNalycWwAA"
+			"MJ2lWpxbAADgx4NbnFsAAHA06FucWwAAgPYjWpxbAACgOadanFsAABBqrFqcWwAAsBjdW5xbAAAA"
+			"AAAAAAAAABBEAAAAAAAAwILfW5xbAADAqmpcnFsAABDBuFqcWwAA8M2DW5xbAADgfsFbnFsAAMD2"
+			"I1qcWwAAUDunWpxbAABgbKxanFsAADBDMlucWwAAAAp8WpxbAAAAAAAAAAAAAAAAAAAAAAAAgKtq"
+			"XJxbAADQwbhanFsAAEDTg1ucWwAAgH7uW5xbAACwXCRanFsAAFBLp1qcWwAAYA=="
 		)
 	)
+	(label "USB_D+"
+		(at 165.1 73.66 0)
+		(effects
+			(font
+				(size 1.27 1.27)
+			)
+			(justify left bottom)
+		)
+	)
+	(label "USB_R_D+"
+		(at 139.7083 78.74 0)
+		(effects
+			(font
+				(size 1.27 1.27)
+			)
+			(justify left bottom)
+		)
+	)
+	(label "USB_R_D-"
+		(at 139.7 73.66 0)
+		(effects
+			(font
+				(size 1.27 1.27)
+			)
+			(justify left bottom)
+		)
+	)
+	(label "USB_D-"
+		(at 165.1 76.2 0)
+		(effects
+			(font
+				(size 1.27 1.27)
+			)
+			(justify left bottom)
+		)
+	)
