File: usb-charging-hub.kicad_sch (KiCad schematic)
At the start: 3 parts

Commit message: updated journal, pin headers footprint, etc. added labels to rp2350b, finished pcb routing. time to start on other modules yay
Signed-off-by: Toby Cm <toby@vsus.app>
Parts:
- added C1, C2: 50V,1000uF, Capacitor_THT:CP_Radial_D13.0mm_P7.50mm, symbol Device:C_Polarized_Small
- added J1, J2: Conn_01x01_Pin, MountingHole:MountingHole_4.3x6.2mm_M4_Pad_Via, symbol Connector:Conn_01x01_Pin
Connections:
- net GND: now also C2.2, J2.1 (Pin_1)
- net VDC: now also C1.1, J1.1 (Pin_1)
- new net: C1.2, C2.1
Other:
- removed sheet Neopixel

Commit message: no more modules, its gonna work first try :fire: i love infineon and their ICs so much
Signed-off-by: Toby Cm <toby@vsus.app>
Other:
- sheet USB A renamed USB 1
- removed sheet USB C
- removed sheet rp2350b
- added sheet USB 2 (usb2.kicad_sch)
- added sheet USB 3 (usb3.kicad_sch)
- added sheet USB 4 (usb4.kicad_sch)
- added sheet USB 5 (usb5.kicad_sch)
- added sheet rp2040 (rp2040.kicad_sch)
- sheet USB 1: file usba.kicad_sch -> usb1.kicad_sch
- note removed: "USB A Ports"
Changed lines of the file:
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@@
 		(company "DaCloud")
-	)
-	(text "USB A Ports"
-		(exclude_from_sim no)
-		(at 211.582 161.544 0)
-		(effects
-			(font
-				(size 3.81 3.81)
-			)
-		)
 	)
 	(text "power led\n"
@@
 		)
 	)
-	(polyline
-		(pts
-			(xy 191.77 12.7) (xy 191.77 165.1)
-		)
-		(stroke
-			(width 0)
-			(type default)
-		)
-	)
 	(symbol
 		(lib_id "Jumper:SolderJumper_2_Bridged")
@@
 	)
 	(sheet
+		(at 124.46 101.6)
+		(size 12.7 3.81)
+		(exclude_from_sim no)
+		(in_bom yes)
+		(on_board yes)
+		(dnp no)
+		(fields_autoplaced yes)
+		(stroke
+			(width 0.1524)
+			(type solid)
+		)
+		(fill
+			(color 0 0 0 0.0000)
+		)
+		(property "Sheetname" "USB 5"
+			(at 124.46 100.8884 0)
+			(effects
+				(font
+					(size 1.27 1.27)
+				)
+				(justify left bottom)
+			)
+		)
+		(property "Sheetfile" "usb5.kicad_sch"
+			(at 124.46 105.9946 0)
+			(effects
+				(font
+					(size 1.27 1.27)
+				)
+				(justify left top)
+			)
+		)
+		(instances
+			(project "usb-charging-hub"
+				(path "/04e54dfe-f06f-40ed-b860-573373578cb0"
+					(page "9")
+				)
+			)
+		)
+	)
+	(sheet
+		(at 73.66 101.6)
+		(size 12.7 3.81)
+		(exclude_from_sim no)
+		(in_bom yes)
+		(on_board yes)
+		(dnp no)
+		(fields_autoplaced yes)
+		(stroke
+			(width 0.1524)
+			(type solid)
+		)
+		(fill
+			(color 0 0 0 0.0000)
+		)
+		(property "Sheetname" "USB 3"
+			(at 73.66 100.8884 0)
+			(effects
+				(font
+					(size 1.27 1.27)
+				)
+				(justify left bottom)
+			)
+		)
+		(property "Sheetfile" "usb3.kicad_sch"
+			(at 73.66 105.9946 0)
+			(effects
+				(font
+					(size 1.27 1.27)
+				)
+				(justify left top)
+			)
+		)
+		(instances
+			(project "usb-charging-hub"
+				(path "/04e54dfe-f06f-40ed-b860-573373578cb0"
+					(page "7")
+				)
+			)
+		)
+	)
+	(sheet
+		(at 22.86 101.6)
+		(size 12.7 3.81)
+		(exclude_from_sim no)
+		(in_bom yes)
+		(on_board yes)
+		(dnp no)
+		(fields_autoplaced yes)
+		(stroke
+			(width 0.1524)
+			(type solid)
+		)
+		(fill
+			(color 0 0 0 0.0000)
+		)
+		(property "Sheetname" "USB 1"
+			(at 22.86 100.8884 0)
+			(effects
+				(font
+					(size 1.27 1.27)
+				)
+				(justify left bottom)
+			)
+		)
+		(property "Sheetfile" "usb1.kicad_sch"
+			(at 22.86 105.9946 0)
+			(effects
+				(font
+					(size 1.27 1.27)
+				)
+				(justify left top)
+			)
+		)
+		(instances
+			(project "usb-charging-hub"
+				(path "/04e54dfe-f06f-40ed-b860-573373578cb0"
+					(page "5")
+				)
+			)
+		)
+	)
+	(sheet
+		(at 73.66 88.9)
+		(size 12.7 3.81)
+		(exclude_from_sim no)
+		(in_bom yes)
+		(on_board yes)
+		(dnp no)
+		(fields_autoplaced yes)
+		(stroke
+			(width 0.1524)
+			(type solid)
+		)
+		(fill
+			(color 0 0 0 0.0000)
+		)
+		(property "Sheetname" "5V Buck Regulator"
+			(at 73.66 88.1884 0)
+			(effects
+				(font
+					(size 1.27 1.27)
+				)
+				(justify left bottom)
+			)
+		)
+		(property "Sheetfile" "5v.kicad_sch"
+			(at 73.66 93.2946 0)
+			(effects
+				(font
+					(size 1.27 1.27)
+				)
+				(justify left top)
+			)
+		)
+		(instances
+			(project "usb-charging-hub"
+				(path "/04e54dfe-f06f-40ed-b860-573373578cb0"
+					(page "4")
+				)
+			)
+		)
+	)
+	(sheet
+		(at 99.06 101.6)
+		(size 12.7 3.81)
+		(exclude_from_sim no)
+		(in_bom yes)
+		(on_board yes)
+		(dnp no)
+		(fields_autoplaced yes)
+		(stroke
+			(width 0.1524)
+			(type solid)
+		)
+		(fill
+			(color 0 0 0 0.0000)
+		)
+		(property "Sheetname" "USB 4"
+			(at 99.06 100.8884 0)
+			(effects
+				(font
+					(size 1.27 1.27)
+				)
+				(justify left bottom)
+			)
+		)
+		(property "Sheetfile" "usb4.kicad_sch"
+			(at 99.06 105.9946 0)
+			(effects
+				(font
+					(size 1.27 1.27)
+				)
+				(justify left top)
+			)
+		)
+		(instances
+			(project "usb-charging-hub"
+				(path "/04e54dfe-f06f-40ed-b860-573373578cb0"
+					(page "8")
+				)
+			)
+		)
+	)
+	(sheet
 		(at 22.86 88.9)
 		(size 12.7 3.81)
@@
 			(color 0 0 0 0.0000)
 		)
-		(property "Sheetname" "rp2350b"
+		(property "Sheetname" "rp2040"
 			(at 22.86 88.1884 0)
 			(effects
@@
 			)
 		)
-		(property "Sheetfile" "rp2350b.kicad_sch"
+		(property "Sheetfile" "rp2040.kicad_sch"
 			(at 22.86 93.2946 0)
+			(effects
+				(font
+					(size 1.27 1.27)
+				)
+				(justify left top)
+			)
+		)
+		(instances
+			(project "usb-charging-hub"
+				(path "/04e54dfe-f06f-40ed-b860-573373578cb0"
+					(page "2")
+				)
+			)
+		)
+	)
+	(sheet
+		(at 48.26 88.9)
+		(size 12.7 3.81)
+		(exclude_from_sim no)
+		(in_bom yes)
+		(on_board yes)
+		(dnp no)
+		(fields_autoplaced yes)
+		(stroke
+			(width 0.1524)
+			(type solid)
+		)
+		(fill
+			(color 0 0 0 0.0000)
+		)
+		(property "Sheetname" "3.3V Buck Regulator"
+			(at 48.26 88.1884 0)
+			(effects
+				(font
+					(size 1.27 1.27)
+				)
+				(justify left bottom)
+			)
+		)
+		(property "Sheetfile" "3.3v.kicad_sch"
+			(at 48.26 93.2946 0)
 			(effects
 				(font
@@
 			(color 0 0 0 0.0000)
 		)
-		(property "Sheetname" "USB A"
+		(property "Sheetname" "USB 2"
 			(at 48.26 100.8884 0)
 			(effects
@@
 			)
 		)
-		(property "Sheetfile" "usba.kicad_sch"
+		(property "Sheetfile" "usb2.kicad_sch"
 			(at 48.26 105.9946 0)
 			(effects
@@
 				)
 			)
-		)
-	)
-	(sheet
-		(at 22.86 101.6)
-		(size 12.7 3.81)
-		(exclude_from_sim no)
-		(in_bom yes)
-		(on_board yes)
-		(dnp no)
-		(fields_autoplaced yes)
-		(stroke
-			(width 0.1524)
-			(type solid)
-		)
-		(fill
-			(color 0 0 0 0.0000)
-		)
-		(property "Sheetname" "USB C"
-			(at 22.86 100.8884 0)
-			(effects
-				(font
-					(size 1.27 1.27)
-				)
-				(justify left bottom)
-			)
-		)
-		(property "Sheetfile" "usbc.kicad_sch"
-			(at 22.86 105.9946 0)
-			(effects
-				(font
-					(size 1.27 1.27)
-				)
-				(justify left top)
-			)
-		)
-		(instances
-			(project "usb-charging-hub"
-				(path "/04e54dfe-f06f-40ed-b860-573373578cb0"
-					(page "9")
-				)
-			)
-		)
-	)
-	(sheet
-		(at 73.66 88.9)
-		(size 12.7 3.81)
-		(exclude_from_sim no)
-		(in_bom yes)
-		(on_board yes)
-		(dnp no)
-		(fields_autoplaced yes)
-		(stroke
-			(width 0.1524)
-			(type solid)
-		)
-		(fill
-			(color 0 0 0 0.0000)
-		)
-		(property "Sheetname" "5V Buck Regulator"
-			(at 73.66 88.1884 0)
-			(effects
-				(font
-					(size 1.27 1.27)
-				)
-				(justify left bottom)
-			)
-		)
-		(property "Sheetfile" "5v.kicad_sch"
-			(at 73.66 93.2946 0)
-			(effects
-				(font
-					(size 1.27 1.27)
-				)
-				(justify left top)
-			)
-		)
-		(instances
-			(project "usb-charging-hub"
-				(path "/04e54dfe-f06f-40ed-b860-573373578cb0"
-					(page "8")
-				)
-			)
-		)
-	)
-	(sheet
-		(at 48.26 88.9)
-		(size 12.7 3.81)
-		(exclude_from_sim no)
-		(in_bom yes)
-		(on_board yes)
-		(dnp no)
-		(fields_autoplaced yes)
-		(stroke
-			(width 0.1524)
-			(type solid)
-		)
-		(fill
-			(color 0 0 0 0.0000)
-		)
-		(property "Sheetname" "3.3V Buck Regulator"
-			(at 48.26 88.1884 0)
-			(effects
-				(font
-					(size 1.27 1.27)
-				)
-				(justify left bottom)
-			)
-		)
-		(property "Sheetfile" "3.3v.kicad_sch"
-			(at 48.26 93.2946 0)
-			(effects
-				(font
-					(size 1.27 1.27)
-				)
-				(justify left top)
-			)
-		)
-		(instances
-			(project "usb-charging-hub"
-				(path "/04e54dfe-f06f-40ed-b860-573373578cb0"
-					(page "7")
-				)
-			)

Commit message: finished schematic yay!! now onto pcb routing :fire:
Parts:
- removed JP1: SolderJumper_2_Bridged, Jumper:SolderJumper-2_P1.3mm_Bridged_Pad1.0x1.5mm, symbol Jumper:SolderJumper_2_Bridged
- added JP1: SolderJumper_2_Open, Jumper:SolderJumper-2_P1.3mm_Open_RoundedPad1.0x1.5mm, symbol Jumper:SolderJumper_2_Open
Connections:
- net GND: now also C1.2
- net VDC: now also C2.1, JP1.2 (B)
- net at R1.1: now also JP1.1 (A)
Other:
- added sheet Neopixels (neopixels.kicad_sch)
- sheet rp2040 ports: added NEOPIXELS; removed none
- moved on the sheet: C1, C2, J1, J2

Commit message: made huge progress today, finished wiring up the rp2040, finished one usb a and usb c layout :fire::fire::fire:
Other:
- sheet Neopixels ports: added none; removed NEOPIXELS
- sheet rp2040 ports: added none; removed NEOPIXELS
Changed lines of the file:
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@@
-	(wire
-		(pts
-			(xy 38.1 83.82) (xy 97.79 83.82)
-		)
-		(stroke
-			(width 0)
-			(type default)
-		)
-	)
 	(wire
 		(pts
@@
 	(wire
 		(pts
-			(xy 35.56 91.44) (xy 38.1 91.44)
-		)
-		(stroke
-			(width 0)
-			(type default)
-		)
-	)
-	(wire
-		(pts
 			(xy 24.13 25.4) (xy 24.13 27.94)
-		)
-		(stroke
-			(width 0)
-			(type default)
-		)
-	)
-	(wire
-		(pts
-			(xy 97.79 91.44) (xy 100.33 91.44)
 		)
 		(stroke
@@
 		(pts
 			(xy 82.55 25.4) (xy 82.55 27.94)
-		)
-		(stroke
-			(width 0)
-			(type default)
-		)
-	)
-	(wire
-		(pts
-			(xy 38.1 91.44) (xy 38.1 83.82)
-		)
-		(stroke
-			(width 0)
-			(type default)
-		)
-	)
-	(wire
-		(pts
-			(xy 97.79 83.82) (xy 97.79 91.44)
 		)
 		(stroke
@@
 			)
 		)
-		(pin "NEOPIXELS" input
-			(at 100.33 91.44 180)
-			(effects
-				(font
-					(size 1.27 1.27)
-				)
-				(justify left)
-			)
-		)
 		(instances
 			(project "usb-charging-hub"
@@
 			)
 		)
-		(pin "NEOPIXELS" input
-			(at 35.56 91.44 0)
-			(effects
-				(font
-					(size 1.27 1.27)
-				)
-				(justify right)
-			)
-		)

Commit message: holyyy i actually finished all of the bare pcb adding lots of art soon:tm:
Signed-off-by: Toby Cm <toby@vsus.app>
Parts:
- added H1, H2, H3, H4: MountingHole_Pad, MountingHole:MountingHole_4mm_Pad_Via, symbol Mechanical:MountingHole_Pad
Connections:
- net GND: now also H1.1, H2.1, H3.1, H4.1
