File: usb1.kicad_sch (KiCad schematic)
At the start: 67 parts, among them J10 XDUF-0426-081_C18202150, J11 TYPE-C 16PLT-H10.0, J12 Conn_01x04_Pin, J8 TYPE-C 16PLT-H10.0, J9 Conn_01x04_Pin, Q1 PMOS, Q2 PMOS, U10 LS0505EVD22, U11 LS0505EVD22, U12 NDP23511KC, U13 CYPD3175-24LQXQ, U6 XXL1509-5.0, U7 XXL1509-5.0, U8 NDP23511KC, U9 CYPD3175-24LQXQ

Commit message: finished schematic yay!! now onto pcb routing :fire:
Parts:
- J11, J8: symbol EasyEDA:TYPE-C16PLT-H10.0 -> easyeda2kicad:TYPE-C16PLT-H10.0
- U6, U7: symbol EasyEDA:XXL1509-5.0 -> easyeda2kicad:XXL1509-5.0
Connections:
- net SDA: now reaches U9.12 (P2.2)
- net SCL: now reaches U9.13 (P2.3)
- net at L6.1, R32.1: now also U12.5 (SW), U12.6 (SW); no longer U12.5,6 (SW)
- net at L5.1, R23.1: now also U8.5 (SW), U8.6 (SW); no longer U8.5,6 (SW)

Commit message: made huge progress today, finished wiring up the rp2040, finished one usb a and usb c layout :fire::fire::fire:
Parts:
- added SW5, SW6, SW7, SW8: Latching, easyeda2kicad:SW-TH_6P-L8.0-W8.0-P2.50, symbol Switch:SW_Push
- U13, U9: footprint Package_DFN_QFN:QFN-24-1EP_4x4mm_P0.5mm_EP2.75x2.75mm -> Package_DFN_QFN:QFN-24-1EP_4x4mm_P0.5mm_EP2.7x2.7mm_ThermalVias
Connections:
- net D_EN: no longer U13.1 (P1.0)
- net GND: now also SW5.1, SW6.1, SW7.1, SW8.1; no longer J11.0 (EH), J8.0 (EH)
- net SCL: now also U13.13 (P2.3)
- net SDA: now also U13.12 (P2.2)
- net U_EN: no longer U9.1 (P1.0)
- net VDC: now also U12.4 (VIN), U8.4 (VIN)
- net at U9.10 (P2.1): now also SW6.2
- net at J8.A1 (GND), J8.A12 (GND), J8.B1 (GND)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: now also J8.0 (EH)
- net at U9.9 (P2.0/AXRES): now also SW5.2
- net 2_BUCK_EN: now reaches U12.3 (EN)
- net 2_BUCK_EN: now also U13.1 (P1.0)
- net at U13.10 (P2.1): now also SW8.2
- net at J11.A1 (GND), J11.A12 (GND), J11.B1 (GND)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: now also J11.0 (EH)
- net at U13.9 (P2.0/AXRES): now also SW7.2
- net 1_BUCK_EN: now reaches U8.3 (EN)
- net 1_BUCK_EN: now also U9.1 (P1.0)

Commit message: holyyy i actually finished all of the bare pcb adding lots of art soon:tm:
Signed-off-by: Toby Cm <toby@vsus.app>
Connections:
- net GND: no longer R34.2, U13.22 (GND), U13.25 (GND)
- net 1_D-: now reaches J8.A7 (DN1), J8.B7 (DN2), U9.16 (DM0/P3.1)
- net 1_D+: now reaches J8.A6 (DP1), J8.B6 (DP2), U9.17 (DP0/P3.0)
- net 2_D-: now reaches J11.A7 (DN1), J11.B7 (DN2), U13.16 (DM0/P3.1)
- net 2_D+: now reaches J11.A6 (DP1), J11.B6 (DP2), U13.17 (DP0/P3.0)
- new net: R34.2, U13.22 (GND), U13.25 (GND)
Changed lines of the file:
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@@
 	)
 	(junction
-		(at 242.57 242.57)
-		(diameter 0)
-		(color 0 0 0 0)
-	)
-	(junction
 		(at 26.67 153.67)
 		(diameter 0)
@@
 		)
 	)
+	(label "1_D+"
+		(at 294.64 107.95 0)
+		(effects
+			(font
+				(size 1.27 1.27)
+			)
+			(justify left bottom)
+		)
+	)
+	(label "2_D-"
+		(at 294.724 201.93 0)
+		(effects
+			(font
+				(size 1.27 1.27)
+			)
+			(justify left bottom)
+		)
+	)
+	(label "1_D-"
+		(at 294.724 110.49 0)
+		(effects
+			(font
+				(size 1.27 1.27)
+			)
+			(justify left bottom)
+		)
+	)
+	(label "2_D+"
+		(at 294.64 199.39 0)
+		(effects
+			(font
+				(size 1.27 1.27)
+			)
+			(justify left bottom)
+		)
+	)
 	(global_label "SDA"
 		(shape bidirectional)
@@
 		(exclude_from_sim no)
 		(in_bom yes)
-		(on_board yes)
+		(on_board no)
 		(dnp no)
 		(property "Reference" "SW7"
@@
 	)
 	(symbol
-		(lib_id "power:GND")
-		(at 242.57 242.57 0)
-		(unit 1)
-		(exclude_from_sim no)
-		(in_bom yes)
-		(on_board yes)
-		(dnp no)
-		(fields_autoplaced yes)
-		(property "Reference" "#PWR089"
-			(at 242.57 248.92 0)
-			(effects
-				(font
-					(size 1.27 1.27)
-				)
-				(hide yes)
-			)
-		)
-		(property "Value" "GND"
-			(at 242.57 247.65 0)
-			(effects
-				(font
-					(size 1.27 1.27)
-				)
-			)
-		)
-		(property "Footprint" ""
-			(at 242.57 242.57 0)
-			(effects
-				(font
-					(size 1.27 1.27)
-				)
-				(hide yes)
-			)
-		)
-		(property "Datasheet" ""
-			(at 242.57 242.57 0)
-			(effects
-				(font
-					(size 1.27 1.27)
-				)
-				(hide yes)
-			)
-		)
-		(property "Description" "Power symbol creates a global label with name \"GND\" , ground"
-			(at 242.57 242.57 0)
-			(effects
-				(font
-					(size 1.27 1.27)
-				)
-				(hide yes)
-			)
-		)
-		(pin "1"
-		)
-		(instances
-			(project "usb-charging-hub"
-				(path "/04e54dfe-f06f-40ed-b860-573373578cb0/6cd18a35-eac9-4d54-ab2a-e3d56b6afb11"
-					(reference "#PWR089")
-					(unit 1)
-				)
-			)
-		)
-	)
-	(symbol
 		(lib_id "Device:R_Small")
 		(at 227.33 30.48 180)
@@
 		(exclude_from_sim no)
 		(in_bom yes)
-		(on_board yes)
+		(on_board no)
 		(dnp no)
 		(property "Reference" "SW6"
@@
 		(exclude_from_sim no)
 		(in_bom yes)
-		(on_board yes)
+		(on_board no)
 		(dnp no)
 		(property "Reference" "SW5"
@@
 		(exclude_from_sim no)
 		(in_bom yes)
-		(on_board yes)
+		(on_board no)
 		(dnp no)
 		(property "Reference" "SW8"
