File: usb2.kicad_sch (KiCad schematic)
At the start: 67 parts, among them J13 TYPE-C 16PLT-H10.0, J14 Conn_01x04_Pin, J15 XDUF-0426-081_C18202150, J16 TYPE-C 16PLT-H10.0, J17 Conn_01x04_Pin, Q3 PMOS, Q4 PMOS, U14 XXL1509-5.0, U15 XXL1509-5.0, U16 NDP23511KC, U17 CYPD3175-24LQXQ, U18 LS0505EVD22, U19 LS0505EVD22, U20 NDP23511KC, U21 CYPD3175-24LQXQ

Commit message: finished schematic yay!! now onto pcb routing :fire:
Parts:
- J13, J16: symbol EasyEDA:TYPE-C16PLT-H10.0 -> easyeda2kicad:TYPE-C16PLT-H10.0
- U14, U15: symbol EasyEDA:XXL1509-5.0 -> easyeda2kicad:XXL1509-5.0
Connections:
- net at L9.1, R39.1: now also U16.5 (SW), U16.6 (SW); no longer U16.5,6 (SW)
- net at L10.1, R48.1: now also U20.5 (SW), U20.6 (SW); no longer U20.5,6 (SW)

Commit message: made huge progress today, finished wiring up the rp2040, finished one usb a and usb c layout :fire::fire::fire:
Parts:
- added SW10, SW11, SW12, SW9: Latching, easyeda2kicad:SW-TH_6P-L8.0-W8.0-P2.50, symbol Switch:SW_Push
- U17, U21: footprint Package_DFN_QFN:QFN-24-1EP_4x4mm_P0.5mm_EP2.75x2.75mm -> Package_DFN_QFN:QFN-24-1EP_4x4mm_P0.5mm_EP2.7x2.7mm_ThermalVias
Connections:
- net D_EN: no longer U21.1 (P1.0)
- net GND: now also SW10.1, SW11.1, SW12.1, SW9.1; no longer J13.0 (EH), J16.0 (EH)
- net U_EN: no longer U17.1 (P1.0)
- net VDC: now also U16.4 (VIN), U20.4 (VIN)
- net at U17.10 (P2.1): now also SW10.2
- net SDA: now reaches U17.12 (P2.2)
- net SDA: now also U21.12 (P2.2)
- net SCL: now reaches U17.13 (P2.3)
- net SCL: now also U21.13 (P2.3)
- net at J13.A1 (GND), J13.A12 (GND), J13.B1 (GND)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: now also J13.0 (EH)
- net at U17.9 (P2.0/AXRES): now also SW9.2
- net at U21.10 (P2.1): now also SW12.2
- net at J16.A1 (GND), J16.A12 (GND), J16.B1 (GND)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: now also J16.0 (EH)
- net at U21.9 (P2.0/AXRES): now also SW11.2
- net 1_BUCK_EN: now reaches U16.3 (EN)
- net 1_BUCK_EN: now also U17.1 (P1.0)
- net 2_BUCK_EN: now reaches U20.3 (EN)
- net 2_BUCK_EN: now also U21.1 (P1.0)

Commit message: holyyy i actually finished all of the bare pcb adding lots of art soon:tm:
Signed-off-by: Toby Cm <toby@vsus.app>
Connections:
- net 1_D-: now reaches J13.A7 (DN1), J13.B7 (DN2), U17.16 (DM0/P3.1)
- net 1_D+: now reaches J13.A6 (DP1), J13.B6 (DP2), U17.17 (DP0/P3.0)
- net 2_D-: now reaches J16.A7 (DN1), J16.B7 (DN2), U21.16 (DM0/P3.1)
- net 2_D+: now reaches J16.A6 (DP1), J16.B6 (DP2), U21.17 (DP0/P3.0)
Changed lines of the file:
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@@
 		)
 	)
+	(label "1_D-"
+		(at 294.724 110.49 0)
+		(effects
+			(font
+				(size 1.27 1.27)
+			)
+			(justify left bottom)
+		)
+	)
+	(label "1_D+"
+		(at 294.64 107.95 0)
+		(effects
+			(font
+				(size 1.27 1.27)
+			)
+			(justify left bottom)
+		)
+	)
+	(label "2_D-"
+		(at 294.724 201.93 0)
+		(effects
+			(font
+				(size 1.27 1.27)
+			)
+			(justify left bottom)
+		)
+	)
+	(label "2_D+"
+		(at 294.64 199.39 0)
+		(effects
+			(font
+				(size 1.27 1.27)
+			)
+			(justify left bottom)
+		)
+	)
 	(global_label "SDA"
 		(shape bidirectional)
@@
 		(exclude_from_sim no)
 		(in_bom yes)
-		(on_board yes)
+		(on_board no)
 		(dnp no)
 		(property "Reference" "SW10"
@@
 		(exclude_from_sim no)
 		(in_bom yes)
-		(on_board yes)
+		(on_board no)
 		(dnp no)
 		(property "Reference" "SW11"
@@
 		(exclude_from_sim no)
 		(in_bom yes)
-		(on_board yes)
+		(on_board no)
 		(dnp no)
 		(property "Reference" "SW9"
@@
 		(exclude_from_sim no)
 		(in_bom yes)
-		(on_board yes)
+		(on_board no)
 		(dnp no)
 		(property "Reference" "SW12"
