File: usb3.kicad_sch (KiCad schematic)
At the start: 67 parts, among them J18 TYPE-C 16PLT-H10.0, J19 Conn_01x04_Pin, J20 XDUF-0426-081_C18202150, J21 TYPE-C 16PLT-H10.0, J22 Conn_01x04_Pin, Q5 PMOS, Q6 PMOS, U22 XXL1509-5.0, U23 XXL1509-5.0, U24 NDP23511KC, U25 CYPD3175-24LQXQ, U26 LS0505EVD22, U27 LS0505EVD22, U28 NDP23511KC, U29 CYPD3175-24LQXQ

Commit message: finished schematic yay!! now onto pcb routing :fire:
Parts:
- removed J20: XDUF-0426-081_C18202150, easyeda2kicad:USB-A-TH_XDUF-0426-081, symbol easyeda2kicad:XDUF-0426-081_C18202150
- added J20, J21: GT-USB-7010ASV, easyeda2kicad:USB-C-SMD_G-SWITCH_GT-USB-7010ASV, symbol easyeda2kicad:GT-USB-7010ASV
- added R57, R58, R62, R63: 10k, Resistor_SMD:R_0402_1005Metric_Pad0.72x0.64mm_HandSolder, symbol Device:R_Small
- J18: symbol EasyEDA:TYPE-C16PLT-H10.0 -> easyeda2kicad:TYPE-C16PLT-H10.0
- J22: renamed from J21; symbol EasyEDA:TYPE-C16PLT-H10.0 -> easyeda2kicad:TYPE-C16PLT-H10.0
- U22, U23: symbol EasyEDA:XXL1509-5.0 -> easyeda2kicad:XXL1509-5.0
- renumbered J22 to J23, R58 to R59, R59 to R60, R57 to R61, R60 to R64, R61 to R65, R62 to R66, R63 to R67, R64 to R68, R65 to R69, R66 to R70
Connections:
- net D_D+: now also J21.A6 (DP1), J21.B6 (DP2)
- net D_D-: now also J21.A7 (DN1), J21.B7 (DN2)
- net GND: now also J20.1 (SHELL), J20.2 (SHELL), J20.3 (SHELL), J20.4 (SHELL), J20.A1B12 (GND), J20.B1A12 (GND), J21.1 (SHELL), J21.2 (SHELL), J21.3 (SHELL), J21.4 (SHELL), J21.A1B12 (GND), J21.B1A12 (GND)
- net U_D+: now also J20.A6 (DP1), J20.B6 (DP2)
- net U_D-: now also J20.A7 (DN1), J20.B7 (DN2)
- net at L14.1, R68.1: now also U28.5 (SW), U28.6 (SW); no longer U28.5,6 (SW)
- net at L13.1, R55.1: now also U24.5 (SW), U24.6 (SW); no longer U24.5,6 (SW)
- net at C97.2, C98.2, U26.8 (OUT): now also J20.A4B9 (VBUS), J20.B4A9 (VBUS), R57.1, R58.1
- net at C101.2, C102.2, U27.8 (OUT): now also J21.A4B9 (VBUS), J21.B4A9 (VBUS), R62.1, R63.1
- new net: J20.A5 (CC1), R57.2
- new net: J20.B5 (CC2), R58.2
- new net: J21.A5 (CC1), R62.2
- new net: J21.B5 (CC2), R63.2
Other:
- moved on the sheet: C100, C101, C102, C97, C98, C99, R59, R60, U26

Commit message: made huge progress today, finished wiring up the rp2040, finished one usb a and usb c layout :fire::fire::fire:
Parts:
- added SW13, SW14, SW15, SW16: Latching, easyeda2kicad:SW-TH_6P-L8.0-W8.0-P2.50, symbol Switch:SW_Push
- U25, U29: footprint Package_DFN_QFN:QFN-24-1EP_4x4mm_P0.5mm_EP2.75x2.75mm -> Package_DFN_QFN:QFN-24-1EP_4x4mm_P0.5mm_EP2.7x2.7mm_ThermalVias
Connections:
- net D_EN: no longer U29.1 (P1.0)
- net GND: now also SW13.1, SW14.1, SW15.1, SW16.1; no longer J18.0 (EH), J22.0 (EH)
- net U_EN: no longer U25.1 (P1.0)
- net VDC: now also U24.4 (VIN), U28.4 (VIN)
- net 1_BUCK_EN: now reaches U24.3 (EN)
- net 1_BUCK_EN: now also U25.1 (P1.0)
- net at J22.A1 (GND), J22.A12 (GND), J22.B1 (GND)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: now also J22.0 (EH)
- net at U29.10 (P2.1): now also SW16.2
- net SDA: now reaches U29.12 (P2.2)
- net SDA: now also U25.12 (P2.2)
- net SCL: now reaches U29.13 (P2.3)
- net SCL: now also U25.13 (P2.3)
- net at U29.9 (P2.0/AXRES): now also SW15.2
- net at U25.10 (P2.1): now also SW14.2
- net at J18.A1 (GND), J18.A12 (GND), J18.B1 (GND)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: now also J18.0 (EH)
- net at U25.9 (P2.0/AXRES): now also SW13.2
- net 2_BUCK_EN: now reaches U28.3 (EN)
- net 2_BUCK_EN: now also U29.1 (P1.0)

Commit message: holyyy i actually finished all of the bare pcb adding lots of art soon:tm:
Signed-off-by: Toby Cm <toby@vsus.app>
Connections:
- net 2_D-: now reaches J22.A7 (DN1), J22.B7 (DN2), U29.16 (DM0/P3.1)
- net 2_D+: now reaches J22.A6 (DP1), J22.B6 (DP2), U29.17 (DP0/P3.0)
- net 1_D-: now reaches J18.A7 (DN1), J18.B7 (DN2), U25.16 (DM0/P3.1)
- net 1_D+: now reaches J18.A6 (DP1), J18.B6 (DP2), U25.17 (DP0/P3.0)
Changed lines of the file:
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@@
 		)
 	)
+	(label "2_D-"
+		(at 294.724 201.93 0)
+		(effects
+			(font
+				(size 1.27 1.27)
+			)
+			(justify left bottom)
+		)
+	)
+	(label "1_D-"
+		(at 294.724 110.49 0)
+		(effects
+			(font
+				(size 1.27 1.27)
+			)
+			(justify left bottom)
+		)
+	)
+	(label "1_D+"
+		(at 294.64 107.95 0)
+		(effects
+			(font
+				(size 1.27 1.27)
+			)
+			(justify left bottom)
+		)
+	)
+	(label "2_D+"
+		(at 294.64 199.39 0)
+		(effects
+			(font
+				(size 1.27 1.27)
+			)
+			(justify left bottom)
+		)
+	)
 	(global_label "SDA"
 		(shape bidirectional)
@@
 		(exclude_from_sim no)
 		(in_bom yes)
-		(on_board yes)
+		(on_board no)
 		(dnp no)
 		(property "Reference" "SW15"
@@
 		(exclude_from_sim no)
 		(in_bom yes)
-		(on_board yes)
+		(on_board no)
 		(dnp no)
 		(property "Reference" "SW13"
@@
 		(exclude_from_sim no)
 		(in_bom yes)
-		(on_board yes)
+		(on_board no)
 		(dnp no)
 		(property "Reference" "SW16"
@@
 		(exclude_from_sim no)
 		(in_bom yes)
-		(on_board yes)
+		(on_board no)
 		(dnp no)
 		(property "Reference" "SW14"
