File: usb4.kicad_sch (KiCad schematic)
At the start: 67 parts, among them J23 TYPE-C 16PLT-H10.0, J24 Conn_01x04_Pin, J25 XDUF-0426-081_C18202150, J26 TYPE-C 16PLT-H10.0, J27 Conn_01x04_Pin, Q7 PMOS, Q8 PMOS, U30 XXL1509-5.0, U31 XXL1509-5.0, U32 NDP23511KC, U33 CYPD3175-24LQXQ, U34 LS0505EVD22, U35 LS0505EVD22, U36 NDP23511KC, U37 CYPD3175-24LQXQ

Commit message: finished schematic yay!! now onto pcb routing :fire:
Parts:
- removed J23, J26: TYPE-C 16PLT-H10.0, easyeda2kicad:TYPE-C-SMD_USB4120-03-C, symbol EasyEDA:TYPE-C16PLT-H10.0
- removed J24, J27: Conn_01x04_Pin, Connector_PinHeader_2.54mm:PinHeader_2x02_P2.54mm_Vertical, symbol Connector:Conn_01x04_Pin
- removed J25: XDUF-0426-081_C18202150, easyeda2kicad:USB-A-TH_XDUF-0426-081, symbol easyeda2kicad:XDUF-0426-081_C18202150
- removed R67, R68: 100k, Resistor_SMD:R_0402_1005Metric_Pad0.72x0.64mm_HandSolder, symbol Device:R_Small
- removed R69: 40k, Resistor_SMD:R_0603_1608Metric_Pad0.98x0.95mm_HandSolder, symbol Device:R_Small
- removed R70: 1k, Resistor_SMD:R_0402_1005Metric_Pad0.72x0.64mm_HandSolder, symbol Device:R_Small
- removed U30, U31: XXL1509-5.0, easyeda2kicad:SOIC-8_L4.9-W3.9-P1.27-LS6.0-BL, symbol EasyEDA:XXL1509-5.0
- added J24, J28: TYPE-C 16PLT-H10.0, easyeda2kicad:TYPE-C-SMD_USB4120-03-C, symbol easyeda2kicad:TYPE-C16PLT-H10.0
- added J25, J29: Conn_01x04_Pin, Connector_PinHeader_2.54mm:PinHeader_2x02_P2.54mm_Vertical, symbol Connector:Conn_01x04_Pin
- added J26, J27: GT-USB-7010ASV, easyeda2kicad:USB-C-SMD_G-SWITCH_GT-USB-7010ASV, symbol easyeda2kicad:GT-USB-7010ASV
- added R83, R85, R89: 10k, Resistor_SMD:R_0402_1005Metric_Pad0.72x0.64mm_HandSolder, symbol Device:R_Small
- added R84: 249k, Resistor_SMD:R_0402_1005Metric_Pad0.72x0.64mm_HandSolder, symbol Device:R_Small
- added R86: 40k, Resistor_SMD:R_0603_1608Metric_Pad0.98x0.95mm_HandSolder, symbol Device:R_Small
- added R87: 1k, Resistor_SMD:R_0402_1005Metric_Pad0.72x0.64mm_HandSolder, symbol Device:R_Small
- added R88: 6.8, Resistor_SMD:R_0402_1005Metric_Pad0.72x0.64mm_HandSolder, symbol Device:R_Small
- added R90: 5mOhm 1% Shunt, Resistor_SMD:R_1206_3216Metric_Pad1.30x1.75mm_HandSolder, symbol Device:R_Small
- added U30, U31: XXL1509-5.0, easyeda2kicad:SOIC-8_L4.9-W3.9-P1.27-LS6.0-BL, symbol easyeda2kicad:XXL1509-5.0
- R71: value 6.8 -> 100k
- R72: value 10k -> 100k
- R73: value 5mOhm 1% Shunt -> 40k; footprint Resistor_SMD:R_1206_3216Metric_Pad1.30x1.75mm_HandSolder -> Resistor_SMD:R_0603_1608Metric_Pad0.98x0.95mm_HandSolder
- R74: value 249k -> 1k
- R75: value 10k -> 6.8
- R76: value 249k -> 10k
- R78: value 40k -> 10k; footprint Resistor_SMD:R_0603_1608Metric_Pad0.98x0.95mm_HandSolder -> Resistor_SMD:R_0402_1005Metric_Pad0.72x0.64mm_HandSolder
- R79: value 1k -> 249k
- R80: value 6.8 -> 10k
- R81: value 10k -> 5mOhm 1% Shunt; footprint Resistor_SMD:R_0402_1005Metric_Pad0.72x0.64mm_HandSolder -> Resistor_SMD:R_1206_3216Metric_Pad1.30x1.75mm_HandSolder
- R82: value 5mOhm 1% Shunt -> 10k; footprint Resistor_SMD:R_1206_3216Metric_Pad1.30x1.75mm_HandSolder -> Resistor_SMD:R_0402_1005Metric_Pad0.72x0.64mm_HandSolder
Connections:
- net D_5V: now also U31.3 (FB)
- net D_BUCK_EN: now also R72.2, U31.4 (EN)
- net D_D+: now also J27.A6 (DP1), J27.B6 (DP2)
- net D_D-: now also J27.A7 (DN1), J27.B7 (DN2)
- net D_EN: now also R85.1; no longer R77.1
- net GND: now also R71.1, R72.1, R79.2, R80.2, J24.0 (EH), J25.3 (Pin_3), J25.4 (Pin_4), J26.1 (SHELL), J26.2 (SHELL), J26.3 (SHELL), J26.4 (SHELL), J26.A1B12 (GND), J26.B1A12 (GND), J27.1 (SHELL), J27.2 (SHELL), J27.3 (SHELL), J27.4 (SHELL), J27.A1B12 (GND), J27.B1A12 (GND), J28.0 (EH), J29.3 (Pin_3), J29.4 (Pin_4), R84.2, R85.2, R89.2, R90.2, U30.5 (GND), U30.6 (GND), U30.7 (GND), U30.8 (GND), U31.5 (GND), U31.6 (GND), U31.7 (GND), U31.8 (GND); no longer R72.2, R73.2, R74.2, R75.2, R77.2, R82.2
- net U_5V: now also U30.3 (FB)
- net U_BUCK_EN: now also R71.2, U30.4 (EN)
- net U_D+: now also J26.A6 (DP1), J26.B6 (DP2)
- net U_D-: now also J26.A7 (DN1), J26.B7 (DN2)
- net U_EN: now also R80.1; no longer R75.1
- net VDC: now also U30.1 (VIN), U31.1 (VIN)
- net at C140.1, U36.1 (VFB): now also R86.2, R89.1; no longer R78.2, R81.1
- net at R74.1: now also L17.2, Q7.1 (D), R73.1, U32.2 (VSEN), U33.18 (VBUS_IN_DIS); no longer U34.7 (ILIM)
- net at C140.2, U37.20 (FB): now also R87.2; no longer R79.2
- net at C124.1, U32.1 (VFB): now also R73.2, R76.1; no longer R72.1
- net at U35.7 (ILIM): now also R84.1; no longer R76.1
- net at C131.2, C132.2, U35.8 (OUT): now also R82.1, J27.A4B9 (VBUS), J27.B4A9 (VBUS), R83.1
- net at L18.2, Q8.1 (D), U36.2 (VSEN)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: now also R86.1, R87.1; no longer R78.1, R79.1
- net at C141.1: now also R88.2; no longer R80.2
- net at Q8.3 (S), U37.11 (VBUS_C_MON_DIS): now also J28.A4 (VBUS), J28.A9 (VBUS), J28.B4 (VBUS), J28.B9 (VBUS)
- net at U33.7 (P0.0/SWD_DAT_0): now also J25.1 (Pin_1)
- net at U33.8 (P0.1/SWD_CLK_0): now also J25.2 (Pin_2)
- net at U37.7 (P0.0/SWD_DAT_0): now also J29.1 (Pin_1)
- net at U37.8 (P0.1/SWD_CLK_0): now also J29.2 (Pin_2)
- net at D19.1 (K), L15.1: now also U30.2 (OUTPUT)
- net at C127.2, C128.2, U34.8 (OUT): now also R77.1, R78.1, J26.A4B9 (VBUS), J26.B4A9 (VBUS)
- net at C139.1, U37.15 (CC1): now also J28.A5 (CC1)
- net at C124.2, U33.20 (FB): now also R74.2
- net at C123.1, U33.15 (CC1): now also J24.A5 (CC1)
- net at C122.1, U33.14 (CC2): now also J24.B5 (CC2)
- net at C138.1, U37.14 (CC2): now also J28.B5 (CC2)
- net at D20.1 (K), L16.1: now also U31.2 (OUTPUT)
- net at C125.1: now also R75.2; no longer R71.2
- net at U33.19 (CSP): now also R81.1, J24.A1 (GND), J24.A12 (GND), J24.B1 (GND), J24.B12 (GND); no longer R73.1
- net at Q7.3 (S), U33.11 (VBUS_C_MON_DIS): now also J24.A4 (VBUS), J24.A9 (VBUS), J24.B4 (VBUS), J24.B9 (VBUS)
- net at U33.16 (DM0/P3.1): now also J24.A7 (DN1), J24.B7 (DN2)
- net at U33.17 (DP0/P3.0): now also J24.A6 (DP1), J24.B6 (DP2)
- net at U37.19 (CSP): now also J28.A1 (GND), J28.A12 (GND), J28.B1 (GND), J28.B12 (GND), R90.1; no longer R82.1
- net at U37.17 (DP0/P3.0): now also J28.A6 (DP1), J28.B6 (DP2)
- net at U37.16 (DM0/P3.1): now also J28.A7 (DN1), J28.B7 (DN2)
- new net: J26.A5 (CC1), R77.2
- new net: J26.B5 (CC2), R78.2
- new net: L18.1, R88.1, U36.5 (SW), U36.6 (SW)
- new net: R79.1, U34.7 (ILIM)
- new net: L17.1, R75.1, U32.5 (SW), U32.6 (SW)
- new net: J27.A5 (CC1), R82.2
- new net: J27.B5 (CC2), R83.2

Commit message: made huge progress today, finished wiring up the rp2040, finished one usb a and usb c layout :fire::fire::fire:
Parts:
- added SW17, SW18, SW19, SW20: Latching, easyeda2kicad:SW-TH_6P-L8.0-W8.0-P2.50, symbol Switch:SW_Push
- U33, U37: footprint Package_DFN_QFN:QFN-24-1EP_4x4mm_P0.5mm_EP2.75x2.75mm -> Package_DFN_QFN:QFN-24-1EP_4x4mm_P0.5mm_EP2.7x2.7mm_ThermalVias
Connections:
- net D_EN: no longer U37.1 (P1.0)
- net GND: now also SW17.1, SW18.1, SW19.1, SW20.1; no longer J24.0 (EH), J28.0 (EH)
- net U_EN: no longer U33.1 (P1.0)
- net VDC: now also U32.4 (VIN), U36.4 (VIN)
- net at J24.A1 (GND), J24.A12 (GND), J24.B1 (GND)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: now also J24.0 (EH)
- net 2_BUCK_EN: now reaches U36.3 (EN)
- net 2_BUCK_EN: now also U37.1 (P1.0)
- net at J28.A1 (GND), J28.A12 (GND), J28.B1 (GND)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: now also J28.0 (EH)
- net 1_BUCK_EN: now reaches U32.3 (EN)
- net 1_BUCK_EN: now also U33.1 (P1.0)
- net at U33.10 (P2.1): now also SW18.2
- net SDA: now reaches U33.12 (P2.2)
- net SDA: now also U37.12 (P2.2)
- net SCL: now reaches U33.13 (P2.3)
- net SCL: now also U37.13 (P2.3)
- net at U33.9 (P2.0/AXRES): now also SW17.2
- net at U37.10 (P2.1): now also SW20.2
- net at U37.9 (P2.0/AXRES): now also SW19.2
