File: usb5.kicad_sch (KiCad schematic)
At the start: 67 parts, among them J28 TYPE-C 16PLT-H10.0, J29 Conn_01x04_Pin, J30 XDUF-0426-081_C18202150, J31 TYPE-C 16PLT-H10.0, J32 Conn_01x04_Pin, Q10 PMOS, Q9 PMOS, U38 XXL1509-5.0, U39 XXL1509-5.0, U40 NDP23511KC, U41 CYPD3175-24LQXQ, U42 LS0505EVD22, U43 LS0505EVD22, U44 NDP23511KC, U45 CYPD3175-24LQXQ

Commit message: finished schematic yay!! now onto pcb routing :fire:
Parts:
- J30: renamed from J28; symbol EasyEDA:TYPE-C16PLT-H10.0 -> easyeda2kicad:TYPE-C16PLT-H10.0
- J33: renamed from J31; symbol EasyEDA:TYPE-C16PLT-H10.0 -> easyeda2kicad:TYPE-C16PLT-H10.0
- U38, U39: symbol EasyEDA:XXL1509-5.0 -> easyeda2kicad:XXL1509-5.0
- renumbered J29 to J31, J30 to J32, J32 to J34, R92 to R100, R93 to R101, R94 to R102, R95 to R103, R96 to R104, R97 to R105, R98 to R106, R83 to R91, R84 to R92, R85 to R93, R86 to R94, R87 to R95, R88 to R96, R89 to R97, R90 to R98, R91 to R99
Connections:
- net at L22.1, R104.1: now also U44.5 (SW), U44.6 (SW); no longer U44.5,6 (SW)
- net at L21.1, R95.1: now also U40.5 (SW), U40.6 (SW); no longer U40.5,6 (SW)

Commit message: made huge progress today, finished wiring up the rp2040, finished one usb a and usb c layout :fire::fire::fire:
Parts:
- added SW21, SW22, SW23, SW24: Latching, easyeda2kicad:SW-TH_6P-L8.0-W8.0-P2.50, symbol Switch:SW_Push
Connections:
- net D_EN: no longer U45.1 (P1.0)
- net GND: now also SW21.1, SW22.1, SW23.1, SW24.1; no longer J30.0 (EH), J33.0 (EH)
- net U_EN: no longer U41.1 (P1.0)
- net VDC: now also U40.4 (VIN), U44.4 (VIN)
- net at U41.10 (P2.1): now also SW22.2
- net SDA: now reaches U41.12 (P2.2)
- net SDA: now also U45.12 (P2.2)
- net SCL: now reaches U41.13 (P2.3)
- net SCL: now also U45.13 (P2.3)
- net at J30.A1 (GND), J30.A12 (GND), J30.B1 (GND)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: now also J30.0 (EH)
- net at U41.9 (P2.0/AXRES): now also SW21.2
- net 1_BUCK_EN: now reaches U40.3 (EN)
- net 1_BUCK_EN: now also U41.1 (P1.0)
- net 2_BUCK_EN: now reaches U44.3 (EN)
- net 2_BUCK_EN: now also U45.1 (P1.0)
- net at J33.A1 (GND), J33.A12 (GND), J33.B1 (GND)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: now also J33.0 (EH)
- net at U45.10 (P2.1): now also SW24.2
- net at U45.9 (P2.0/AXRES): now also SW23.2
